File: Schematics/2005903A/2005903A.sch (KiCad schematic (older format))
At the start: 87 parts

Commit message: In the existing schematics, fixed all connectors that I had misinterpreted as global nets.  Found a few connections that didn't quite connect.  All schematics now pass the KiCad ERC.
Parts:
- added J1: ConnectorD8, symbol AGC_DSKY:ConnectorD8
Connections:
- net labels removed: 1, 10, 11, 12, 13, 14, 15, 16, 17, 18, 19, 2, 20, 21, 22, 23, 24, 25, 26, 27, 28, 29, 3, 30, 31, 32, 33, 34, 35, 4, 5, 6, 7, 8, 9
Other:
- note added: "Notes from the Virtual AGC Project:\na) This CAD drawing was manually transcribed from the original Apollo Program \n drawing 2005903A, but is not itself from the time of the Apollo Program — RSB\n 2018\nb) The title-block notation at the lower left of the "MIT" sub-block was illegible in\n the surviving drawing, and has been omitted — RSB 2018\nc) A label in the right-hand border margin reading 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"
- note removed: "Notes from the Virtual AGC Project:\na) This CAD drawing was manually transcribed from the original Apollo Program \n drawing 2005903A, but is not itself from the time of the Apollo Program — RSB\n 2018\nb) The title-block notation at the lower left of the "MIT" sub-block was illegible in\n the surviving drawing, and has been omitted — RSB 2018\nc) A label just outside the right margin of the dra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"

Commit message: On all of the electrical drawings transcribed so far, fixed the visual appearance of the multipart connectors ("ovals") so that they much more-closely match the original drawings, both in terms of the ovals with wires exiting at 90 degrees, and the textual positioning in the oval.
Parts:
- added N35: Node, symbol AGC_DSKY:Node
Connections:
- wire segments 224 -> 225
Changed lines of the file:
@@
 Connection ~ 8000 17400
 Wire Wire Line
-	8700 17950 8700 17400
+	8700 17950 8700 17775
 Wire Wire Line
 	8700 17400 8650 17400
@@
 $Comp
 L AGC_DSKY:ConnectorD8 J1
-U 12 1 5B736B01
-P 8700 18175
-F 0 "J1" H 8425 18400 50  0001 C CNN
-F 1 "ConnectorD8" H 8400 18475 50  0001 C CNN
-F 2 "" H 8550 18350 50  0001 C CNN
-F 3 "" H 8550 18350 50  0001 C CNN
-	12   8700 18175
-	0    -1   -1   0
-$EndComp
-$Comp
-L AGC_DSKY:ConnectorD8 J1
-U 28 1 5B736CCB
-P 9650 18175
-F 0 "J1" H 9375 18400 50  0001 C CNN
-F 1 "ConnectorD8" H 9350 18475 50  0001 C CNN
-F 2 "" H 9500 18350 50  0001 C CNN
-F 3 "" H 9500 18350 50  0001 C CNN
-	28   9650 18175
-	0    -1   -1   0
-$EndComp
-$Comp
-L AGC_DSKY:ConnectorD8 J1
-U 33 1 5B736E48
-P 10675 18175
-F 0 "J1" H 10400 18400 50  0001 C CNN
-F 1 "ConnectorD8" H 10375 18475 50  0001 C CNN
-F 2 "" H 10525 18350 50  0001 C CNN
-F 3 "" H 10525 18350 50  0001 C CNN
-	33   10675 18175
-	0    -1   -1   0
-$EndComp
-$Comp
-L AGC_DSKY:ConnectorD8 J1
-U 29 1 5B737FCA
-P 12125 18175
-F 0 "J1" H 11850 18400 50  0001 C CNN
-F 1 "ConnectorD8" H 11825 18475 50  0001 C CNN
-F 2 "" H 11975 18350 50  0001 C CNN
-F 3 "" H 11975 18350 50  0001 C CNN
-	29   12125 18175
-	0    -1   -1   0
-$EndComp
-$Comp
-L AGC_DSKY:ConnectorD8 J1
-U 31 1 5B739172
-P 13625 18175
-F 0 "J1" H 13350 18400 50  0001 C CNN
-F 1 "ConnectorD8" H 13325 18475 50  0001 C CNN
-F 2 "" H 13475 18350 50  0001 C CNN
-F 3 "" H 13475 18350 50  0001 C CNN
-	31   13625 18175
-	0    -1   -1   0
-$EndComp
-$Comp
-L AGC_DSKY:ConnectorD8 J1
-U 4 1 5B73A7CF
-P 16550 18175
-F 0 "J1" H 16275 18400 50  0001 C CNN
-F 1 "ConnectorD8" H 16250 18475 50  0001 C CNN
-F 2 "" H 16400 18350 50  0001 C CNN
-F 3 "" H 16400 18350 50  0001 C CNN
-	4    16550 18175
-	0    -1   -1   0
-$EndComp
-$Comp
-L AGC_DSKY:ConnectorD8 J1
-U 7 1 5B73BEFA
-P 19550 18175
-F 0 "J1" H 19275 18400 50  0001 C CNN
-F 1 "ConnectorD8" H 19250 18475 50  0001 C CNN
-F 2 "" H 19400 18350 50  0001 C CNN
-F 3 "" H 19400 18350 50  0001 C CNN
-	7    19550 18175
-	0    -1   -1   0
+U 12 2 5B736B01
+P 8700 18125
+F 0 "J1" H 8425 18350 50  0001 C CNN
+F 1 "ConnectorD8" H 8400 18425 50  0001 C CNN
+F 2 "" H 8550 18300 50  0001 C CNN
+F 3 "" H 8550 18300 50  0001 C CNN
+	12   8700 18125
+	1    0    0    -1
+$EndComp
+$Comp
+L AGC_DSKY:ConnectorD8 J1
+U 28 2 5B736CCB
+P 9650 18125
+F 0 "J1" H 9375 18350 50  0001 C CNN
+F 1 "ConnectorD8" H 9350 18425 50  0001 C CNN
+F 2 "" H 9500 18300 50  0001 C CNN
+F 3 "" H 9500 18300 50  0001 C CNN
+	28   9650 18125
+	1    0    0    -1
+$EndComp
+$Comp
+L AGC_DSKY:ConnectorD8 J1
+U 33 2 5B736E48
+P 10675 18125
+F 0 "J1" H 10400 18350 50  0001 C CNN
+F 1 "ConnectorD8" H 10375 18425 50  0001 C CNN
+F 2 "" H 10525 18300 50  0001 C CNN
+F 3 "" H 10525 18300 50  0001 C CNN
+	33   10675 18125
+	1    0    0    -1
+$EndComp
+$Comp
+L AGC_DSKY:ConnectorD8 J1
+U 29 2 5B737FCA
+P 12125 18125
+F 0 "J1" H 11850 18350 50  0001 C CNN
+F 1 "ConnectorD8" H 11825 18425 50  0001 C CNN
+F 2 "" H 11975 18300 50  0001 C CNN
+F 3 "" H 11975 18300 50  0001 C CNN
+	29   12125 18125
+	1    0    0    -1
+$EndComp
+$Comp
+L AGC_DSKY:ConnectorD8 J1
+U 31 2 5B739172
+P 13625 18125
+F 0 "J1" H 13350 18350 50  0001 C CNN
+F 1 "ConnectorD8" H 13325 18425 50  0001 C CNN
+F 2 "" H 13475 18300 50  0001 C CNN
+F 3 "" H 13475 18300 50  0001 C CNN
+	31   13625 18125
+	1    0    0    -1
+$EndComp
+$Comp
+L AGC_DSKY:ConnectorD8 J1
+U 4 2 5B73A7CF
+P 16550 18125
+F 0 "J1" H 16275 18350 50  0001 C CNN
+F 1 "ConnectorD8" H 16250 18425 50  0001 C CNN
+F 2 "" H 16400 18300 50  0001 C CNN
+F 3 "" H 16400 18300 50  0001 C CNN
+	4    16550 18125
+	1    0    0    -1
+$EndComp
+$Comp
+L AGC_DSKY:ConnectorD8 J1
+U 7 2 5B73BEFA
+P 19550 18125
+F 0 "J1" H 19275 18350 50  0001 C CNN
+F 1 "ConnectorD8" H 19250 18425 50  0001 C CNN
+F 2 "" H 19400 18300 50  0001 C CNN
+F 3 "" H 19400 18300 50  0001 C CNN
+	7    19550 18125
+	1    0    0    -1
 $EndComp
 $Comp
@@
 $Comp
 L AGC_DSKY:ConnectorD8 J1
-U 1 1 5B7423EF
-P 16575 1675
-F 0 "J1" H 16300 1900 50  0001 C CNN
-F 1 "ConnectorD8" H 16275 1975 50  0001 C CNN
-F 2 "" H 16425 1850 50  0001 C CNN
-F 3 "" H 16425 1850 50  0001 C CNN
-	1    16575 1675
-	0    1    1    0
-$EndComp
-$Comp
-L AGC_DSKY:ConnectorD8 J1
-U 35 1 5B743D74
-P 14600 1675
-F 0 "J1" H 14325 1900 50  0001 C CNN
-F 1 "ConnectorD8" H 14300 1975 50  0001 C CNN
-F 2 "" H 14450 1850 50  0001 C CNN
-F 3 "" H 14450 1850 50  0001 C CNN
-	35   14600 1675
-	0    1    1    0
-$EndComp
-$Comp
-L AGC_DSKY:ConnectorD8 J1
-U 34 1 5B744032
-P 14000 1675
-F 0 "J1" H 13725 1900 50  0001 C CNN
-F 1 "ConnectorD8" H 13700 1975 50  0001 C CNN
-F 2 "" H 13850 1850 50  0001 C CNN
-F 3 "" H 13850 1850 50  0001 C CNN
-	34   14000 1675
-	0    1    1    0
-$EndComp
-$Comp
-L AGC_DSKY:ConnectorD8 J1
-U 6 1 5B744313
-P 13375 1675
-F 0 "J1" H 13100 1900 50  0001 C CNN
-F 1 "ConnectorD8" H 13075 1975 50  0001 C CNN
-F 2 "" H 13225 1850 50  0001 C CNN
-F 3 "" H 13225 1850 50  0001 C CNN
-	6    13375 1675
-	0    1    1    0
-$EndComp
-$Comp
-L AGC_DSKY:ConnectorD8 J1
-U 2 1 5B7444DC
-P 12800 1675
-F 0 "J1" H 12525 1900 50  0001 C CNN
-F 1 "ConnectorD8" H 12500 1975 50  0001 C CNN
-F 2 "" H 12650 1850 50  0001 C CNN
-F 3 "" H 12650 1850 50  0001 C CNN
-	2    12800 1675
-	0    1    1    0
-$EndComp
-$Comp
-L AGC_DSKY:ConnectorD8 J1
-U 23 1 5B747039
-P 10625 1675
-F 0 "J1" H 10350 1900 50  0001 C CNN
-F 1 "ConnectorD8" H 10325 1975 50  0001 C CNN
-F 2 "" H 10475 1850 50  0001 C CNN
-F 3 "" H 10475 1850 50  0001 C CNN
-	23   10625 1675
-	0    1    1    0
-$EndComp
+U 1 2 5B7423EF
+P 16575 1725
+F 0 "J1" H 16300 1950 50  0001 C CNN
+F 1 "ConnectorD8" H 16275 2025 50  0001 C CNN
+F 2 "" H 16425 1900 50  0001 C CNN
+F 3 "" H 16425 1900 50  0001 C CNN
+	1    16575 1725
+	-1   0    0    1
+$EndComp
+$Comp
+L AGC_DSKY:ConnectorD8 J1
+U 35 2 5B743D74
+P 14600 1725
+F 0 "J1" H 14325 1950 50  0001 C CNN
+F 1 "ConnectorD8" H 14300 2025 50  0001 C CNN
+F 2 "" H 14450 1900 50  0001 C CNN
+F 3 "" H 14450 1900 50  0001 C CNN
+	35   14600 1725
+	-1   0    0    1
+$EndComp
+$Comp
+L AGC_DSKY:ConnectorD8 J1
+U 34 2 5B744032
+P 14000 1725
+F 0 "J1" H 13725 1950 50  0001 C CNN
+F 1 "ConnectorD8" H 13700 2025 50  0001 C CNN
+F 2 "" H 13850 1900 50  0001 C CNN
+F 3 "" H 13850 1900 50  0001 C CNN
+	34   14000 1725
+	-1   0    0    1
+$EndComp
+$Comp
+L AGC_DSKY:ConnectorD8 J1
+U 6 2 5B744313
+P 13375 1725
+F 0 "J1" H 13100 1950 50  0001 C CNN
+F 1 "ConnectorD8" H 13075 2025 50  0001 C CNN
+F 2 "" H 13225 1900 50  0001 C CNN
+F 3 "" H 13225 1900 50  0001 C CNN
+	6    13375 1725
+	-1   0    0    1
+$EndComp
+$Comp
+L AGC_DSKY:ConnectorD8 J1
+U 2 2 5B7444DC
+P 12800 1725
+F 0 "J1" H 12525 1950 50  0001 C CNN
+F 1 "ConnectorD8" H 12500 2025 50  0001 C CNN
+F 2 "" H 12650 1900 50  0001 C CNN
+F 3 "" H 12650 1900 50  0001 C CNN
+	2    12800 1725
+	-1   0    0    1
+$EndComp
+$Comp
+L AGC_DSKY:ConnectorD8 J1
+U 23 2 5B747039
+P 10625 1725
+F 0 "J1" H 10350 1950 50  0001 C CNN
+F 1 "ConnectorD8" H 10325 2025 50  0001 C CNN
+F 2 "" H 10475 1900 50  0001 C CNN
+F 3 "" H 10475 1900 50  0001 C CNN
+	23   10625 1725
+	-1   0    0    1
+$EndComp
+$Comp
+L AGC_DSKY:Node N35
+U 1 1 64D23AC7
+P 8700 17775
+F 0 "N35" H 8700 17875 50  0001 C CNN
+F 1 "Node" H 8700 17950 50  0001 C CNN
+F 2 "" H 8700 17775 50  0001 C CNN
+F 3 "" H 8700 17775 50  0001 C CNN
+	1    8700 17775
+	1    0    0    -1
+$EndComp
+Connection ~ 8700 17775
+Wire Wire Line
+	8700 17775 8700 17400
 $EndSCHEMATC
