File: Schematics/2005937r/2005937r.sch (KiCad schematic (older format))
At the start: 35 parts, among them J1 ConnectorD7, Q1 Transistor-NPN-dual, Q2 Transistor-NPN-big, Q3 Transistor-NPN-big, Q4 Transistor-NPN-dual, T1 Transformer-centertap, T2 Transformer-centertap

Commit message: Added the reconstructed drawing 2005937(r), and corrected minor typo in 2005921-.
Other:
- note added: "2005937"
- note added: "Notes from the Virtual AGC Project:\n1. No surviving copy of drawing 2005937- was known as of the time this CAD file\n was created. It is a recreation of what drawing 2005937- was probably like,\n using an earlier version of the circuit (2005921-) as a model, and supplementing\n it with the circuitry from Figure 4-232 (pp. 4-673/40674) of AC Electronics\n document ND-1021042, which is a redrafted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"
- note added: "TBD"
- note removed: "2005921"
- note removed: "80230"
- note removed: "INITIAL RELEASE PER TDRR"
- note removed: "Notes from the Virtual AGC Project:\n1. This CAD file was manually transcribed from the original Apollo Program\n drawing 2005921-, but did not itself come from the Apollo Program. \n — RSB 2018\n2. A notation in the right-hand margin reading "2005921" has been omitted\n because it would conflict with the label for the "B" area that is there.\n — RSB 2018"
Changed lines of the file:
@@
 EESchema Schematic File Version 4
-LIBS:2005921--cache
+LIBS:2005937r-cache
 EELAYER 26 0
 EELAYER END
@@
 Comment4 ""
 $EndDescr
-Wire Notes Line style solid
-	33500 1175 27953 1175
 Text Notes 29800 19750 0    250  ~ 50
 SCHEMATIC
@@
 MODULE D7
 Text Notes 30875 21150 0    250  ~ 50
-2005921
+2005937
 Text Notes 32400 21425 0    140  ~ 28
 1
@@
 Text Notes 28850 21450 0    140  ~ 28
 NONE
-Text Notes 28275 21100 0    250  ~ 50
-80230
+Text Notes 28575 21100 0    250  ~ 50
+TBD
 $Comp
 L AGC_DSKY:ConnectorD7 J1
@@
 Text Notes 9050 18075 0    130  ~ 26
 REFERENCE\n       1. ASSEMBLY DRAWING NO.2003901
-Text Notes 11000 21150 0    130  ~ 26
-Notes from the Virtual AGC Project:\n1. This CAD file was manually transcribed from the original Apollo Program\n   drawing 2005921-, but did not itself come from the Apollo Program. \n   — RSB 2018\n2. A notation in the right-hand margin reading "2005921" has been omitted\n   because it would conflict with the label for the "B" area that is there.\n   — RSB 2018
+Text Notes 11100 21250 0    130  ~ 26
+Notes from the Virtual AGC Project:\n1. No surviving copy of drawing 2005937- was known as of the time this CAD file\n   was created.  It is a recreation of what drawing 2005937- was probably like,\n   using  an earlier version of the circuit (2005921-) as a model, and supplementing\n   it with the circuitry from Figure 4-232 (pp. 4-673/40674) of AC Electronics\n   document ND-1021042, which is a redrafted form of drawing 2005937.  All known\n   versions of this circuit differ only in resistor and capacitor values. — RSB 2018\n2. Document ND-1021042 explains that the values of resistors R1 & R2, and\n   capacitor C1, were chosen after electrical testing.  The tables at the top of \n   this drawing list the possible substitutions for R1, R2, and C1.  However, this is\n   the list from drawing 2005921-, and it may not be complete. — RSB 2018
 $Bitmap
-Pos 10725 19850
+Pos 10825 19050
 Scale 1.000000
 Data
@@
 Text Notes 17325 4975 0    130  ~ 26
 4500
-Text Notes 28500 1150 0    150  ~ 30
-INITIAL RELEASE PER TDRR
-Wire Notes Line style solid
-	32472 917  32472 1175
-Wire Notes Line style solid
-	31831 917  31831 1175
-Wire Notes Line style solid
-	28453 917  28453 1175
-Wire Notes Line style solid
-	27953 917  27953 1175
 Wire Notes Line style solid
 	18125 5250 15375 5250

Commit message: On all of the electrical drawings transcribed so far, fixed the visual appearance of the multipart connectors ("ovals") so that they much more-closely match the original drawings, both in terms of the ovals with wires exiting at 90 degrees, and the textual positioning in the oval.
Changed lines of the file:
@@
 $Comp
 L AGC_DSKY:ConnectorD7 J1
-U 9 1 5B70E926
-P 17475 8875
-F 0 "J1" H 17475 9100 50  0001 C CNN
-F 1 "ConnectorD7" H 17500 9175 50  0001 C CNN
-F 2 "" H 17425 9050 50  0001 C CNN
-F 3 "" H 17425 9050 50  0001 C CNN
-	9    17475 8875
-	0    -1   1    0
+U 9 2 5B70E926
+P 17475 8925
+F 0 "J1" H 17475 9150 50  0001 C CNN
+F 1 "ConnectorD7" H 17500 9225 50  0001 C CNN
+F 2 "" H 17425 9100 50  0001 C CNN
+F 3 "" H 17425 9100 50  0001 C CNN
+	9    17475 8925
+	1    0    0    1
 $EndComp
 $Comp
@@
 $Comp
 L AGC_DSKY:ConnectorD7 J1
-U 2 1 5B70EB01
-P 18525 17175
-F 0 "J1" H 18525 17400 50  0001 C CNN
-F 1 "ConnectorD7" H 18550 17475 50  0001 C CNN
-F 2 "" H 18475 17350 50  0001 C CNN
-F 3 "" H 18475 17350 50  0001 C CNN
-	2    18525 17175
-	0    -1   -1   0
+U 2 2 5B70EB01
+P 18525 17125
+F 0 "J1" H 18525 17350 50  0001 C CNN
+F 1 "ConnectorD7" H 18550 17425 50  0001 C CNN
+F 2 "" H 18475 17300 50  0001 C CNN
+F 3 "" H 18475 17300 50  0001 C CNN
+	2    18525 17125
+	1    0    0    -1
 $EndComp
 $Comp
 L AGC_DSKY:ConnectorD7 J1
-U 12 1 5B70EC02
-P 19000 8875
-F 0 "J1" H 19000 9100 50  0001 C CNN
-F 1 "ConnectorD7" H 19025 9175 50  0001 C CNN
-F 2 "" H 18950 9050 50  0001 C CNN
-F 3 "" H 18950 9050 50  0001 C CNN
-	12   19000 8875
-	0    1    1    0
+U 12 2 5B70EC02
+P 19000 8925
+F 0 "J1" H 19000 9150 50  0001 C CNN
+F 1 "ConnectorD7" H 19025 9225 50  0001 C CNN
+F 2 "" H 18950 9100 50  0001 C CNN
+F 3 "" H 18950 9100 50  0001 C CNN
+	12   19000 8925
+	-1   0    0    1
 $EndComp
 $Comp
@@
 $Comp
 L AGC_DSKY:ConnectorD7 J1
-U 1 1 5B710008
-P 23175 8850
-F 0 "J1" H 23175 9075 50  0001 C CNN
-F 1 "ConnectorD7" H 23200 9150 50  0001 C CNN
-F 2 "" H 23125 9025 50  0001 C CNN
-F 3 "" H 23125 9025 50  0001 C CNN
-	1    23175 8850
-	0    1    1    0
+U 1 2 5B710008
+P 23175 8900
+F 0 "J1" H 23175 9125 50  0001 C CNN
+F 1 "ConnectorD7" H 23200 9200 50  0001 C CNN
+F 2 "" H 23125 9075 50  0001 C CNN
+F 3 "" H 23125 9075 50  0001 C CNN
+	1    23175 8900
+	-1   0    0    1
 $EndComp
 $Comp
@@
 $Comp
 L AGC_DSKY:ConnectorD7 J1
-U 10 1 5B7113E2
-P 25200 17200
-F 0 "J1" H 25200 17425 50  0001 C CNN
-F 1 "ConnectorD7" H 25225 17500 50  0001 C CNN
-F 2 "" H 25150 17375 50  0001 C CNN
-F 3 "" H 25150 17375 50  0001 C CNN
-	10   25200 17200
-	0    -1   -1   0
+U 10 2 5B7113E2
+P 25200 17150
+F 0 "J1" H 25200 17375 50  0001 C CNN
+F 1 "ConnectorD7" H 25225 17450 50  0001 C CNN
+F 2 "" H 25150 17325 50  0001 C CNN
+F 3 "" H 25150 17325 50  0001 C CNN
+	10   25200 17150
+	1    0    0    -1
 $EndComp
 $Comp

Commit message: Standardized styling of library symbols to more-closely match appearance of the original drawings.  Updated all of the CAD drawings accordingly. Added a BASH script (dependent on sed and ImageMagick) to post-process KiCad schematics plotted to Postscript, to give back PNGs instead. Juiced up the connector-creation script to allow for physically omitted pins on the connectors.
Changed lines of the file:
@@
 L AGC_DSKY:ConnectorD7 J1
 U 3 1 5B70B39C
-P 1950 10250
-F 0 "J1" H 1950 10475 50  0001 C CNN
-F 1 "ConnectorD7" H 1975 10550 50  0001 C CNN
-F 2 "" H 1900 10425 50  0001 C CNN
-F 3 "" H 1900 10425 50  0001 C CNN
-	3    1950 10250
+P 1900 10250
+F 0 "J1" H 1900 10475 50  0001 C CNN
+F 1 "ConnectorD7" H 1925 10550 50  0001 C CNN
+F 2 "" H 1850 10425 50  0001 C CNN
+F 3 "" H 1850 10425 50  0001 C CNN
+	3    1900 10250
 	1    0    0    -1
 $EndComp
@@
 L AGC_DSKY:ConnectorD7 J1
 U 7 1 5B70B3C9
-P 1950 11900
-F 0 "J1" H 1950 12125 50  0001 C CNN
-F 1 "ConnectorD7" H 1975 12200 50  0001 C CNN
-F 2 "" H 1900 12075 50  0001 C CNN
-F 3 "" H 1900 12075 50  0001 C CNN
-	7    1950 11900
+P 1900 11900
+F 0 "J1" H 1900 12125 50  0001 C CNN
+F 1 "ConnectorD7" H 1925 12200 50  0001 C CNN
+F 2 "" H 1850 12075 50  0001 C CNN
+F 3 "" H 1850 12075 50  0001 C CNN
+	7    1900 11900
 	1    0    0    -1
 $EndComp
@@
 L AGC_DSKY:ConnectorD7 J1
 U 5 1 5B70B43D
-P 1950 13475
-F 0 "J1" H 1950 13700 50  0001 C CNN
-F 1 "ConnectorD7" H 1975 13775 50  0001 C CNN
-F 2 "" H 1900 13650 50  0001 C CNN
-F 3 "" H 1900 13650 50  0001 C CNN
-	5    1950 13475
+P 1900 13475
+F 0 "J1" H 1900 13700 50  0001 C CNN
+F 1 "ConnectorD7" H 1925 13775 50  0001 C CNN
+F 2 "" H 1850 13650 50  0001 C CNN
+F 3 "" H 1850 13650 50  0001 C CNN
+	5    1900 13475
 	1    0    0    -1
 $EndComp
@@
 L AGC_DSKY:ConnectorD7 J1
 U 11 1 5B70B484
-P 1950 15125
-F 0 "J1" H 1950 15350 50  0001 C CNN
-F 1 "ConnectorD7" H 1975 15425 50  0001 C CNN
-F 2 "" H 1900 15300 50  0001 C CNN
-F 3 "" H 1900 15300 50  0001 C CNN
-	11   1950 15125
+P 1900 15125
+F 0 "J1" H 1900 15350 50  0001 C CNN
+F 1 "ConnectorD7" H 1925 15425 50  0001 C CNN
+F 2 "" H 1850 15300 50  0001 C CNN
+F 3 "" H 1850 15300 50  0001 C CNN
+	11   1900 15125
 	1    0    0    -1
 $EndComp
@@
 L AGC_DSKY:ConnectorD7 J1
 U 6 1 5B71155A
-P 27125 14225
-F 0 "J1" H 27125 14450 50  0001 C CNN
-F 1 "ConnectorD7" H 27150 14525 50  0001 C CNN
-F 2 "" H 27075 14400 50  0001 C CNN
-F 3 "" H 27075 14400 50  0001 C CNN
-	6    27125 14225
+P 27175 14225
+F 0 "J1" H 27175 14450 50  0001 C CNN
+F 1 "ConnectorD7" H 27200 14525 50  0001 C CNN
+F 2 "" H 27125 14400 50  0001 C CNN
+F 3 "" H 27125 14400 50  0001 C CNN
+	6    27175 14225
 	-1   0    0    1
 $EndComp
@@
 L AGC_DSKY:ConnectorD7 J1
 U 4 1 5B711638
-P 27125 12800
-F 0 "J1" H 27125 13025 50  0001 C CNN
-F 1 "ConnectorD7" H 27150 13100 50  0001 C CNN
-F 2 "" H 27075 12975 50  0001 C CNN
-F 3 "" H 27075 12975 50  0001 C CNN
-	4    27125 12800
+P 27175 12800
+F 0 "J1" H 27175 13025 50  0001 C CNN
+F 1 "ConnectorD7" H 27200 13100 50  0001 C CNN
+F 2 "" H 27125 12975 50  0001 C CNN
+F 3 "" H 27125 12975 50  0001 C CNN
+	4    27175 12800
 	-1   0    0    1
 $EndComp
@@
 L AGC_DSKY:ConnectorD7 J1
 U 8 1 5B711797
-P 27125 10025
-F 0 "J1" H 27125 10250 50  0001 C CNN
-F 1 "ConnectorD7" H 27150 10325 50  0001 C CNN
-F 2 "" H 27075 10200 50  0001 C CNN
-F 3 "" H 27075 10200 50  0001 C CNN
-	8    27125 10025
+P 27175 10025
+F 0 "J1" H 27175 10250 50  0001 C CNN
+F 1 "ConnectorD7" H 27200 10325 50  0001 C CNN
+F 2 "" H 27125 10200 50  0001 C CNN
+F 3 "" H 27125 10200 50  0001 C CNN
+	8    27175 10025
 	-1   0    0    1
 $EndComp
@@
 	4325 11875 4225 11875
 NoConn ~ 4225 11875
-Text Notes 1650 10325 2    130  ~ 26
+Text Notes 1600 10325 2    130  ~ 26
 14VSW
-Text Notes 1650 11975 2    130  ~ 26
+Text Notes 1600 11975 2    130  ~ 26
 POTHI
-Text Notes 1650 13550 2    130  ~ 26
+Text Notes 1600 13550 2    130  ~ 26
 POTLO
-Text Notes 1650 15200 2    130  ~ 26
+Text Notes 1600 15200 2    130  ~ 26
 800CPS
 Text Notes 22750 16225 2    130  ~ 26
@@
 Text Notes 24200 17875 0    130  ~ 26
       OSGRD\n(OFF SEGMENT GRD)
-Text Notes 27325 14000 2    130  ~ 26
+Text Notes 27375 14000 2    130  ~ 26
 EVLO
-Text Notes 27375 12575 2    130  ~ 26
+Text Notes 27425 12575 2    130  ~ 26
 EV250
-Text Notes 27375 9775 2    130  ~ 26
+Text Notes 27425 9775 2    130  ~ 26
 EVHII
-Text Notes 27450 10100 0    130  ~ 26
+Text Notes 27500 10100 0    130  ~ 26
 (VERB-NOUN FLASH)
 Text Notes 22600 8550 0    130  ~ 26
