File: Schematics/fixed_erasable_memory/fixed_erasable_memory-1.sch (KiCad schematic (older format))
At the start: 92 parts, among them J1 ConnectorA1-100, U101 D3NOR-+4SW-0VDCA-ABC-_E_, U102 D3NOR-+4SW-0VDCA-_B_-DEF, U103 D3NOR-+4SW-0VDCA-ABC-_E_, U104 D3NOR-+4SW-0VDCA-ABC-D_F, U105 D3NOR-+4SW-0VDCA-A_C-D_F, U106 D3NOR-+4SW-0VDCA-ABC-_E_, U107 D3NOR-+4SW-0VDCA-ABC-D_F, U108 D3NOR-+4SW-0VDCA-_B_-DEF, U109 D3NOR-+4SW-0VDCA-A_C-D_F, U110 D3NOR-+4SW-0VDCA-ABC-DEF, U111 D3NOR-+4SW-0VDCA-ABC-D_F, U112 D3NOR-+4SW-0VDCA-A_C-D_F, U113 D3NOR-+4SW-0VDCA-_B_-D_F, U114 D3NOR-+4SW-0VDCA-A_C-D_F, U115 D3NOR-+4SW-0VDCA-A_C-D_F, U116 D3NOR-+4SW-0VDCA-A_C-D_F, U117 D3NOR-+4SW-0VDCA-A_C-D_F, U118 D3NOR-+4SW-0VDCA-A_C-D_F, U119 D3NOR-+4SW-0VDCA-_B_-D_F, U120 D3NOR-+4SW-0VDCA-_B_-DEF, U121 D3NOR-+4SW-0VDCA-_B_-_E_, U122 D3NOR-+4SW-0VDCA-A_C-D_F, U123 D3NOR-+4SW-0VDCA-A_C-_E_, U124 D3NOR-+4SW-0VDCA-A_C-D_F, U125 D3NOR-+4SW-0VDCA-_B_-D_F, U126 D3NOR-+4SW-0VDCA-_B_-D_F, U127 D3NOR-+4SW-0VDCA-A_C-D_F, U128 D3NOR-+4SW-0VDCA-_B_-D_F, U129 D3NOR-+4SW-0VDCA-_B_-_E_, U130 D3NOR-+4SW-0VDCA-_B_-_E_, U131 D3NOR-+4SW-0VDCA-_B_-D_F, U132 D3NOR-+4SW-0VDCA-_B_-_E_, U133 D3NOR-+4SW-0VDCA-_B_-_E_, U134 D3NOR-+4SW-0VDCA-_B_-D_F, U135 D3NOR-+4SW-0VDCA-_B_-_E_, U136 D3NOR-+4SW-0VDCA-_B_-_E_, U137 D3NOR-+4SW-0VDCA-A_C-D_F, U138 D3NOR-+4SW-0VDCA-A_C-D_F, U139 D3NOR-+4SW-0VDCA-_B_-_E_, U140 D3NOR-+4SW-0VDCA-_B_-_E_, U141 D3NOR-+4SW-0VDCA-_B_-_E_, U142 D3NOR-+4SW-0VDCA-_B_-DEF, X201 Node2, X202 Node2, X203 Node2, X204 Node2, X205 Node2, X206 Node2, X207 Node2, X208 Node2, X210 Node2, X211 Node2, X212 Node2, X213 Node2, X214 Node2, X215 Node2, X216 Node2, X217 Node2, X218 Node2, X219 Node2, X220 Node2, X221 Node2, X222 Node2, X223 Node2, X224 Node2, X225 Node2, X226 Node2, X227 Node2, X228 Node2, X229 Node2

Commit message: Tweaking fixed_erasable_memory, to try and reach the point where its connectivity to the backplane matches Mike's.  Not there yet, but making progress.
Parts:
- removed unit 7 of J1
- removed unit 3 of J1
- removed unit 2 of J1
- removed unit 1 of J1
- removed unit 6 of J1
- removed unit 5 of J1
- removed unit 4 of J1
- removed unit 9 of J1
- removed unit 8 of J1
- removed unit 49 of J1
- removed unit 50 of J1
- removed unit 52 of J1
- removed unit 48 of J1
- removed unit 47 of J1
- removed unit 46 of J1
- removed unit 45 of J1
- removed unit 44 of J1
- removed unit 43 of J1
- removed unit 42 of J1
- removed unit 25 of J1
- removed unit 53 of J1
- removed unit 20 of J1
- removed unit 23 of J1
- removed unit 22 of J1
- removed unit 24 of J1
- removed unit 12 of J1
- removed unit 13 of J1
- removed unit 14 of J1
- removed unit 15 of J1
- removed unit 16 of J1
- removed unit 17 of J1
- removed unit 18 of J1
- removed unit 19 of J1
- removed unit 10 of J1
- removed unit 11 of J1
- added N221, N? (x7): Node2, symbol AGC_DSKY:Node2
Connections:
- net STR19: now reaches U137.2 (C), U137.6 (D)
- net STR19: now also U118.4 (A), N?.1
- net STR311: now reaches U137.8 (F)
- net STR311: now also U118.6 (D), N?.1
- net LOMOD: now reaches U101.3 (B), U103.3 (B), U106.3 (B), U107.3 (B), U110.3 (B), U111.3 (B), U113.6 (D)
- net CLROPE: now reaches U115.4 (A), U116.6 (D), U127.6 (D)
- net RESETC: now reaches U117.4 (A), U134.8 (F)
- net RESETA: now reaches U114.4 (A), U128.8 (F)
- net RESETA: now also U123.7 (E), N?.1
- net RESETB: now reaches U115.6 (D), U131.8 (F)
- net RESETB: now also U121.3 (B)
- net STR210: now reaches U118.2 (C)
- net STR210: now also U137.4 (A), N?.1
- net STR412: now reaches U118.8 (F)
- net SBF: now reaches U119.3 (B)
- net STR14: now reaches U101.2 (C), U103.2 (C), U106.2 (C), U106.7 (E), U110.2 (C)
- net STR912: now reaches U104.2 (C), U108.3 (B), U108.8 (F)
- net ROPER: now reaches U101.7 (E), U102.6 (D), U106.4 (A)
- net ROPER: now also U120.6 (D), N221.1
- net ROPES: now reaches U102.3 (B), U103.4 (A), U108.6 (D), U110.4 (A)
- net ROPES: now also U120.7 (E), N?.1
- net ROPET: now reaches U103.7 (E), U104.4 (A), U107.4 (A)
- net ROPET: now also U120.8 (F), N?.1
- net HIMOD: now reaches U104.3 (B), U107.8 (F), U108.7 (E), U110.7 (E), U112.6 (D)
- net STR58: now reaches U112.8 (F), U113.3 (B)
- net IL03: now reaches U141.3 (B)
- net IL02: now reaches U141.7 (E)
- net IL01: now reaches U142.3 (B)
- net IL05: now reaches U140.3 (B)
- net IL04: now reaches U140.7 (E)
- net IL06: now reaches U139.7 (E)
- net IL07: now reaches U139.3 (B)
- net RESETD: now reaches U126.3 (B)
- net SETAB: now reaches U121.7 (E)
- net SETCD: now reaches U125.3 (B)

Commit message: Finished reworking of my version of fixed_erasable_memory schematics, and I think it now very closely matches Mike's, except that I have AGC style NOR gates and 69-pin connectors rather than the 74-series NOR gates and DIN connectors Mike used, so some translation, presumably at the netlist level, would be needed to exactly match the two.
Parts:
- removed J1: ConnectorA1-100, symbol AGC_DSKY:ConnectorA1-100
- removed N201, N202, N203, N204, N205, N206, N207, N208, N209, N210, N211, N212, N213, N214, N215, N216, N217, N218, N219, N220, N221, N? (x7), X201, X202, X203, X204, X205, X206, X207, X208, X210, X211, X212, X213, X214, X215, X216, X217, X218, X219, X220, X221, X222, X223, X224, X225, X226, X227, X228, X229: Node2, symbol AGC_DSKY:Node2
Connections:
- net CQA: now also U122.8 (F)
- net CQB: now also U124.8 (F)
- net CQC: now also U127.2 (C)
- net SA01: now reaches B1.29 (DQ0)
- net SA09: now reaches B1.30 (DQ8)
- net SA02: now reaches B1.31 (DQ1)
- net SA10: now reaches B1.32 (DQ9)
- net SA03: now reaches B1.33 (DQ2)
- net SA11: now reaches B1.34 (DQ10)
- net SA04: now reaches B1.35 (DQ3)
- net SA12: now reaches B1.36 (DQ11)
- net SA05: now reaches B1.38 (DQ4)
- net SA13: now reaches B1.39 (DQ12)
- net SA06: now reaches B1.40 (DQ5)
- net SA14: now reaches B1.41 (DQ13)
- net SA07: now reaches B1.42 (DQ6)
- net SAP: now reaches B1.43 (DQ14)
- net SA08: now reaches B1.44 (DQ7)
- net SA16: now reaches B1.45 (DQ15)
- no-connect marks 16 -> 0
Other:
- note removed: "SPARE PINS"

Commit message: Made several corrections to the fixed_erasable_memory drawings, but I believe they were just corrections to the notes.
Parts:
- renumbered B1 to U1
Changed lines of the file:
@@
 $EndDescr
 Text Notes 1375 33125 0    140  ~ 28
-Notes from the Virtual AGC Project:\n1. Though having an MIT/MSC title block, this\n   drawing was not transcribed from an Apollo\n   Project drawing.  It is a memory interface to\n   original Apollo Project AGC design, intended \n   to assist in Verilog simulation or synthesis of \n   logically-compatible designs. — RSB 2018\n2. To conform to the conventions of original\n   Apollo Program drawings, reference \n   designators are not shown on components.\n   For the purposes of ERC and netlist generation, \n   NOR gates have reference designators U1nn, \n   where nn is the 2-digit number shown on the\n   NOR gate.  The oval pads numbered 101-171\n   comprise connector J1, while those numbered\n   201-271 comprise connector J2. — RSB 2018\n3. This design is based on similarly-named\n   drawings and Verilog memory interfaces by\n   Mike Stewart. — RSB 2018
+Notes from the Virtual AGC Project:\n1. Though having an MIT/MSC title block, this\n   drawing was not transcribed from an Apollo\n   Project drawing.  It is a memory interface to\n   original Apollo Project AGC design, intended \n   to assist in Verilog simulation or synthesis of \n   logically-compatible designs. — RSB 2018\n2. To conform to the conventions of original\n   Apollo Program drawings, reference \n   designators are not shown on NOR gates.\n   For the purposes of ERC and netlist generation, \n   NOR gates have reference designators U1nn, \n   where nn is the 2-digit number shown on the\n   NOR gate. — RSB 2018\n3. This design is based on similarly-named\n   drawings and Verilog memory interfaces by\n   Mike Stewart. — RSB 2018
 $Comp
 L D3NOR-+4SW-0VDCA:D3NOR-+4SW-0VDCA-_B_-_E_ U129
@@
 NOROPE
 $Bitmap
-Pos 1075 28875
+Pos 1100 29350
 Scale 1.000000
 Data
@@
 $EndBitmap
 $Comp
-L AGC_DSKY:ROM B1
+L AGC_DSKY:ROM U1
 U 1 1 5BDECA96
 P 32400 2825
-AR Path="/5BDECA96" Ref="B1"  Part="1"
-AR Path="/5B8E7731/5BDECA96" Ref="B1"  Part="1"
-F 0 "B1" H 32400 2825 140 0001 C CNN
+F 0 "U1" H 32225 2750 140 0000 C CNB
 F 1 "ROM" H 32400 2825 140 0001 C CNN
 F 2 "" H 32400 2825 140 0001 C CNN
