File: Schematics/2005256A/2005256A-p2of2.sch (KiCad schematic (older format))
At the start: 66 parts, among them J3 ConnectorA1-300, J4 ConnectorA1-400, U201 D3NOR-+4SW-0VDCA-B_C-EDF, U202 D3NOR-+4SW-0VDCA-B_C-E_F, U203 D3NOR-+4SW-0VDCA-ABC-DEF, U204 D3NOR-+4SW-0VDCA-B_C-E_F, U205 D3NOR-FAP-0VDCA-expander-ACB-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, U206 D3NOR-+4SW-0VDCA-B_C-DFE, U207 D3NOR-+4SW-0VDCA-B_C-E_F, U208 D3NOR-+4SW-0VDCA-B_C-EDF, U209 D3NOR-+4SW-0VDCA-ABC-E_F, U210 D3NOR-+4SW-0VDCA-B_C-E_F, U211 D3NOR-+4SW-0VDCA-B_C-E_F, U212 D3NOR-+4SW-0VDCA-B_C-DFE, U213 D3NOR-+4SW-0VDCA-B_C-E_F, U214 D3NOR-+4SW-0VDCA-B_C-_F_, U215 D3NOR-+4SW-0VDCA-B_C-E_F, U216 D3NOR-+4SW-0VDCA-B_C-E_F, U217 D3NOR-+4SW-0VDCA-BAC-DEF, U218 D3NOR-FAP-0VDCA-expander-B_C-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, U219 D3NOR-+4SW-0VDCA-B_C-E_F, U220 D3NOR-+4SW-0VDCA-B_C-E_F, U221 D3NOR-FAP-0VDCA-expander-ABC-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, U222 D3NOR-+4SW-0VDCA-B_C-DFE, U223 D3NOR-+4SW-0VDCA-B_C-E_F, U224 D3NOR-+4SW-0VDCA-B_C-E_F, U225 D3NOR-+4SW-0VDCA-B_C-E_F, U226 D3NOR-+4SW-0VDCA-B_C-_F_, U227 D3NOR-FAP-0VDCA-expander-ACB-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, U228 D3NOR-+4SW-0VDCA-B_C-_F_, U229 D3NOR-+4SW-0VDCA-B_C-_F_, U230 D3NOR-+4SW-0VDCA-B_C-_F_, U231 D3NOR-+4SW-0VDCA-B_C-EDF, U232 D3NOR-+4SW-0VDCA-B_C-E_F, U233 D3NOR-+4SW-0VDCA-ABC-DEF, U234 D3NOR-+4SW-0VDCA-B_C-E_F, U235 D3NOR-+4SW-0VDCA-B_C-E_F, U236 D3NOR-FAP-0VDCA-expander-ACB-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, U237 D3NOR-+4SW-0VDCA-B_C-E_F, U238 D3NOR-+4SW-0VDCA-B_C-EDF, U239 D3NOR-+4SW-0VDCA-ABC-E_F, U240 D3NOR-+4SW-0VDCA-B_C-E_F, U241 D3NOR-+4SW-0VDCA-B_C-E_F, U242 D3NOR-+4SW-0VDCA-B_C-DEF, U243 D3NOR-+4SW-0VDCA-B_C-E_F, U244 D3NOR-+4SW-0VDCA-B_C-_F_, U245 D3NOR-+4SW-0VDCA-B_C-DEF, U246 D3NOR-+4SW-0VDCA-B_C-E_F, U247 D3NOR-+4SW-0VDCA-ABC-DEF, U248 D3NOR-FAP-0VDCA-expander-B_C-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, U249 D3NOR-+4SW-0VDCA-B_C-E_F, U250 D3NOR-+4SW-0VDCA-B_C-E_F, U251 D3NOR-FAP-0VDCA-expander-ABC-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, U252 D3NOR-+4SW-0VDCA-B_C-DFE, U253 D3NOR-+4SW-0VDCA-B_C-E_F, U254 D3NOR-+4SW-0VDCA-B_C-E_F, U255 D3NOR-+4SW-0VDCA-B_C-E_F, U256 D3NOR-+4SW-0VDCA-B_C-_F_, U257 D3NOR-FAP-0VDCA-expander-ACB-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, U258 D3NOR-+4SW-0VDCA-B_C-_F_, U259 D3NOR-+4SW-0VDCA-B_C-_F_, U260 D3NOR-+4SW-0VDCA-B_C-_F_, X301 ArrowTwiddle, X302 ArrowTwiddle, X303 ArrowTwiddle

Commit message: Completed 2005258A CAD files.  As with 2005256A and 2005257A, it was simply adapted from the original 2005255- transcription, and hence errors could easily have slipped through which need to be detected in proofing (that hasn't yet been performed).
Parts:
- J4: Caption CGA8 -> CGA9
Changed lines of the file:
@@
 F 2 "" H 36575 28650 140 0001 C CNN
 F 3 "" H 36575 28650 140 0001 C CNN
-F 4 "CGA8" H 35925 28200 140 0000 C CNB "Caption"
+F 4 "CGA9" H 35925 28200 140 0000 C CNB "Caption"
 	1    36575 28175
 	-1   0    0    1

Commit message: Resolved all issues vs pin database in module A1-A8 schematics that remained after yesterday's mods.
Parts:
- J3: Caption PIPAY+ -> PIPAY+/
- J3, J4: Caption (none) -> 0VDCA
- J3: Caption PIPAX- -> PIPAX-/
- J3, J4: Caption (none) -> +4SW
- J4: Caption SUMMA07/ -> SUMA07/
Changed lines of the file:
@@
 F 2 "" H 40450 25175 140 0001 C CNN
 F 3 "" H 40450 25175 140 0001 C CNN
-F 4 "" H 40450 25000 140 0000 C CNB "Caption"
+F 4 "0VDCA" H 40450 25000 140 0001 C CNB "Caption"
 	12   40450 24700
 	1    0    0    -1
@@
 F 2 "" H 36575 26150 140 0001 C CNN
 F 3 "" H 36575 26150 140 0001 C CNN
-F 4 "" H 36575 25975 140 0000 C CNB "Caption"
+F 4 "0VDCA" H 36575 25975 140 0001 C CNB "Caption"
 	60   36575 25675
 	1    0    0    -1
@@
 F 2 "" H 34900 14000 140 0001 C CNN
 F 3 "" H 34900 14000 140 0001 C CNN
-F 4 "PIPAY+" H 34250 13550 140 0000 C CNB "Caption"
+F 4 "PIPAY+/" H 34150 13550 140 0000 C CNB "Caption"
 	56   34900 13525
 	1    0    0    -1
@@
 F 2 "" H 40425 26150 140 0001 C CNN
 F 3 "" H 40425 26150 140 0001 C CNN
-F 4 "" H 40425 25975 140 0000 C CNB "Caption"
+F 4 "0VDCA" H 40425 25975 140 0001 C CNB "Caption"
 	60   40425 25675
 	1    0    0    -1
@@
 F 2 "" H 40450 25650 140 0001 C CNN
 F 3 "" H 40450 25650 140 0001 C CNN
-F 4 "" H 40450 25475 140 0000 C CNB "Caption"
+F 4 "0VDCA" H 40450 25475 140 0001 C CNB "Caption"
 	36   40450 25175
 	1    0    0    -1
@@
 F 2 "" H 40425 27475 140 0001 C CNN
 F 3 "" H 40425 27475 140 0001 C CNN
-F 4 "" H 40425 27300 140 0000 C CNB "Caption"
+F 4 "+4SW" H 40425 27300 140 0001 C CNB "Caption"
 	48   40425 27000
 	1    0    0    -1
@@
 F 2 "" H 36575 26950 140 0001 C CNN
 F 3 "" H 36575 26950 140 0001 C CNN
-F 4 "" H 36575 26775 140 0000 C CNB "Caption"
+F 4 "+4SW" H 36575 26775 140 0001 C CNB "Caption"
 	24   36575 26475
 	1    0    0    -1
@@
 F 2 "" H 34900 12675 140 0001 C CNN
 F 3 "" H 34900 12675 140 0001 C CNN
-F 4 "PIPAX-" H 34200 12225 140 0000 C CNB "Caption"
+F 4 "PIPAX-/" H 34100 12225 140 0000 C CNB "Caption"
 	15   34900 12200
 	1    0    0    -1
@@
 F 2 "" H 40425 26975 140 0001 C CNN
 F 3 "" H 40425 26975 140 0001 C CNN
-F 4 "" H 40425 26800 140 0000 C CNB "Caption"
+F 4 "+4SW" H 40425 26800 140 0001 C CNB "Caption"
 	24   40425 26500
 	1    0    0    -1
@@
 F 2 "" H 36600 25150 140 0001 C CNN
 F 3 "" H 36600 25150 140 0001 C CNN
-F 4 "" H 36600 24975 140 0000 C CNB "Caption"
+F 4 "0VDCA" H 36600 24975 140 0001 C CNB "Caption"
 	12   36600 24675
 	1    0    0    -1
@@
 F 2 "" H 12875 4175 140 0001 C CNN
 F 3 "" H 12875 4175 140 0001 C CNN
-F 4 "SUMMA07/" H 13025 4025 140 0000 C CNB "Caption"
+F 4 "SUMA07/" H 13025 4025 140 0000 C CNB "Caption"
 	33   12875 3700
 	1    0    0    -1
