File: msSchematics/four_bit_2/two_bit_columns.sch (KiCad schematic (older format))
At the start: 48 parts, among them U8004 74HC27, U8009 74HC02, U8017 74HC27, U8021 74HC02, U8022 74HC27, U8033 74HC02, U8035 74HC02, U8036 74HC27, U8037 74HC02, U8038 74HC27, U8039 74HC04, U8040 74HC02, U8041 74LVC07, U8042 74HC27, U8043 74HC02, U8044 74HC27, U8045 74HC02, U8046 74HC02, U8047 74HC02, U8048 74HC02, U8049 74HC27, U8050 74LVC07, U8051 74HC02, U8052 74HC4002, U8053 74HC02, U8054 74HC27, U8055 74HC02, U8056 74HC02, U8057 74HC27, U8058 74HC02, U8059 74HC27, U8060 74HC02, U8061 74LVC07, U8062 74HC02, U8063 74HC02, U8064 74HC02, U8065 74HC04, U8066 74HC4002, U8068 74LVC06

Commit message: I seem to have lost the resistors in the first commit.  Hopefully that's fixed now.
Parts:
- R8011, R8012, R8013, R8015, R8016, R8017, R8018, R8019, R8020: symbol device:R -> four_bit_2-rescue:R-device
Changed lines of the file:
@@
 EESchema Schematic File Version 4
-EELAYER 28 0
+LIBS:four_bit_2-cache
+EELAYER 29 0
 EELAYER END
 $Descr A2 23386 16535
@@
 	8200 1100 8200 1050
 $Comp
-L device:R R8011
+L four_bit_2-rescue:R-device R8011
 U 1 1 56853F32
 P 8200 900
@@
 AR Path="/568CD527/56853F32" Ref="R11001"  Part="1"
 AR Path="/568CD532/56853F32" Ref="R11011"  Part="1"
+AR Path="/56853F32" Ref="R9011"  Part="1"
 F 0 "R9011" V 8280 900 50  0000 C CNN
 F 1 "5k" V 8200 900 50  0000 C CNN
@@
 $EndComp
 $Comp
-L device:R R8012
+L four_bit_2-rescue:R-device R8012
 U 1 1 56859114
 P 8800 3500
@@
 AR Path="/568CD527/56859114" Ref="R11002"  Part="1"
 AR Path="/568CD532/56859114" Ref="R11012"  Part="1"
+AR Path="/56859114" Ref="R9012"  Part="1"
 F 0 "R9012" V 8880 3500 50  0000 C CNN
 F 1 "5k" V 8800 3500 50  0000 C CNN
@@
 	4750 5550 3850 5550
 $Comp
-L device:R R8013
+L four_bit_2-rescue:R-device R8013
 U 1 1 56862FDE
 P 4750 5100
@@
 AR Path="/568CD527/56862FDE" Ref="R11003"  Part="1"
 AR Path="/568CD532/56862FDE" Ref="R11013"  Part="1"
+AR Path="/56862FDE" Ref="R9013"  Part="1"
 F 0 "R9013" V 4830 5100 50  0000 C CNN
 F 1 "5k" V 4750 5100 50  0000 C CNN
@@
 	6650 5300 6650 6500
 $Comp
-L device:R R8015
+L four_bit_2-rescue:R-device R8015
 U 1 1 56875BCB
 P 4750 8000
@@
 AR Path="/568CD527/56875BCB" Ref="R11005"  Part="1"
 AR Path="/568CD532/56875BCB" Ref="R11015"  Part="1"
+AR Path="/56875BCB" Ref="R9015"  Part="1"
 F 0 "R9015" V 4830 8000 50  0000 C CNN
 F 1 "5k" V 4750 8000 50  0000 C CNN
@@
 Connection ~ 5400 12750
 $Comp
-L device:R R8016
+L four_bit_2-rescue:R-device R8016
 U 1 1 568920B9
 P 5400 12100
@@
 AR Path="/568CD527/568920B9" Ref="R11006"  Part="1"
 AR Path="/568CD532/568920B9" Ref="R11016"  Part="1"
+AR Path="/568920B9" Ref="R9016"  Part="1"
 F 0 "R9016" V 5480 12100 50  0000 C CNN
 F 1 "5k" V 5400 12100 50  0000 C CNN
@@
 $EndComp
 $Comp
-L device:R R8017
+L four_bit_2-rescue:R-device R8017
 U 1 1 568B9EF2
 P 19550 3500
@@
 AR Path="/568CD527/568B9EF2" Ref="R11007"  Part="1"
 AR Path="/568CD532/568B9EF2" Ref="R11017"  Part="1"
+AR Path="/568B9EF2" Ref="R9017"  Part="1"
 F 0 "R9017" V 19630 3500 50  0000 C CNN
 F 1 "5k" V 19550 3500 50  0000 C CNN
@@
 _WL_EXTRA2_2
 $Comp
-L device:R R8019
+L four_bit_2-rescue:R-device R8019
 U 1 1 568B9FE7
 P 15500 8000
@@
 AR Path="/568CD527/568B9FE7" Ref="R11009"  Part="1"
 AR Path="/568CD532/568B9FE7" Ref="R11019"  Part="1"
+AR Path="/568B9FE7" Ref="R9019"  Part="1"
 F 0 "R9019" V 15580 8000 50  0000 C CNN
 F 1 "5k" V 15500 8000 50  0000 C CNN
@@
 $EndComp
 $Comp
-L device:R R8018
+L four_bit_2-rescue:R-device R8018
 U 1 1 568B9F7B
 P 15500 5100
@@
 AR Path="/568CD527/568B9F7B" Ref="R11008"  Part="1"
 AR Path="/568CD532/568B9F7B" Ref="R11018"  Part="1"
+AR Path="/568B9F7B" Ref="R9018"  Part="1"
 F 0 "R9018" V 15580 5100 50  0000 C CNN
 F 1 "5k" V 15500 5100 50  0000 C CNN
@@
 Connection ~ 16150 12750
 $Comp
-L device:R R8020
+L four_bit_2-rescue:R-device R8020
 U 1 1 568BA085
 P 16150 12100
@@
 AR Path="/568CD527/568BA085" Ref="R11010"  Part="1"
 AR Path="/568CD532/568BA085" Ref="R11020"  Part="1"
+AR Path="/568BA085" Ref="R9020"  Part="1"
 F 0 "R9020" V 16230 12100 50  0000 C CNN
 F 1 "5k" V 16150 12100 50  0000 C CNN
