File: msSchematics/inout_ii/a17_1.sch (KiCad schematic (older format))
At the start: 54 parts, among them U17001 74HC02, U17002 74HC04, U17003 74LVC07, U17004 74HC02, U17005 74HC02, U17006 74HC27, U17007 74HC02, U17008 74HC27, U17009 74HC02, U17010 74HC02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

Commit message: I seem to have lost the resistors in the first commit.  Hopefully that's fixed now.
Parts:
- R17001, R17002, R17003, R17004, R17005, R17006, R17007, R17008, R17009, R17010, R17011, R17012, R17013, R17014, R17015, R17016, R17017, R17018: symbol device:R -> inout_ii-rescue:R-device
