File: msSchematics/inout_v/a22_1.sch (KiCad schematic (older format))
At the start: 33 parts, among them U22001 74HC02, U22002 74HC27, U22003 74HC04, U22004 74HC02, U22005 74HC02, U22006 74HC27, U22007 74HC02, U22008 74HC04, U22009 74HC27, U22010 74HC02, U22011 74HC27, U22012 74HC02, U22013 74HC27, U22014 74HC04, U22015 74HC02, U22016 74HC27, U22017 74HC02, U22018 74HC02, U22019 74HC02, U22020 74HC04, U22021 74HC02, U22022 74HC27, U22023 74HC04, U22024 74HC27, U22025 74HC27, U22026 74HC02, U22027 74HC27, U22028 74LVC07, U22029 74HC02, U22068 74HC27, U22130 74HC27, U22131 74HC04

Commit message: I seem to have lost the resistors in the first commit.  Hopefully that's fixed now.
Parts:
- R22001: symbol device:R -> inout_v-rescue:R-device
Changed lines of the file:
@@
 Connection ~ 20800 8550
 $Comp
-L device:R R22001
+L inout_v-rescue:R-device R22001
 U 1 1 572D7077
 P 20800 8350
+AR Path="/572D7077" Ref="R22001"  Part="1"
+AR Path="/5726BFDE/572D7077" Ref="R22001"  Part="1"
 F 0 "R22001" V 20880 8350 50  0000 C CNN
 F 1 "5k" V 20800 8350 50  0000 C CNN
