File: msSchematics/parity_s_register/a12_1.sch (KiCad schematic (older format))
At the start: 33 parts, among them U12001 74HC04, U12002 74HC27, U12003 74HC27, U12004 74HC4002, U12005 74HC04, U12006 74HC27, U12007 74HC27, U12008 74HC4002, U12009 74HC04, U12010 74HC27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

Commit message: I seem to have lost the resistors in the first commit.  Hopefully that's fixed now.
Parts:
- R12001, R12002, R12003, R12004: symbol device:R -> parity_s_register-rescue:R-device
Changed lines of the file:
@@
 $EndComp
 $Comp
-L device:R R12001
+L parity_s_register-rescue:R-device R12001
 U 1 1 56B2175D
 P 10650 3950
@@
 $EndComp
 $Comp
-L device:R R12002
+L parity_s_register-rescue:R-device R12002
 U 1 1 56B158D1
 P 16250 4950
@@
 $EndComp
 $Comp
-L device:R R12003
+L parity_s_register-rescue:R-device R12003
 U 1 1 56B21848
 P 16250 6150
@@
 Connection ~ 20950 11600
 $Comp
-L device:R R12004
+L parity_s_register-rescue:R-device R12004
 U 1 1 56B98837
 P 20950 11400
