File: Schematics/2005920B/2005920B-p2of2.sch (KiCad schematic (older format))
At the start: 0 parts

Commit message: Completed the CAD transcription of drawing 2005920B.
Other:
- note added: "-"
- note added: "-119"
- note added: "-121"
- note added: "-122"
- note added: "-123"
- note added: "-124"
- note added: "-125"
- note added: "-126"
- note added: "-127"
- note added: "-128"
- note added: "-129"
- note added: "-130"
- note added: "-16"
- note added: "-17"
- note added: "-18"
- note added: "-19"
- note added: "-20"
- note added: "-21"
- note added: "-22"
- note added: "-23"
- note added: "-24"
- note added: "-25"
- note added: "-26"
- note added: "-27"
- note added: "-28"
- note added: "-29"
- note added: "-30"
- note added: "-31"
- note added: "-32"
- note added: "-33"
- note added: "-34"
- note added: "-35"
- note added: "-36"
- note added: "-37"
- note added: "-38"
- note added: "-39"
- note added: "-40"
- note added: "-41"
- note added: "-42"
- note added: "-43"
- note added: "-44"
- note added: "-45"
- note added: "-46"
- note added: "-47"
- note added: "-48"
- note added: "-49"
- note added: "001"
- note added: "002"
- note added: "0VDC"
- note added: "1"
- note added: "1 UF"
- note added: "1/4 W"
- note added: "1/4W"
- note added: "1000"
- note added: "1006293"
- note added: "1006750"
- note added: "1006750-"
- note added: "1006755-69"
- note added: "101"
- note added: "102"
- note added: "104"
- note added: "105"
- note added: "107"
- note added: "109"
- note added: "110"
- note added: "1100"
- note added: "113"
- note added: "114"
- note added: "116"
- note added: "118"
- note added: "12"
- note added: "120"
- note added: "1200"
- note added: "121"
- note added: "123"
- note added: "125"
- note added: "127"
- note added: "1300"
- note added: "136"
- note added: "138"
- note added: "140"
- note added: "1400"
- note added: "142"
- note added: "143"
- note added: "145"
- note added: "147"
- note added: "15"
- note added: "150"
- note added: "1500"
- note added: "151"
- note added: "152"
- note added: "154"
- note added: "156"
- note added: "157"
- note added: "158"
- note added: "1600"
- note added: "162"
- note added: "164"
- note added: "1700"
- note added: "1800"
- note added: "1900"
- note added: "2"
- note added: "2 2"
- note added: "200"
- note added: "2000"
- note added: "2004003-001"
- note added: "2004004"
- note added: "2004004-002"
- note added: "2004103-001"
- note added: "2004112-002"
- note added: "2005920"
- note added: "201"
- note added: "202"
- note added: "203"
- note added: "204"
- note added: "205"
- note added: "207"
- note added: "208"
- note added: "209"
- note added: "20K"
- note added: "210"
- note added: "2100"
- note added: "212"
- note added: "214"
- note added: "215"
- note added: "216"
- note added: "218"
- note added: "219"
- note added: "220"
- note added: "2200"
- note added: "221"
- note added: "222"
- note added: "223"
- note added: "225"
- note added: "226"
- note added: "2300"
- note added: "233"
- note added: "237"
- note added: "238"
- note added: "239"
- note added: "24"
- note added: "240"
- note added: "2400"
- note added: "241"
- note added: "242"
- note added: "244"
- note added: "245"
- note added: "246"
- note added: "248"
- note added: "249"
- note added: "25"
- note added: "252"
- note added: "253"
- note added: "255"
- note added: "2550"
- note added: "256"
- note added: "258"
- note added: "260"
- note added: "261"
- note added: "262"
- note added: "263"
- note added: "265"
- note added: "270"
- note added: "2700"
- note added: "2850"
- note added: "3"
- note added: "300"
- note added: "3000"
- note added: "3150"
- note added: "32"
- note added: "330"
- note added: "3300"
- note added: "3450"
- note added: "35VDC"
- note added: "36"
- note added: "360"
- note added: "3600"
- note added: "3750"
- note added: "39"
- note added: "390"
- note added: "3900"
- note added: "4"
- note added: "400611"
- note added: "400613"
- note added: "400615"
- note added: "400617"
- note added: "400619"
- note added: "400621"
- note added: "400623"
- note added: "400625"
- note added: "40601"
- note added: "40602"
- note added: "40603"
- note added: "40604"
- note added: "40605"
- note added: "40606"
- note added: "40607"
- note added: "40608"
- note added: "4100"
- note added: "43"
- note added: "430"
- note added: "4300"
- note added: "470"
- note added: "4700"
- note added: "49"
- note added: "5"
- note added: "510"
- note added: "5100"
- note added: "560"
- note added: "6"
- note added: "620"
- note added: "63"
- note added: "680"
- note added: "7"
- note added: "750"
- note added: "8"
- note added: "80230"
- note added: "820"
- note added: "910"
- note added: "A"
- note added: "B"
- note added: "B13"
- note added: "C"
- note added: "C1"
- note added: "C2"
- note added: "C3"
- note added: "C4"
- note added: "CAPACITOR"
- note added: "CHART A"
- note added: "CHART B"
- note added: "COMP\nPREFIX\n NO."
- note added: "CR1"
- note added: "CR10"
- note added: "CR11"
- note added: "CR12"
- note added: "CR13"
- note added: "CR14"
- note added: "CR15"
- note added: "CR16"
- note added: "CR17"
- note added: "CR2"
- note added: "CR3"
- note added: "CR4"
- note added: "CR5"
- note added: "CR6"
- note added: "CR7"
- note added: "CR8"
- note added: "CR9"
- note added: "D"
- note added: "DESCRIPTION"
- note added: "DIODE"
- note added: "E"
- note added: "ERASABLE MEMORY B13"
- note added: "F"
- note added: "G"
- note added: "H"
- note added: "I"
- note added: "J"
- note added: "NOM"
- note added: "NONE"
- note added: "PART NO."
- note added: "PIN NO."
- note added: "Q1"
- note added: "Q10"
- note added: "Q11"
- note added: "Q2"
- note added: "Q3"
- note added: "Q4"
- note added: "Q5"
- note added: "Q6"
- note added: "Q7"
- note added: "Q8"
- note added: "Q9"
- note added: "R1"
- note added: "R10"
- note added: "R11"
- note added: "R12"
- note added: "R13"
- note added: "R14"
- note added: "R15"
- note added: "R16"
- note added: "R17"
- note added: "R18"
- note added: "R19"
- note added: "R2"
- note added: "R20"
- note added: "R21"
- note added: "R22"
- note added: "R23"
- note added: "R23, R27 AND R32"
- note added: "R24"
- note added: "R25"
- note added: "R26"
- note added: "R27"
- note added: "R28"
- note added: "R29"
- note added: "R3"
- note added: "R30"
- note added: "R31"
- note added: "R32"
- note added: "R33"
- note added: "R34"
- note added: "R35"
- note added: "R36"
- note added: "R37"
- note added: "R38"
- note added: "R4"
- note added: "R5"
- note added: "R6"
- note added: "R7"
- note added: "R8"
- note added: "R9"
- note added: "R9 AND R10"
- note added: "RATING"
- note added: "REF DES"
- note added: "RELEASED PER TDRR"
- note added: "RESISTOR"
- note added: "REVISED PER TDRR 29077\nDR CHK APPD"
- note added: "REVISED PER TDRR 29821\nDR CHK APPD"
- note added: "SA02"
- note added: "SA04"
- note added: "SA06"
- note added: "SA08"
- note added: "SA1"
- note added: "SA10"
- note added: "SA12"
- note added: "SA14"
- note added: "SA16"
- note added: "SA2"
- note added: "SAF 01"
- note added: "SAF 02"
- note added: "SAF 03"
- note added: "SAF 04"
- note added: "SAF 05"
- note added: "SAF 06"
- note added: "SAF 07"
- note added: "SAF 08"
- note added: "SAF 09"
- note added: "SAF 10"
- note added: "SAF 11"
- note added: "SAF 12"
- note added: "SAF 13"
- note added: "SAF 14"
- note added: "SAF 15"
- note added: "SAF 16"
- note added: "SBF 01"
- note added: "SBF 02"
- note added: "SBF 03"
- note added: "SBF 04"
- note added: "SBF 05"
- note added: "SBF 06"
- note added: "SBF 07"
- note added: "SBF 08"
- note added: "SBF 09"
- note added: "SBF 10"
- note added: "SBF 11"
- note added: "SBF 12"
- note added: "SBF 13"
- note added: "SBF 14"
- note added: "SBF 15"
- note added: "SBF 16"
- note added: "SCHEMATIC"
- note added: "SEE CHART A"
- note added: "SEE CHART B"
- note added: "SENSE AMPL"
- note added: "SENSE AMPLIFIER MODULE,"
- note added: "SIGNAL"
- note added: "T1"
- note added: "T2"
- note added: "TOL"
- note added: "TRANSFORMER"
- note added: "TRANSISTOR"
- note added: "VALUE"
- note added: "VYE"
- note added: "___"
- note added: "_____"
- note added: "____________"
- note added: "{"
- note added: "±10%"
- note added: "±2%"
