File: Schematics/2005920B/original.sch (KiCad schematic (older format))
At the start: 0 parts

Commit message: Completed the CAD transcription of drawing 2005920B.
Other:
- note added: "-"
- note added: "2005920"
- note added: "80230"
- note added: "A"
- note added: "B"
- note added: "ERASABLE MEMORY B13"
- note added: "NONE"
- note added: "RELEASED PER TDRR"
- note added: "REVISED PER TDRR 29077\nDR CHK APPD"
- note added: "REVISED PER TDRR 29821\nDR CHK APPD"
- note added: "SCHEMATIC"
- note added: "SENSE AMPLIFIER MODULE,"
- note added: "___"
- note added: "_____"
- note added: "____________"
Changed lines of the file:
@@
 Text Notes 1550 32850 0    500  ~ 100
 NOTE: The sheets of this CAD drawing are \nintended to match only the appearance\nof the original Apollo Program drawing,\nand are not ELECTRICALLY valid.
+Wire Notes Line style solid
+	37958 910  37958 2290
+Wire Notes Line style solid
+	37968 2290 43493 2290
+Wire Notes Line style solid
+	37968 1715 43493 1715
+Wire Notes Line style solid
+	42458 910  42458 2290
+Wire Notes Line style solid
+	41793 910  41793 2290
+Wire Notes Line style solid
+	38458 910  38458 2290
+Text Notes 38118 1540 0    140  ~ 28
+A
+Text Notes 38118 2090 0    140  ~ 28
+B
+Text Notes 38543 1665 0    140  ~ 28
+REVISED PER TDRR 29077\nDR     CHK      APPD
+Text Notes 38543 2240 0    140  ~ 28
+REVISED PER TDRR 29821\nDR     CHK      APPD
+Wire Notes Line style solid
+	43493 1165 37968 1165
+Text Notes 38093 1115 0    140  ~ 28
+-
+Text Notes 38543 1140 0    140  ~ 28
+RELEASED PER TDRR
+Text Notes 39659 31724 0    250  ~ 50
+SCHEMATIC
+Text Notes 40884 33124 0    250  ~ 50
+2005920
+Text Notes 38259 33124 0    250  ~ 50
+80230
+Text Notes 38659 32074 0    200  ~ 40
+SENSE AMPLIFIER MODULE,
+Text Notes 38909 32399 0    200  ~ 40
+ERASABLE MEMORY B13
+Text Notes 33509 32324 0    140  ~ 28
+____________
+Text Notes 33509 32899 0    140  ~ 28
+____________
+Text Notes 33509 33374 0    140  ~ 28
+____________
+Wire Notes Line style solid
+	34009 33424 34134 33249
+Text Notes 35109 31774 0    140  ~ 28
+___
+Text Notes 34134 31774 0    140  ~ 28
+___
+Text Notes 33134 31774 0    140  ~ 28
+___
+Wire Notes Line style solid
+	33284 31799 33359 31699
+Wire Notes Line style solid
+	34309 31799 34384 31699
+Wire Notes Line style solid
+	35284 31799 35359 31699
+Text Notes 40334 33424 0    140  ~ 28
+_____
+Wire Notes Line style solid
+	40559 33449 40659 33349
+Text Notes 38809 33474 0    140  ~ 28
+NONE
+Wire Notes Line style solid
+	34109 33424 34234 33249
+Wire Notes Line style solid
+	34109 32949 34234 32774
+Wire Notes Line style solid
+	34009 32949 34134 32774
+Wire Notes Line style solid
+	34109 32374 34234 32199
+Wire Notes Line style solid
+	34009 32374 34134 32199
+Wire Notes Line style solid
+	33234 31799 33309 31699
+Wire Notes Line style solid
+	34259 31799 34334 31699
+Wire Notes Line style solid
+	35234 31799 35309 31699
 $EndSCHEMATC
