File: Schematics/Block-I-A33/Fig-4-181.sch (KiCad schematic (older format))
At the start: 14 parts

Commit message: I've completed inputting the A33 schematics from ND-1021041.  There are several connector pads that are either definitely misnumbered or else likely renumbered ... but without any way to cross-check them against anything else as far as I know.  For now, I've arbitrarily replaced some with otherwise unused pads that they could plausibly be typos for.  My next step is to superimpose the A34 schematics atop this, and that may reveal some of the correct answers.
Parts:
- gave numbers to parts that had none: 5
Changed lines of the file:
@@
 $EndDescr
 $Comp
-L AGC_DSKY:ConnectorGeneric J?
+L AGC_DSKY:ConnectorGeneric J1
 U 23 1 5BF0114A
 P 4450 2850
-F 0 "J?" H 4450 3175 140 0001 C CNN
+F 0 "J1" H 4450 3175 140 0001 C CNN
 F 1 "ConnectorGeneric" H 4450 3275 140 0001 C CNN
 F 2 "" H 4450 3025 140 0001 C CNN
@@
 $EndComp
 $Comp
-L AGC_DSKY:ConnectorGeneric J?
+L AGC_DSKY:ConnectorGeneric J1
 U 24 1 5BF1AECC
 P 4450 5575
-F 0 "J?" H 4450 5900 140 0001 C CNN
+F 0 "J1" H 4450 5900 140 0001 C CNN
 F 1 "ConnectorGeneric" H 4450 6000 140 0001 C CNN
 F 2 "" H 4450 5750 140 0001 C CNN
@@
 $EndComp
 $Comp
-L AGC_DSKY:ConnectorGeneric J?
+L AGC_DSKY:ConnectorGeneric J1
 U 47 1 5BF28105
 P 4450 1650
-F 0 "J?" H 4450 1975 140 0001 C CNN
+F 0 "J1" H 4450 1975 140 0001 C CNN
 F 1 "ConnectorGeneric" H 4450 2075 140 0001 C CNN
 F 2 "" H 4450 1825 140 0001 C CNN
@@
 $EndComp
 $Comp
-L AGC_DSKY:ConnectorGeneric J?
+L AGC_DSKY:ConnectorGeneric J1
 U 48 1 5BF31F8C
 P 4450 4375
-F 0 "J?" H 4450 4700 140 0001 C CNN
+F 0 "J1" H 4450 4700 140 0001 C CNN
 F 1 "ConnectorGeneric" H 4450 4800 140 0001 C CNN
 F 2 "" H 4450 4550 140 0001 C CNN
@@
 $EndComp
 $Comp
-L AGC_DSKY:ConnectorGeneric J?
+L AGC_DSKY:ConnectorGeneric J1
 U 71 1 5BF42565
 P 4450 3250
-F 0 "J?" H 4450 3575 140 0001 C CNN
+F 0 "J1" H 4450 3575 140 0001 C CNN
 F 1 "ConnectorGeneric" H 4450 3675 140 0001 C CNN
 F 2 "" H 4450 3425 140 0001 C CNN
@@
 $EndComp
 $Comp
-L AGC_DSKY:ConnectorGeneric J?
+L AGC_DSKY:ConnectorGeneric J1
 U 72 1 5BF4A0A2
 P 4450 5975
-F 0 "J?" H 4450 6300 140 0001 C CNN
+F 0 "J1" H 4450 6300 140 0001 C CNN
 F 1 "ConnectorGeneric" H 4450 6400 140 0001 C CNN
 F 2 "" H 4450 6150 140 0001 C CNN
@@
 $EndComp
 $Comp
-L AGC_DSKY:ConnectorGeneric J?
+L AGC_DSKY:ConnectorGeneric J1
 U 95 1 5BF5221C
 P 4450 2050
-F 0 "J?" H 4450 2375 140 0001 C CNN
+F 0 "J1" H 4450 2375 140 0001 C CNN
 F 1 "ConnectorGeneric" H 4450 2475 140 0001 C CNN
 F 2 "" H 4450 2225 140 0001 C CNN
@@
 $EndComp
 $Comp
-L AGC_DSKY:ConnectorGeneric J?
+L AGC_DSKY:ConnectorGeneric J1
 U 96 1 5BF5534D
 P 4450 4775
-F 0 "J?" H 4450 5100 140 0001 C CNN
+F 0 "J1" H 4450 5100 140 0001 C CNN
 F 1 "ConnectorGeneric" H 4450 5200 140 0001 C CNN
 F 2 "" H 4450 4950 140 0001 C CNN
@@
 $EndComp
 $Comp
-L AGC_DSKY:ConnectorGeneric J?
+L AGC_DSKY:ConnectorGeneric J1
 U 119 1 5BF5A7AF
 P 4450 3650
-F 0 "J?" H 4450 3975 140 0001 C CNN
+F 0 "J1" H 4450 3975 140 0001 C CNN
 F 1 "ConnectorGeneric" H 4450 4075 140 0001 C CNN
 F 2 "" H 4450 3825 140 0001 C CNN
@@
 $EndComp
 $Comp
-L AGC_DSKY:ConnectorGeneric J?
+L AGC_DSKY:ConnectorGeneric J1
 U 120 1 5BF5DC10
 P 4450 6375
-F 0 "J?" H 4450 6700 140 0001 C CNN
+F 0 "J1" H 4450 6700 140 0001 C CNN
 F 1 "ConnectorGeneric" H 4450 6800 140 0001 C CNN
 F 2 "" H 4450 6550 140 0001 C CNN
@@
 $EndComp
 $Comp
-L AGC_DSKY:Capacitor C?
+L AGC_DSKY:Capacitor C501
 U 1 1 5C08E632
 P 5800 2200
-F 0 "C?" H 5965 2213 130 0001 L CNN
+F 0 "C501" H 5965 2213 130 0001 L CNN
 F 1 "Capacitor" H 6350 2000 130 0001 C CNN
 F 2 "" H 5800 2600 130 0001 C CNN
@@
 $EndComp
 $Comp
-L AGC_DSKY:Capacitor C?
+L AGC_DSKY:Capacitor C503
 U 1 1 5C08EFFD
 P 6575 2200
-F 0 "C?" H 6740 2213 130 0001 L CNN
+F 0 "C503" H 6740 2213 130 0001 L CNN
 F 1 "Capacitor" H 7125 2000 130 0001 C CNN
 F 2 "" H 6575 2600 130 0001 C CNN
@@
 Connection ~ 6575 1650
 $Comp
-L AGC_DSKY:Capacitor C?
+L AGC_DSKY:Capacitor C502
 U 1 1 5C0914F3
 P 5800 4925
-F 0 "C?" H 5965 4938 130 0001 L CNN
+F 0 "C502" H 5965 4938 130 0001 L CNN
 F 1 "Capacitor" H 6350 4725 130 0001 C CNN
 F 2 "" H 5800 5325 130 0001 C CNN
@@
 $EndComp
 $Comp
-L AGC_DSKY:Capacitor C?
+L AGC_DSKY:Capacitor C504
 U 1 1 5C0914FD
 P 6575 4925
-F 0 "C?" H 6740 4938 130 0001 L CNN
+F 0 "C504" H 6740 4938 130 0001 L CNN
 F 1 "Capacitor" H 7125 4725 130 0001 C CNN
 F 2 "" H 6575 5325 130 0001 C CNN

Commit message: I've been adding various Block I module-A34 things to the module-A33 schematics.  It's going well, but it's slow-going.
Parts:
- J1: Caption2 (none) -> 0VDC
- J1: Caption2 (none) -> +3A
Changed lines of the file:
@@
 F 2 "" H 4450 3025 140 0001 C CNN
 F 3 "" H 4450 3025 140 0001 C CNN
-F 4 "0VDC" H 3600 2475 140 0000 C CNB "Caption"
+F 4 "0VDC" H 3600 2550 140 0000 C CNB "Caption"
+F 5 "0VDC" H 3600 2350 140 0000 C CNB "Caption2"
 	23   4450 2850
 	1    0    0    -1
@@
 F 2 "" H 4450 5750 140 0001 C CNN
 F 3 "" H 4450 5750 140 0001 C CNN
-F 4 "0VDC" H 3600 5200 140 0000 C CNB "Caption"
+F 4 "0VDC" H 3600 5275 140 0000 C CNB "Caption"
+F 5 "0VDC" H 3600 5075 140 0000 C CNB "Caption2"
 	24   4450 5575
 	1    0    0    -1
@@
 F 2 "" H 4450 1825 140 0001 C CNN
 F 3 "" H 4450 1825 140 0001 C CNN
-F 4 "+3A" H 3700 1475 140 0000 C CNB "Caption"
+F 4 "+3A" H 3700 1550 140 0000 C CNB "Caption"
+F 5 "+3A" H 3700 1350 140 0000 C CNB "Caption2"
 	47   4450 1650
 	1    0    0    -1
@@
 F 2 "" H 4450 4550 140 0001 C CNN
 F 3 "" H 4450 4550 140 0001 C CNN
-F 4 "+3A" H 3725 4175 140 0000 C CNB "Caption"
+F 4 "+3A" H 3700 4275 140 0000 C CNB "Caption"
+F 5 "+3A" H 3700 4075 140 0000 C CNB "Caption2"
 	48   4450 4375
 	1    0    0    -1
@@
 F 3 "" H 4450 3425 140 0001 C CNN
 F 4 "0VDC" H 3825 3250 140 0001 C CNB "Caption"
+F 5 "0VDC" H 4450 3250 50  0001 C CNN "Caption2"
 	71   4450 3250
 	1    0    0    -1
@@
 F 3 "" H 4450 6150 140 0001 C CNN
 F 4 "0VDC" H 3800 5975 140 0001 C CNB "Caption"
+F 5 "0VDC" H 4450 5975 50  0001 C CNN "Caption2"
 	72   4450 5975
 	1    0    0    -1
@@
 F 3 "" H 4450 2225 140 0001 C CNN
 F 4 "+3A" H 3850 2050 140 0001 C CNB "Caption"
+F 5 "+3A" H 4450 2050 140 0001 C CNB "Caption2"
 	95   4450 2050
 	1    0    0    -1
@@
 F 3 "" H 4450 4950 140 0001 C CNN
 F 4 "+3A" H 3875 4775 140 0001 C CNB "Caption"
+F 5 "+3A" H 4450 4775 50  0001 C CNN "Caption2"
 	96   4450 4775
 	1    0    0    -1
@@
 F 3 "" H 4450 3825 140 0001 C CNN
 F 4 "0VDC" H 3825 3650 140 0001 C CNB "Caption"
+F 5 "0VDC" H 4450 3650 50  0001 C CNN "Caption2"
 	119  4450 3650
 	1    0    0    -1
@@
 F 3 "" H 4450 6550 140 0001 C CNN
 F 4 "0VDC" H 3800 6400 140 0001 C CNB "Caption"
+F 5 "0VDC" H 4450 6375 50  0001 C CNN "Caption2"
 	120  4450 6375
 	1    0    0    -1
