File: Schematics/1006549r/module.sch (KiCad schematic (older format))
At the start: 34 parts, among them J1 ConnectorGeneric, U401 D3NOR-+3VDC-0VDC-nd1021041-_B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, U402 D3NOR-+3VDC-0VDC-nd1021041-A_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, U403 D3NOR-NC-0VDC-expander-nd1021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, U404 D3NOR-+3VDC-0VDC-nd1021041-AB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, U405 D3NOR-+3VDC-0VDC-nd1021041-_B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, U406 D3NOR-+3VDC-0VDC-nd1021041-_B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, U407 D3NOR-+3VDC-0VDC-nd1021041-AB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, U408 D3NOR-+3VDC-0VDC-nd1021041-AB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, U409 D3NOR-+3VDC-0VDC-nd1021041-AB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, U410 D3NOR-+3VDC-0VDC-nd1021041-AB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, U411 D3NOR-+3VDC-0VDC-nd1021041-CB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, U412 D3NOR-+3VDC-0VDC-nd1021041-AB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, U413 D3NOR-+3VDC-0VDC-nd1021041-CB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, U414 D3NOR-+3VDC-0VDC-nd1021041-AB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, U415 D3NOR-+3VDC-0VDC-nd1021041-AB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, U416 D3NOR-NC-0VDC-expander-nd1021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, U417 D3NOR-+3VDC-0VDC-nd1021041-A_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, U418 D3NOR-+3VDC-0VDC-nd1021041-A_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, U419 D3NOR-+3VDC-0VDC-nd1021041-A_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, U420 D3NOR-+3VDC-0VDC-nd1021041-A_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, U421 D3NOR-+3VDC-0VDC-nd1021041-_B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, U422 D3NOR-+3VDC-0VDC-nd1021041-_B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, U423 D3NOR-+3VDC-0VDC-nd1021041-_B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, U424 D3NOR-+3VDC-0VDC-nd1021041-_B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, U425 D3NOR-+3VDC-0VDC-nd1021041-_B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, U426 D3NOR-+3VDC-0VDC-nd1021041-_B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, U427 D3NOR-+3VDC-0VDC-nd1021041-_B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, U428 D3NOR-+3VDC-0VDC-nd1021041-_B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, U429 D3NOR-+3VDC-0VDC-nd1021041-_B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, U430 D3NOR-+3VDC-0VDC-nd1021041-_B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, U431 D3NOR-+3VDC-0VDC-nd1021041-_B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, U432 D3NOR-NC-0VDC-expander-nd1021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, U433 D3NOR-+3VDC-0VDC-nd1021041-_B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

Commit message: Added CAD transcription for drawing 1006549, Block I module A26, "logic flow J".  Updated the Block I pin DB to add this module to it.
Parts:
- removed J1: ConnectorGeneric, symbol AGC_DSKY:ConnectorGeneric
- removed U401, U405, U406, U421, U422, U423, U424, U425, U426, U427, U428, U429, U430, U431, U433: D3NOR-+3VDC-0VDC-nd1021041-_B_-___, symbol D3NOR-+3VDC-0VDC-nd1021041:D3NOR-+3VDC-0VDC-nd1021041-_B_-___
- removed U402, U417, U418, U419, U420: D3NOR-+3VDC-0VDC-nd1021041-A_C-___, symbol D3NOR-+3VDC-0VDC-nd1021041:D3NOR-+3VDC-0VDC-nd1021041-A_C-___
- removed U403: D3NOR-NC-0VDC-expander-nd1021041-ABC-___, symbol D3NOR-NC-0VDC-expander-nd1021041:D3NOR-NC-0VDC-expander-nd1021041-ABC-___
- removed U404, U412, U414, U415: D3NOR-+3VDC-0VDC-nd1021041-AB_-___, symbol D3NOR-+3VDC-0VDC-nd1021041:D3NOR-+3VDC-0VDC-nd1021041-AB_-___
- removed U407, U408, U409, U410: D3NOR-+3VDC-0VDC-nd1021041-ABC-___, symbol D3NOR-+3VDC-0VDC-nd1021041:D3NOR-+3VDC-0VDC-nd1021041-ABC-___
- removed U411, U413: D3NOR-+3VDC-0VDC-nd1021041-CB_-___, symbol D3NOR-+3VDC-0VDC-nd1021041:D3NOR-+3VDC-0VDC-nd1021041-CB_-___
- removed U416: D3NOR-NC-0VDC-expander-nd1021041-A_C-___, symbol D3NOR-NC-0VDC-expander-nd1021041:D3NOR-NC-0VDC-expander-nd1021041-A_C-___
- removed U432: D3NOR-NC-0VDC-expander-nd1021041-_B_-___, symbol D3NOR-NC-0VDC-expander-nd1021041:D3NOR-NC-0VDC-expander-nd1021041-_B_-___
Connections:
- net labels removed: +3VDC, 0VDC, GNHNC, STPB, T11
- wire segments 167 -> 4
Other:
- note added: "Notes from the Virtual AGC Project:\n1. None of the official Block I AGC electrical-schematic drawings were available at\n the time this CAD drawing was made. Rather, it is a transcription of the schematic\n drawings in the figures of AC Electronics document ND-1021041, which are also\n believed to comprise a complete but unofficial set of schematics. — RSB 2018\n2. The figures in ND-1021041 do n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"
- note removed: "(TO PRIORITY CONTROL)"
- note removed: "Notes from the Virtual AGC Project:\n4. In ND-1021041, gate 51320 is drawn with an inverting circle on the output,\n similar to how expander Block II expander gates are represented. All expander\n gates, whether or not depicted with the inverting circle, are NOR gates. Since all\n other expander NOR gates in the ND-1021041 Figures associated with this drawing\n are depicted without the circles, 5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"
