File: Schematics/1006541B/module.sch (KiCad schematic (older format))
At the start: 0 parts

Commit message: Proofed/corrected CAD for drawing 1006541B (Block I AGC module A35 electrical schematic).
Other:
- note added: "//"
- note added: "1006541"
- note added: "A REVISED PER TDRR 04150"
- note added: "B REVISED PER TDRR 04503"
- note added: "LOGIC FLOW "A""
- note added: "LOGIC MODULE NO. A35"
- note added: "NONE"
- note added: "____"
- note added: "________"
- note added: "____________"
Changed lines of the file:
@@
 F1 "1006541B.sch" 140
 $EndSheet
+Wire Notes Line style solid
+	37965 1170 43500 1170
+Text Notes 38125 1150 0    140  ~ 28
+A   REVISED PER TDRR 04150
+Wire Notes Line style solid
+	37965 1445 43500 1445
+Text Notes 38105 1420 0    140  ~ 28
+B   REVISED PER TDRR 04503
+Wire Notes Line style solid
+	37965 910  37965 1445
+Wire Notes Line style solid
+	38465 910  38465 1445
+Wire Notes Line style solid
+	41795 910  41795 1445
+Wire Notes Line style solid
+	42465 910  42465 1445
+Text Notes 39300 31850 0    275  ~ 55
+LOGIC FLOW "A"
+Text Notes 40780 33105 0    250  ~ 50
+1006541
+Text Notes 39375 32325 0    200  ~ 40
+LOGIC MODULE NO. A35
+Text Notes 33125 31755 0    140  ~ 28
+____
+Text Notes 33210 31820 0    140  ~ 28
+//
+Text Notes 39300 33025 2    140  ~ 28
+________
+Text Notes 39375 33475 2    140  ~ 28
+NONE
+Text Notes 34125 31755 0    140  ~ 28
+____
+Text Notes 34210 31820 0    140  ~ 28
+//
+Text Notes 35050 31755 0    140  ~ 28
+____
+Text Notes 35135 31820 0    140  ~ 28
+//
+Text Notes 34725 32350 2    140  ~ 28
+____________
+Text Notes 34225 32425 2    140  ~ 28
+//
+Text Notes 34725 32850 2    140  ~ 28
+____________
+Text Notes 34225 32925 2    140  ~ 28
+//
+Text Notes 34675 33325 2    140  ~ 28
+____________
+Text Notes 34175 33400 2    140  ~ 28
+//
 $EndSCHEMATC
