File: Schematics/1006199-/BOM.sch (KiCad schematic (older format))
At the start: 0 parts

Commit message: Finished transcription of drawing 1006199-.  In the process, found and fixed a reference designator in drawing 1006148E and a signal name in drawing 1006099A.
Other:
- note added: "-117"
- note added: "-118"
- note added: "-119"
- note added: "-33"
- note added: "-34"
- note added: "-36"
- note added: "0.1 UF"
- note added: "1006199"
- note added: "1006750-116"
- note added: "1006750-37"
- note added: "1050"
- note added: "1100"
- note added: "1150"
- note added: "1200"
- note added: "1250"
- note added: "1400"
- note added: "1500"
- note added: "1600"
- note added: "470 UUF"
- note added: "6.8 UF"
- note added: "8.2 UH"
- note added: "DASH NO."
- note added: "NOMINAL"
- note added: "OHMS±2%"
- note added: "REPLACES 1006189 WITH CHANGES"
- note added: "SEE CHART"
- note added: "_"
- note added: "◯"
- note removed: ".001UF"
- note removed: "0.1UF"
- note removed: "1006148"
- note removed: "1006777-24"
- note removed: "470UUF"
- note removed: "5.1K"
- note removed: "8.2UH"
- note removed: "A REVISED PER TDRR 04478"
- note removed: "B REVISED PER TDRR 06046"
- note removed: "C REVISED PER TDRR 06232"
- note removed: "C20"
- note removed: "D"
- note removed: "DR CHK"
- note removed: "E"
- note removed: "R34"
- note removed: "R35"
- note removed: "REVISED PER TDRR 07269"
- note removed: "REVISED PER TDRR 07670"
