File: Schematics/1006098H/module.sch (KiCad schematic (older format))
At the start: 0 parts

Commit message: Did some more transcribing on CAD for drawing 1006098H.
Other:
- note added: "*"
- note added: "1/2W"
- note added: "1/4W"
- note added: "1006750-"
- note added: "1006751"
- note added: "1006752"
- note added: "1006760-28"
- note added: "1006760-32"
- note added: "1006760-56"
- note added: "1006815-2"
- note added: "1006829"
- note added: "1006838"
- note added: "1010376-1"
- note added: "10K"
- note added: "18K"
- note added: "2%"
- note added: "25"
- note added: "32"
- note added: "39"
- note added: "42"
- note added: "43"
- note added: "510"
- note added: "56"
- note added: "6.2K"
- note added: "62"
- note added: "62K"
- note added: "75"
- note added: "CR10"
- note added: "CR11"
- note added: "CR12"
- note added: "CR13"
- note added: "CR14"
- note added: "CR15"
- note added: "DIODE"
- note added: "K1"
- note added: "NE"
- note added: "Q10"
- note added: "Q11"
- note added: "Q12"
- note added: "Q5"
- note added: "Q6"
- note added: "Q7"
- note added: "Q8"
- note added: "Q9"
- note added: "R19"
- note added: "R20"
- note added: "R21"
- note added: "R22"
- note added: "R23"
- note added: "R24"
- note added: "R25"
- note added: "R26"
- note added: "R27"
- note added: "R28"
- note added: "R29"
- note added: "R30"
- note added: "R31"
- note added: "R32"
- note added: "R33"
- note added: "R34"
- note added: "R35"
- note added: "R36"
- note added: "R37"
- note added: "R38"
- note added: "R39"
- note added: "R40"
- note added: "R41"
- note added: "R42"
- note added: "R43"
- note added: "RELAY"
- note added: "RES"
- note added: "TSTR"
- note added: "Ω"

Commit message: Completed/proofed CAD transcription of drawing 1006098H.
Parts:
- added CR10, CR11, CR12: Diode, symbol AGC_DSKY:Diode
- added CR13, CR14, CR15: Diode-Zener2, symbol AGC_DSKY:Diode-Zener2
- added J1: ConnectorGeneric, symbol AGC_DSKY:ConnectorGeneric
- added K1: Relay-1006815-2, symbol AGC_DSKY:Relay-1006815-2
- added Q10, Q9: Transistor-PNP, symbol AGC_DSKY:Transistor-PNP
- added Q11, Q12: Transistor-NPN, symbol AGC_DSKY:Transistor-NPN
- added Q5, Q6, Q7, Q8: Transistor-NPN-dual6, symbol AGC_DSKY:Transistor-NPN-dual6
- added R19, R20, R21, R22, R23, R24, R25, R26, R27, R28, R29, R30, R31, R32, R33, R34, R35, R36, R37, R38, R39, R40, R41, R42, R43: Resistor, symbol AGC_DSKY:Resistor
Connections:
- net 1/+28: now also J1.34
- net 1/CNTRL: now also J1.26
- net 1/GND: now also J1.35
- net 1/R: now also J1.27
- net 1/REF1: now also J1.29
- net 1/REF2: now also J1.30
- net 1/S: now also J1.28
- net 1/SHNT1: now also J1.33
- net 1/SHNT2: now also J1.32
- net 1/VPLS: now also J1.31
- net 2/+28: now also J1.2
- net 2/CNTRL: now also J1.10
- net 2/GND: now also J1.1
- net 2/R: now also J1.9
- net 2/REF1: now also J1.7
- net 2/REF2: now also J1.6
- net 2/S: now also J1.8
- net 2/SHNT1: now also J1.3
- net 2/SHNT2: now also J1.4
- net 2/VPLS: now also J1.5
- new net: CR12.1 (K), CR15.2 (A), J1.16, Q11.3 (E), R23.1, R28.1, R33.1, R36.2, R38.1, R41.2
- new net: J1.17, Q10.3 (C), R40.2
- new net: J1.14, R30.2, R37.2
- new net: J1.15, Q9.3 (C), R25.1
- new net: J1.11, R20.2, R29.2
- new net: J1.18, K1.7
- new net: J1.19, K1.6
- new net: J1.25, K1.3
- new net: CR10.1 (K), J1.24, R19.1, R42.1, R43.1
- new net: J1.23, K1.4
- new net: CR11.2 (A), J1.22, K1.5, Q12.1 (C)
- new net: J1.21, K1.2
- new net: J1.20, K1.8
- new net: Q5.1 (C1), Q5.4 (C2), R23.2
- new net: Q5.2 (B1), R20.1
- new net: Q5.3 (E1), Q6.3 (E1), Q9.2 (B), R24.1
- new net: Q5.5 (B2), R22.1
- new net: Q6.1 (C1), Q6.4 (C2), R28.2
- new net: Q6.2 (B1), R27.1
- new net: Q6.5 (B2), R29.1
- new net: Q7.1 (C1), Q7.4 (C2), R33.2
- new net: Q7.2 (B1), R30.1
- new net: Q10.2 (B), Q7.3 (E1), Q8.3 (E1), R39.1
- new net: Q7.5 (B2), R32.1
- new net: Q8.1 (C1), Q8.4 (C2), R38.2
- new net: Q8.2 (B1), R35.1
- new net: Q8.5 (B2), R37.1
- new net: CR13.2 (A), CR14.1 (K)
- new net: CR14.2 (A), CR15.1 (K)
- new net: R21.2, R22.2, R26.1
- new net: R26.2, R27.2, R31.1
- new net: R31.2, R32.2, R34.1
- new net: R34.2, R35.2, R36.1
- new net: Q11.1 (C), Q12.2 (B), R42.2
- new net: Q11.2 (B), R25.2, R40.1, R41.1
- new net: K1.1, R43.2
- new net: CR12.2 (A), Q12.3 (E)
- new net: CR10.2 (A), CR11.1 (K)
- new net 18.6V: CR13.1 (K), Q10.1 (E), Q5.6 (E2), Q6.6 (E2), Q7.6 (E2), Q8.6 (E2), Q9.1 (E), R19.2, R21.1, R24.2, R39.2
Other:
- note added: "1. NOMINAL VALUE, TO BE DETERMINED AT TEST,\n AS SELECTED FROM TABLE 1\n2. N.C. INDICATES NO CONNECTION\n3. PREFIX 1 ON SYMBOL NUMBERS REFERS TO CONTROL CIRCUIT A1.\n PREFIX 2 ON SYMBOL NUMBERS REFERS TO CONTROL CIRCUIT A2.\n WHERE NO PREFIX IS SHOWN THE VALUE APPLIES TO BOTH CIRCUITS."
- note added: "680"
- note added: "NOTES:"
- note added: "Notes from the Virtual AGC Project:\na) This CAD drawing was transcribed from the original Project Apollo drawing \n 1006098H. — RSB 2019\nb) Because the original design used identical circuitry for control blocks A1 and A2,\n in order to faithfully preserve the electrical properties of the circuit within the \n CAD context, this transcription differs visually somewhat from the original \n drawin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"
- note added: "POWER SUPPLY FAILURE\n DETECTION CIRCUIT"
