File: Schematics/1005730B/module.sch (KiCad schematic (older format))
At the start: 0 parts

Commit message: Completed/proofed CAD transcription for drawing 1005730B (Block I DSKY G&N failure-detection module electrical schematics).
Other:
- note added: "1005730"
- note added: "A"
- note added: "B"
- note added: "G&N FAILURE DETECT"
- note added: "REVISED PER TDRR 20410"
- note added: "REVISED PER TDRR 21345"
- note added: "SCHEMATIC,"
- note added: "___"
- note added: "________"
- note added: "____________"
- note added: "________________"
Changed lines of the file:
@@
 F1 "1005730B.sch" 140
 $EndSheet
+Wire Notes Line style solid
+	36480 905  36480 1750
+Wire Notes Line style solid
+	36480 1750 43500 1750
+Wire Notes Line style solid
+	36480 1365 43500 1365
+Wire Notes Line style solid
+	36870 905  36870 1750
+Wire Notes Line style solid
+	37365 905  37365 1750
+Wire Notes Line style solid
+	40830 905  40830 1750
+Wire Notes Line style solid
+	41345 905  41345 1750
+Wire Notes Line style solid
+	41835 905  41835 1750
+Wire Notes Line style solid
+	42460 905  42460 1750
+Text Notes 36600 1250 0    140  ~ 28
+A
+Text Notes 36600 1665 0    140  ~ 28
+B
+Text Notes 37450 1250 0    140  ~ 28
+REVISED PER TDRR 20410
+Text Notes 37460 1660 0    140  ~ 28
+REVISED PER TDRR 21345
+Text Notes 39750 31875 0    250  ~ 50
+SCHEMATIC,
+Text Notes 40650 33125 0    250  ~ 50
+1005730
+Text Notes 39000 32350 0    200  ~ 40
+G&N FAILURE DETECT
+Text Notes 33275 32850 0    140  ~ 28
+____________
+Text Notes 35075 31750 0    140  ~ 28
+___
+Text Notes 34175 31750 0    140  ~ 28
+___
+Text Notes 33200 31750 0    140  ~ 28
+___
+Text Notes 38850 33375 0    140  ~ 28
+___
+Text Notes 38400 32950 0    140  ~ 28
+________
+Text Notes 39800 33350 0    140  ~ 28
+________________
 $EndSCHEMATC
