File: Schematics/1006162B/CDE.sch (KiCad schematic (older format))
At the start: 8 parts

Commit message: Finished CAD transcription of drawing 1006162B.  Had to tweak my hierarchical-block annotator a little bit because it turns out that when KiCad annotates, it doesn't mark blocks that appear only once the same what that it marks blocks that appear more than once.
Parts:
- gave numbers to parts that had none: 8
Other:
- note added: "90012 - 90023 & 90612 - 90623"
- note added: "Notes from the Virtual AGC Project:\ne) This CAD sheet was transcribed from the original Project Apollo drawing\n 1006162B, but with elements not specifically related to circuit blocks\n 90012-90023 and 90612-90623 discarded. — RSB 2019\n"
- note removed: "90012 - 90023 & 90612 - 91623"
