File: Schematics/2005060D/2005060D-p3of3.sch (KiCad schematic (older format))
At the start: 63 parts, among them J3 ConnectorA1-300, J4 ConnectorA1-400, U301 D3NOR-+4SW-0VDC-A_B-EDF, U302 D3NOR-+4SW-0VDC-AC_-EF_, U303 D3NOR-+4SW-0VDC-ACB-FD_, U304 D3NOR-+4SW-0VDC-AC_-E_F, U305 D3NOR-NC-0VDC-expander-B_C-ED_, U306 D3NOR-+4SW-0VDC-ABC-FD_, U307 D3NOR-+4SW-0VDC-AC_-E_F, U308 D3NOR-+4SW-0VDC-ACB-FD_, U309 D3NOR-+4SW-0VDC-AC_-E_F, U310 D3NOR-+4SW-0VDC-ABC-FD_, U311 D3NOR-NC-0VDC-expander-ABC-DEF, U312 D3NOR-+4SW-0VDC-AC_-E_F, U313 D3NOR-+4SW-0VDC-ABC-FD_, U314 D3NOR-+4SW-0VDC-ABC-D_E, U315 D3NOR-+4SW-0VDC-BC_-D_E, U316 D3NOR-+4SW-0VDC-ABC-FD_, U317 D3NOR-+4SW-0VDC-AC_-EF_, U318 D3NOR-+4SW-0VDC-ACB-FD_, U319 D3NOR-+4SW-0VDC-AC_-EF_, U320 D3NOR-+4SW-0VDC-ABC-FD_, U321 D3NOR-+4SW-0VDC-AC_-EF_, U322 D3NOR-+4SW-0VDC-ABC-FD_, U323 D3NOR-+4SW-0VDC-AC_-EF_, U324 D3NOR-+4SW-0VDC-ACB-FD_, U325 D3NOR-+4SW-0VDC-BC_-EF_, U326 D3NOR-+4SW-0VDC-ABC-FD_, U327 D3NOR-+4SW-0VDC-AC_-D_E, U328 D3NOR-+4SW-0VDC-ACB-_F_, U329 D3NOR-+4SW-0VDC-ABC-_F_, U330 D3NOR-+4SW-0VDC-ABC-_D_, U401 D3NOR-+4SW2-0VDC2-_A_-_F_, U402 D3NOR-+4SW2-0VDC2-_A_-_F_, U403 D3NOR-NC-0VDC2-expander-AB_-D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, U404 D3NOR-+4SW2-0VDC2-_C_-_F_, U405 D3NOR-+4SW2-0VDC2-_C_-_D_, U406 D3NOR-+4SW2-0VDC2-_C_-_E_, U407 D3NOR-+4SW2-0VDC2-_C_-_E_, U408 D3NOR-NC-0VDC2-expander-AB_-D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, U409 D3NOR-+4SW2-0VDC2-_C_-_E_, U410 D3NOR-+4SW2-0VDC2-_C_-_E_, U411 D3NOR-+4SW2-0VDC2-_C_-_E_, U412 D3NOR-+4SW2-0VDC2-_C_-_E_, U413 D3NOR-NC-0VDC2-expander-BC_-D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, U414 D3NOR-+4SW2-0VDC2-_C_-_E_, U415 D3NOR-+4SW2-0VDC2-_C_-_E_, U416 D3NOR-+4SW2-0VDC2-_C_-_E_, U417 D3NOR-+4SW2-0VDC2-_C_-_E_, U418 D3NOR-+4SW2-0VDC2-_C_-_E_, U419 D3NOR-NC-0VDC2-expander-BC_-F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, U420 D3NOR-+4SW2-0VDC2-_C_-_E_, U421 D3NOR-+4SW2-0VDC2-_C_-_F_, U422 D3NOR-+4SW2-0VDC2-_C_-_E_, U423 D3NOR-NC-0VDC2-expander-BC_-E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, U424 D3NOR-+4SW2-0VDC2-_C_-_E_, U425 D3NOR-+4SW2-0VDC2-_B_-D_F, U426 D3NOR-+4SW2-0VDC2-_B_-_F_, U427 D3NOR-NC-0VDC2-expander-AB_-D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, U428 D3NOR-+4SW2-0VDC2-_A_-_F_, U429 D3NOR-+4SW2-0VDC2-A_B-_D_, U430 D3NOR-+4SW2-0VDC2-A_B-_D_

Commit message: Some cosmetic cleanups to AGC schematics.
Changed lines of the file:
@@
 EESchema Schematic File Version 4
 LIBS:module-cache
-EELAYER 26 0
+EELAYER 28 0
 EELAYER END
 $Descr E 44000 34000
@@
 	1    0    0    -1
 $EndComp
-Text GLabel 17300 3675 2    140  Input ~ 28
+Text GLabel 17300 3675 2    140  Output ~ 28
 B2
-Text GLabel 17275 5650 2    140  Input ~ 28
+Text GLabel 17275 5650 2    140  Output ~ 28
 B1
 $Comp
@@
 	1    0    0    -1
 $EndComp
-Text GLabel 7050 8800 0    140  Input ~ 28
+Text GLabel 7450 8975 2    140  Output ~ 28
 B19
 $Comp
@@
 	1    0    0    -1
 $EndComp
-Text GLabel 13125 8825 0    140  Input ~ 28
+Text GLabel 13575 9000 2    140  Output ~ 28
 B18
-Text GLabel 18725 8825 0    140  Input ~ 28
+Text GLabel 19075 8975 2    140  Output ~ 28
 B16
-Text GLabel 24525 8825 0    140  Input ~ 28
+Text GLabel 25000 8950 2    140  Output ~ 28
 B14
 $Comp
@@
 	1    0    0    -1
 $EndComp
-Text GLabel 30550 8800 0    140  Input ~ 28
+Text GLabel 31000 9000 2    140  Output ~ 28
 B13
-Text GLabel 38300 9100 2    140  Input ~ 28
+Text GLabel 38300 9100 2    140  Output ~ 28
 B11
 $Comp
@@
 	1    0    0    -1
 $EndComp
-Text GLabel 7750 18450 0    140  Input ~ 28
+Text GLabel 8200 18450 2    140  Output ~ 28
 B9
-Text GLabel 7125 22450 0    140  Output ~ 28
+Text GLabel 7125 22450 0    140  Input ~ 28
 B16
-Text GLabel 1325 22650 0    140  Output ~ 28
+Text GLabel 1325 22650 0    140  Input ~ 28
 B18
 $Comp
@@
 	-1   0    0    1
 $EndComp
-Text GLabel 7075 27625 0    140  Output ~ 28
+Text GLabel 7075 27625 0    140  Input ~ 28
 B7
-Text GLabel 1350 28450 0    140  Output ~ 28
+Text GLabel 1350 28450 0    140  Input ~ 28
 B8
 Text Notes 6625 27450 0    140  ~ 28
@@
 	-1   0    0    1
 $EndComp
-Text GLabel 15125 32275 0    140  Output ~ 28
+Text GLabel 15125 32275 0    140  Input ~ 28
 B3
 Text Notes 14675 32100 0    140  ~ 28
@@
 	-1   0    0    1
 $EndComp
-Text GLabel 13125 27625 0    140  Output ~ 28
+Text GLabel 13125 27625 0    140  Input ~ 28
 B5
-Text GLabel 12825 23650 0    140  Output ~ 28
+Text GLabel 12825 23650 0    140  Input ~ 28
 B14
-Text GLabel 13500 18450 0    140  Input ~ 28
+Text GLabel 13950 18450 2    140  Output ~ 28
 B8
 $Comp
@@
 	-1   0    0    1
 $EndComp
-Text GLabel 25100 18375 0    140  Input ~ 28
+Text GLabel 25500 18375 2    140  Output ~ 28
 B5
-Text GLabel 19325 18425 0    140  Input ~ 28
+Text GLabel 19650 18425 2    140  Output ~ 28
 B7
-Text GLabel 31375 19525 0    140  Input ~ 28
+Text GLabel 31825 19525 2    140  Output ~ 28
 B4
-Text GLabel 19025 23625 0    140  Output ~ 28
+Text GLabel 19025 23625 0    140  Input ~ 28
 B13
-Text GLabel 31975 24625 0    140  Output ~ 28
+Text GLabel 31975 24625 0    140  Input ~ 28
 B9
 Text Notes 31550 24450 0    140  ~ 28
@@
 Text Notes 20750 29875 0    140  ~ 28
 T12
-Text GLabel 19000 27625 0    140  Output ~ 28
+Text GLabel 19000 27625 0    140  Input ~ 28
 B4
-Text GLabel 25975 27625 0    140  Output ~ 28
+Text GLabel 25975 27625 0    140  Input ~ 28
 B11
-Text GLabel 21275 30075 0    140  Output ~ 28
+Text GLabel 21275 30075 0    140  Input ~ 28
 B19
-Text GLabel 39500 23000 0    140  Output ~ 28
+Text GLabel 39500 23000 0    140  Input ~ 28
 B1
-Text GLabel 39500 22000 0    140  Output ~ 28
+Text GLabel 39500 22000 0    140  Input ~ 28
 B2
-Text GLabel 37525 19550 0    140  Output ~ 28
+Text GLabel 38125 19225 2    140  Output ~ 28
 B3
 $Comp
@@
 Text Notes 41125 28925 0    140  ~ 28
 TO PIN 10 OF\n37400 SERIES \nGATES EXCEPT \nFAN-INS. SEE\nNOTE 3
-Text Label 36625 27350 0    140  ~ 28
-0VDC
 Text Label 36350 28175 0    140  ~ 28
 +4SW
@@
 	41625 23000 42325 23000
 Wire Wire Line
-	37525 19550 37825 19550
+	38125 19225 37825 19225
 Wire Wire Line
-	37825 19550 37825 18975
+	37825 19225 37825 18975
 Wire Wire Line
 	37825 18250 37725 18250
@@
 	13600 17100 13800 17100
 Wire Wire Line
-	13800 18450 13500 18450
-Wire Wire Line
 	13500 17875 13800 17875
 Wire Wire Line
@@
 	7975 17100 7975 17900
 Wire Wire Line
-	7975 18450 7750 18450
+	7975 18450 8200 18450
 Wire Wire Line
 	7725 17900 7975 17900
@@
 	17475 19075 17625 19075
 Wire Wire Line
-	19325 18425 19500 18425
-Wire Wire Line
 	19500 17075 19400 17075
 Wire Wire Line
@@
 	23225 19075 23425 19075
 Wire Wire Line
-	25100 18375 25300 18375
+	25500 18375 25300 18375
 Wire Wire Line
 	25300 18375 25300 17775
@@
 	31600 20475 31600 20100
 Wire Wire Line
-	31600 19525 31375 19525
+	31600 19525 31825 19525
 Wire Wire Line
 	31375 20100 31600 20100
@@
 	7250 10125 7250 9375
 Wire Wire Line
-	7250 8800 7050 8800
+	7250 8975 7450 8975
 Wire Wire Line
 	7000 9375 7250 9375
 Connection ~ 7250 9375
 Wire Wire Line
-	7250 9375 7250 8800
+	7250 9375 7250 8975
 Wire Wire Line
 	7825 11900 8400 11900
@@
 	14000 8400 14225 8400
 Wire Wire Line
-	13125 8825 13400 8825
+	13575 9000 13400 9000
 Wire Wire Line
-	13400 8825 13400 9400
+	13400 9000 13400 9400
 Wire Wire Line
 	13400 10125 13125 10125
@@
 	30825 10100 30825 9350
 Wire Wire Line
-	30825 8800 30550 8800
+	30825 9000 31000 9000
 Wire Wire Line
 	30550 9350 30825 9350
 Connection ~ 30825 9350
 Wire Wire Line
-	30825 9350 30825 8800
+	30825 9350 30825 9000
 Wire Wire Line
 	24625 10100 24825 10100
@@
 	24825 10100 24825 9375
 Wire Wire Line
-	24825 8825 24525 8825
+	24825 8950 25000 8950
 Wire Wire Line
 	24525 9375 24825 9375
 Connection ~ 24825 9375
 Wire Wire Line
-	24825 9375 24825 8825
+	24825 9375 24825 8950
 Wire Wire Line
 	31700 9500 31700 9825
@@
 	18950 10125 18950 9400
 Wire Wire Line
-	18950 8825 18725 8825
+	18950 8975 19075 8975
 Wire Wire Line
 	18725 9400 18950 9400
 Connection ~ 18950 9400
 Wire Wire Line
-	18950 9400 18950 8825
+	18950 9400 18950 8975
 Connection ~ 28200 8125
 Wire Wire Line
@@
 	36625 25900 36625 26350
 Connection ~ 36625 26350
+Wire Wire Line
+	19500 18425 19650 18425
+Wire Wire Line
+	13800 18450 13950 18450
 $EndSCHEMATC
