File: Schematics/1005780-/1005780-.sch (KiCad schematic (older format))
At the start: 130 parts, among them J1 ConnectorGeneric, K1 RELAY-1006772-1, K10 RELAY-1006772-1, K11 RELAY-1006772-1, K12 RELAY-1006815-2C, K13 RELAY-1006772-1, K14 RELAY-1006772-1, K15 RELAY-1006772-1, K16 RELAY-1006772-1, K17 RELAY-1006772-1, K18 RELAY-1006815-2C, K19 RELAY-1006772-1, K2 RELAY-1006772-1, K20 RELAY-1006772-1, K21 RELAY-1006772-1, K22 RELAY-1006772-1, K23 RELAY-1006772-1, K24 RELAY-1006772-1, K25 RELAY-1006772-1, K26 RELAY-1006772-1, K27 RELAY-1006772-1, K28 RELAY-1006772-1, K29 RELAY-1006772-1, K3 RELAY-1006772-1, K30 RELAY-1006772-1, K31 RELAY-1006772-1, K32 RELAY-1006772-1, K33 RELAY-1006772-1, K34 RELAY-1006772-1, K35 RELAY-1006772-1, K36 RELAY-1006772-1, K37 RELAY-1006772-1, K38 RELAY-1006772-1, K39 RELAY-1006772-1, K4 RELAY-1006772-1, K40 RELAY-1006772-1, K41 RELAY-1006772-1, K42 RELAY-1006772-1, K5 RELAY-1006772-1, K6 RELAY-1006815-2C, K7 RELAY-1006772-1, K8 RELAY-1006772-1, K9 RELAY-1006772-1

Commit message: Finished/proofed CAD transcription of drawing 1005780-.  Fixed a couple of related textual errors I found in drawing 1006161C as a part of that process.
Parts:
- added unit 70 of J1
- added unit 52 of J1
- added unit 97 of J1
- added unit 101 of J1
- added unit 128 of J1
- added unit 41 of J1
Connections:
- net at K23.4: now also J1.31; no longer J1.52
- net at J1.119: now also K2.4; no longer K5.4
- net at J1.113, K1.3, K10.3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: now also K26.6
- net at J1.94, K13.3, K15.3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: now also K14.6; no longer K14.2, K20.2
- net at J1.36: now also K8.4; no longer K11.4
- net at J1.32, K21.8: now also K20.3
- net at K17.4: now also J1.98; no longer J1.97
- net at J1.80, K2.2, K26.2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: now also K14.2, K20.2; no longer K14.3, K14.6, K20.3, K26.6
- net at J1.73: now also K26.4; no longer K29.4
- net at J1.18: now also K8.8; no longer K8.4
- net at J1.15, K15.8: now also K14.3
- net at J1.79, K14.7, K17.8: no longer K16.6
- net at J1.55: now also K14.8; no longer K14.4
- net at J1.49: now also K32.8
- net at K32.4: now also J1.70
- net at K30.3: now also J1.130
- net at K30.7: now also K24.7
- net at K20.4: now also J1.52
- net at K9.4: now also K11.6
- net at K3.4: now also K5.6
- new net: J1.128, K29.4
- new net: J1.97, K14.4
- new net: J1.101, K11.4
- new net: J1.41, K5.4
- no-connect marks 48 -> 47
Other:
- note added: "(TO SWITCH FROM POSITION SHOWN"
- note added: "1005780"
- note added: "APPLY PLUS VOLTAGE ON PIN 1)"
- note added: "CKT FOR LATCHING RELAYS K1 THRU K5, K7 THRU K11,"
- note removed: "(TO SWITCH FROM POSITION SHOWN,"
- note removed: "1006161"
- note removed: "APPLY PLUS VOLTAGE ON PIN 1"
- note removed: "CKT FOR LATCHING RELAYS K1 THRU K5, K7 THRU K11"
- moved on the sheet: CR1, CR14, CR15, CR16, CR17, CR2, CR23, CR24, CR25, CR26, CR27, CR28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

Commit message: Made some visual but not electrical fixes using eelint.  It does not presently pass ERC (because of a new bug in KiCad), but a before vs after comparison of netlists shows that there are no electrical changes.
Changed lines of the file:
@@
-EESchema Schematic File Version 4
+EESchema Schematic File Version 5
 LIBS:module-cache
 EELAYER 29 0
@@
 	28325 22075 33375 22075
 Wire Wire Line
-	27475 23500 27500 23500
-Wire Wire Line
 	25225 22250 25225 24000
 Wire Wire Line
@@
 	21950 9525 22250 9525
 Wire Wire Line
-	32425 2475 32425 3825
+	32425 2475 32425 3800
 Wire Wire Line
-	32425 3825 30975 3825
+	32425 3800 30975 3800
 Wire Wire Line
-	30975 3825 30975 3850
-Connection ~ 32425 3825
+	30975 3800 30975 3850
+Connection ~ 32425 3800
 Wire Wire Line
-	32425 3825 32425 7025
+	32425 3800 32425 7025
 Wire Wire Line
 	28775 2450 28775 3800
@@
 	28775 3800 28775 7025
 Wire Wire Line
-	32625 2475 32625 3825
+	32625 2475 32625 3800
 Wire Wire Line
-	36275 2500 36275 3825
+	36275 2500 36275 3800
 Wire Wire Line
-	36275 3825 34825 3825
+	36275 3800 34825 3800
 Wire Wire Line
-	34825 3825 34825 3850
-Connection ~ 36275 3825
+	34825 3800 34825 3850
+Connection ~ 36275 3800
 Wire Wire Line
-	36275 3825 36275 7025
+	36275 3800 36275 7025
 Wire Wire Line
-	32625 3825 34075 3825
+	32625 3800 34075 3800
 Wire Wire Line
-	34075 3825 34075 3850
-Connection ~ 32625 3825
+	34075 3800 34075 3850
+Connection ~ 32625 3800
 Wire Wire Line
-	32625 3825 32625 7025
+	32625 3800 32625 7025
 Wire Wire Line
 	27550 15500 28375 15500
@@
 Wire Wire Line
 	21900 25550 22175 25550
-Connection ~ 27500 23500
 Wire Wire Line
 	27500 23500 28325 23500
