File: Schematics/1006556r/Fig-4-74.sch (KiCad schematic (older format))
At the start: 0 parts

Commit message: For module A31, transcribed through Fig 4-87, leaving just 88, 91, 93, 114, 141, and 147 to go, plus their integration into the top-level sheet (and resolution of remaining inconsistencies in ND-1021041).
Parts:
- added J1: ConnectorGeneric, symbol AGC_DSKY:ConnectorGeneric
- added U? (x5): D3NOR-+3VDC-0VDC-nd1021041-A_C-___, symbol D3NOR-+3VDC-0VDC-nd1021041:D3NOR-+3VDC-0VDC-nd1021041-A_C-___
- added U?: D3NOR-NC-0VDC-expander-nd1021041-_B_-___, symbol D3NOR-NC-0VDC-expander-nd1021041:D3NOR-NC-0VDC-expander-nd1021041-_B_-___
- added U? (x2): D3NOR-NC-0VDC-expander-nd1021041-A_C-___, symbol D3NOR-NC-0VDC-expander-nd1021041:D3NOR-NC-0VDC-expander-nd1021041-A_C-___
- added U?: D3NOR-+3VDC-0VDC-nd1021041-_B_-___, symbol D3NOR-+3VDC-0VDC-nd1021041:D3NOR-+3VDC-0VDC-nd1021041-_B_-___
- added U? (x2): D3NOR-+3VDC-0VDC-nd1021041-ABC-___, symbol D3NOR-+3VDC-0VDC-nd1021041:D3NOR-+3VDC-0VDC-nd1021041-ABC-___
Connections:
- net +3VDC: now also U?.6 (+3VDC), U?.6 (+3VDC), U?.6 (+3VDC), U?.6 (+3VDC), U?.6 (+3VDC), U?.6 (+3VDC), U?.6 (+3VDC), U?.6 (+3VDC)
- net 0VDC: now also U?.2 (0VDC), U?.2 (0VDC), U?.3 (0VDC), U?.3 (0VDC), U?.3 (0VDC), U?.3 (0VDC), U?.3 (0VDC), U?.3 (0VDC), U?.3 (0VDC), U?.4 (0VDC), U?.4 (0VDC), U?.5 (0VDC), U?.5 (0VDC), U?.5 (0VDC), U?.5 (0VDC), U?.5 (0VDC), U?.5 (0VDC), U?.5 (0VDC), U?.5 (0VDC), U?.5 (0VDC), U?.5 (0VDC), U?.5 (0VDC)
- new net: J1.82, U?.4 (A)
- new net: J1.41, U?.4 (A), U?.4 (A)
- new net: J1.64, U?.1 (J)
- new net: U?.1 (J), U?.4 (A) (x2)
- new net: U?.1 (J), U?.2 (C), U?.2 (C)
- new net: J1.33, U?.2 (C)
- new net: J1.50, U?.2 (C)
- new net: J1.31, U?.1 (J)
- new net: U?.1 (J), U?.3 (B) (x2)
- new net: U?.1 (J), U?.2 (C)
- new net: J1.13, U?.1 (J)
- new net: J1.109, U?.4 (A), U?.4 (A)
- new net: J1.17, U?.2 (C)
- new net: U?.1 (J), U?.1 (J), U?.3 (B)
- new net: J1.29, U?.2 (C), U?.2 (C)
- new net: J1.21, U?.4 (A), U?.4 (A)
- new net: J1.25, U?.2 (C)
- new net: J1.27, U?.3 (B)

Commit message: Finished up transcription of drawing 1006556 (Block I logic flow S, module A21).  But it may be a total mess, so user beware!
Parts:
- removed unit 82 of J1
- removed unit 41 of J1
- removed unit 50 of J1
- removed unit 33 of J1
- removed unit 109 of J1
- removed unit 27 of J1
- removed unit 21 of J1
- gave numbers to parts that had none: 11
Connections:
- net T03_B: now reaches U502.4 (A)
- net T02_: now reaches U503.4 (A), U506.4 (A)
- net g60036: now reaches U506.1 (J), U510.4 (A)
- net g60039: now reaches U503.1 (J), U509.4 (A)
- net DV1_: now reaches U503.2 (C)
- net DV1_B: now reaches U502.2 (C)
- net g60048: now reaches U502.1 (J), U508.3 (B)
- net g60045: now reaches U504.1 (J), U509.2 (C)
- net T03_: now reaches U504.4 (A), U507.4 (A)
- net MP0: now reaches U501.4 (A), U505.4 (A)
- net MP1: now reaches U507.3 (B)

Commit message: When I started recovering transcribed Block I schematics from document ND-1021041, there was no info available to me on the pinout of the NOR-gates they used, and it didn't occur to me that any might be forthcoming, so I chose a pinout arbitrarily.  It turns out that we now have the required info (SCD 1006771), and my arbitrary choices were wrong. I've therefore updated the NOR-library generator script, the relevant NOR libraries themselves, and all of the so-far-recovered Block I schematics using those gates.  It doesn't really matter in the cosmic sense, since the real Block I schematics have become available in the meantime, so that these recovered schematics are of less interest, but it will come in handy when I eventually want to do cross-checking.  I haven't checked these updated schematics in full detail, but I've spot-checked them, and run some ERCs and netlists, and it looks good to me.
Parts:
- U501, U502, U503, U504, U506: value D3NOR-+3VDC-0VDC-nd1021041-A_C-___ -> D3NOR-+3VDC-0VDC-nd1021041-1_5-___; symbol D3NOR-+3VDC-0VDC-nd1021041:D3NOR-+3VDC-0VDC-nd1021041-A_C-___ -> D3NOR-+3VDC-0VDC-nd1021041:D3NOR-+3VDC-0VDC-nd1021041-1_5-___
- U505, U509: value D3NOR-NC-0VDC-expander-nd1021041-A_C-___ -> D3NOR-NC-0VDC-expander-nd1021041-1_5-___; symbol D3NOR-NC-0VDC-expander-nd1021041:D3NOR-NC-0VDC-expander-nd1021041-A_C-___ -> D3NOR-NC-0VDC-expander-nd1021041:D3NOR-NC-0VDC-expander-nd1021041-1_5-___
- U507, U510: value D3NOR-+3VDC-0VDC-nd1021041-ABC-___ -> D3NOR-+3VDC-0VDC-nd1021041-135-___; symbol D3NOR-+3VDC-0VDC-nd1021041:D3NOR-+3VDC-0VDC-nd1021041-ABC-___ -> D3NOR-+3VDC-0VDC-nd1021041:D3NOR-+3VDC-0VDC-nd1021041-135-___
- U508: value D3NOR-NC-0VDC-expander-nd1021041-_B_-___ -> D3NOR-NC-0VDC-expander-nd1021041-_3_-___; symbol D3NOR-NC-0VDC-expander-nd1021041:D3NOR-NC-0VDC-expander-nd1021041-_B_-___ -> D3NOR-NC-0VDC-expander-nd1021041:D3NOR-NC-0VDC-expander-nd1021041-_3_-___
- U511: value D3NOR-+3VDC-0VDC-nd1021041-_B_-___ -> D3NOR-+3VDC-0VDC-nd1021041-_3_-___; symbol D3NOR-+3VDC-0VDC-nd1021041:D3NOR-+3VDC-0VDC-nd1021041-_B_-___ -> D3NOR-+3VDC-0VDC-nd1021041:D3NOR-+3VDC-0VDC-nd1021041-_3_-___
Connections:
- net +3VDC: now also U501.8 (+3VDC), U502.8 (+3VDC), U503.8 (+3VDC), U504.8 (+3VDC), U506.8 (+3VDC), U507.8 (+3VDC), U510.8 (+3VDC), U511.8 (+3VDC); no longer U501.6 (+3VDC), U502.6 (+3VDC), U503.6 (+3VDC), U504.6 (+3VDC), U506.6 (+3VDC), U507.6 (+3VDC), U510.6 (+3VDC), U511.6 (+3VDC)
- net 0VDC: now also U501.4 (0VDC), U502.4 (0VDC), U503.4 (0VDC), U504.4 (0VDC), U505.4 (0VDC), U506.4 (0VDC), U507.4 (0VDC), U508.1 (0VDC), U509.4 (0VDC), U510.4 (0VDC), U511.1 (0VDC); no longer U501.5 (0VDC), U502.5 (0VDC), U503.5 (0VDC), U504.5 (0VDC), U505.5 (0VDC), U506.5 (0VDC), U507.5 (0VDC), U508.2 (0VDC), U509.5 (0VDC), U510.5 (0VDC), U511.2 (0VDC)
- net DV1_: now also U503.5; no longer U503.2 (C)
- net DV1_B: now also U502.5; no longer U502.2 (C)
- net MP0: now also U501.1, U505.1; no longer U501.4 (A), U505.4 (A)
- net T02_: now also U503.1, U506.1; no longer U503.4 (A), U506.4 (A)
- net T03_: now also U504.1, U507.1; no longer U504.4 (A), U507.4 (A)
- net T03_B: now also U502.1; no longer U502.4 (A)
- net g60036: now also U506.7, U510.1; no longer U506.1 (J), U510.4 (A)
- net g60039: now also U503.7, U509.1; no longer U503.1 (J), U509.4 (A)
- net g60045: now also U504.7, U509.5; no longer U504.1 (J), U509.2 (C)
- net g60048: now also U502.7; no longer U502.1 (J)
- net at J1.64: now also U508.7; no longer U508.1 (J)
- net at J1.31: now also U509.7; no longer U509.1 (J)
- net at J1.13: now also U511.7; no longer U511.1 (J)
- net at U511.3: now also U510.7; no longer U510.1 (J)
- net at U510.2 (NC): no longer J1.17
- net at U507.2 (NC): no longer J1.25
- new net: U501.7, U504.5, U506.5
- new net: U505.7, U507.7, U510.3
- new net: J1.17, U510.5
- new net: J1.29, U501.5, U505.5
- new net: J1.25, U507.5
- now unconnected: U501.2 (C), U504.2 (C), U505.2 (C), U506.2 (C)
Changed lines of the file:
@@
 $EndComp
 $Comp
-L D3NOR-+3VDC-0VDC-nd1021041:D3NOR-+3VDC-0VDC-nd1021041-A_C-___ U506
+L D3NOR-+3VDC-0VDC-nd1021041:D3NOR-+3VDC-0VDC-nd1021041-1_5-___ U506
 U 1 1 5BFAAD8A
 P 7450 4350
 F 0 "U506" H 7450 4675 140 0001 C CNB
-F 1 "D3NOR-+3VDC-0VDC-nd1021041-A_C-___" H 7450 4775 140 0001 C CNN
+F 1 "D3NOR-+3VDC-0VDC-nd1021041-1_5-___" H 7450 4775 140 0001 C CNN
 F 2 "" H 7450 4825 140 0001 C CNN
 F 3 "" H 7450 4825 140 0001 C CNN
@@
 $EndComp
 $Comp
-L D3NOR-+3VDC-0VDC-nd1021041:D3NOR-+3VDC-0VDC-nd1021041-A_C-___ U503
+L D3NOR-+3VDC-0VDC-nd1021041:D3NOR-+3VDC-0VDC-nd1021041-1_5-___ U503
 U 1 1 5BFAAD8B
 P 7400 1475
 F 0 "U503" H 7400 1800 140 0001 C CNB
-F 1 "D3NOR-+3VDC-0VDC-nd1021041-A_C-___" H 7400 1900 140 0001 C CNN
+F 1 "D3NOR-+3VDC-0VDC-nd1021041-1_5-___" H 7400 1900 140 0001 C CNN
 F 2 "" H 7400 1950 140 0001 C CNN
 F 3 "" H 7400 1950 140 0001 C CNN
@@
 $EndComp
 $Comp
-L D3NOR-NC-0VDC-expander-nd1021041:D3NOR-NC-0VDC-expander-nd1021041-_B_-___ U508
+L D3NOR-NC-0VDC-expander-nd1021041:D3NOR-NC-0VDC-expander-nd1021041-_3_-___ U508
 U 1 1 5BFAAD8F
 P 8200 8800
 F 0 "U508" H 8200 9125 140 0001 C CNB
-F 1 "D3NOR-NC-0VDC-expander-nd1021041-_B_-___" H 8200 9225 140 0001 C CNN
+F 1 "D3NOR-NC-0VDC-expander-nd1021041-_3_-___" H 8200 9225 140 0001 C CNN
 F 2 "" H 8200 9275 140 0001 C CNN
 F 3 "" H 8200 9275 140 0001 C CNN
@@
 $EndComp
 $Comp
-L D3NOR-NC-0VDC-expander-nd1021041:D3NOR-NC-0VDC-expander-nd1021041-A_C-___ U509
+L D3NOR-NC-0VDC-expander-nd1021041:D3NOR-NC-0VDC-expander-nd1021041-1_5-___ U509
 U 1 1 5BFAAD90
 P 10175 2100
 F 0 "U509" H 10175 2425 140 0001 C CNB
-F 1 "D3NOR-NC-0VDC-expander-nd1021041-A_C-___" H 10175 2525 140 0001 C CNN
+F 1 "D3NOR-NC-0VDC-expander-nd1021041-1_5-___" H 10175 2525 140 0001 C CNN
 F 2 "" H 10175 2575 140 0001 C CNN
 F 3 "" H 10175 2575 140 0001 C CNN
@@
 $EndComp
 $Comp
-L D3NOR-+3VDC-0VDC-nd1021041:D3NOR-+3VDC-0VDC-nd1021041-_B_-___ U511
+L D3NOR-+3VDC-0VDC-nd1021041:D3NOR-+3VDC-0VDC-nd1021041-_3_-___ U511
 U 1 1 5BFAAD93
 P 13100 5425
 F 0 "U511" H 13100 5750 140 0001 C CNB
-F 1 "D3NOR-+3VDC-0VDC-nd1021041-_B_-___" H 13100 5850 140 0001 C CNN
+F 1 "D3NOR-+3VDC-0VDC-nd1021041-_3_-___" H 13100 5850 140 0001 C CNN
 F 2 "" H 13100 5900 140 0001 C CNN
 F 3 "" H 13100 5900 140 0001 C CNN
@@
 $EndComp
 $Comp
-L D3NOR-+3VDC-0VDC-nd1021041:D3NOR-+3VDC-0VDC-nd1021041-ABC-___ U510
+L D3NOR-+3VDC-0VDC-nd1021041:D3NOR-+3VDC-0VDC-nd1021041-135-___ U510
 U 1 1 5BFAAD94
 P 11125 5425
 F 0 "U510" H 11125 5750 140 0001 C CNB
-F 1 "D3NOR-+3VDC-0VDC-nd1021041-ABC-___" H 11125 5850 140 0001 C CNN
+F 1 "D3NOR-+3VDC-0VDC-nd1021041-135-___" H 11125 5850 140 0001 C CNN
 F 2 "" H 11125 5900 140 0001 C CNN
 F 3 "" H 11125 5900 140 0001 C CNN
@@
 $EndComp
 $Comp
-L D3NOR-+3VDC-0VDC-nd1021041:D3NOR-+3VDC-0VDC-nd1021041-A_C-___ U502
+L D3NOR-+3VDC-0VDC-nd1021041:D3NOR-+3VDC-0VDC-nd1021041-1_5-___ U502
 U 1 1 5BFAAD95
 P 6150 8800
 F 0 "U502" H 6150 9125 140 0001 C CNB
-F 1 "D3NOR-+3VDC-0VDC-nd1021041-A_C-___" H 6150 9225 140 0001 C CNN
+F 1 "D3NOR-+3VDC-0VDC-nd1021041-1_5-___" H 6150 9225 140 0001 C CNN
 F 2 "" H 6150 9275 140 0001 C CNN
 F 3 "" H 6150 9275 140 0001 C CNN
@@
 $EndComp
 $Comp
-L D3NOR-NC-0VDC-expander-nd1021041:D3NOR-NC-0VDC-expander-nd1021041-A_C-___ U505
+L D3NOR-NC-0VDC-expander-nd1021041:D3NOR-NC-0VDC-expander-nd1021041-1_5-___ U505
 U 1 1 5BFAAD97
 P 7400 6475
 F 0 "U505" H 7400 6800 140 0001 C CNB
-F 1 "D3NOR-NC-0VDC-expander-nd1021041-A_C-___" H 7400 6900 140 0001 C CNN
+F 1 "D3NOR-NC-0VDC-expander-nd1021041-1_5-___" H 7400 6900 140 0001 C CNN
 F 2 "" H 7400 6950 140 0001 C CNN
 F 3 "" H 7400 6950 140 0001 C CNN
@@
 $EndComp
 $Comp
-L D3NOR-+3VDC-0VDC-nd1021041:D3NOR-+3VDC-0VDC-nd1021041-A_C-___ U504
+L D3NOR-+3VDC-0VDC-nd1021041:D3NOR-+3VDC-0VDC-nd1021041-1_5-___ U504
 U 1 1 5BFAAD98
 P 7400 2625
 F 0 "U504" H 7400 2950 140 0001 C CNB
-F 1 "D3NOR-+3VDC-0VDC-nd1021041-A_C-___" H 7400 3050 140 0001 C CNN
+F 1 "D3NOR-+3VDC-0VDC-nd1021041-1_5-___" H 7400 3050 140 0001 C CNN
 F 2 "" H 7400 3100 140 0001 C CNN
 F 3 "" H 7400 3100 140 0001 C CNN
@@
 $EndComp
 $Comp
-L D3NOR-+3VDC-0VDC-nd1021041:D3NOR-+3VDC-0VDC-nd1021041-ABC-___ U507
+L D3NOR-+3VDC-0VDC-nd1021041:D3NOR-+3VDC-0VDC-nd1021041-135-___ U507
 U 1 1 5BFAAD99
 P 7450 5425
 F 0 "U507" H 7450 5750 140 0001 C CNB
-F 1 "D3NOR-+3VDC-0VDC-nd1021041-ABC-___" H 7450 5850 140 0001 C CNN
+F 1 "D3NOR-+3VDC-0VDC-nd1021041-135-___" H 7450 5850 140 0001 C CNN
 F 2 "" H 7450 5900 140 0001 C CNN
 F 3 "" H 7450 5900 140 0001 C CNN
@@
 	5525 9150 5125 9150
 $Comp
-L D3NOR-+3VDC-0VDC-nd1021041:D3NOR-+3VDC-0VDC-nd1021041-A_C-___ U501
+L D3NOR-+3VDC-0VDC-nd1021041:D3NOR-+3VDC-0VDC-nd1021041-1_5-___ U501
 U 1 1 615D1A04
 P 3650 2975
 F 0 "U501" H 3650 3300 140 0001 C CNB
-F 1 "D3NOR-+3VDC-0VDC-nd1021041-A_C-___" H 3650 3400 140 0001 C CNN
+F 1 "D3NOR-+3VDC-0VDC-nd1021041-1_5-___" H 3650 3400 140 0001 C CNN
 F 2 "" H 3650 3450 140 0001 C CNN
 F 3 "" H 3650 3450 140 0001 C CNN

Commit message: Fixed up netlistCompare.py, as well as several bugs in both 1006556A and r.  There are still bugs to fix in them, as well as actual structural mismatches to document, but I'm making progress.
Parts:
- removed unit 29 of J1
Connections:
- net DV0: now reaches U501.5, U505.5
Changed lines of the file:
@@
-	1    0    0    -1
-$EndComp
-$Comp
-L AGC_DSKY:ConnectorGeneric J1
-U 29 1 5BFAAD9E
-P 1950 3325
-F 0 "J1" H 1950 3650 140 0001 C CNN
-F 1 "ConnectorGeneric" H 1950 3750 140 0001 C CNN
-F 2 "" H 1950 3800 140 0001 C CNN
-F 3 "" H 1950 3800 140 0001 C CNN
-F 4 "DV0" H 1400 3275 140 0000 C BNB "Caption"
-	29   1950 3325
 	1    0    0    -1
 $EndComp
@@
 Text HLabel 5925 5425 0    140  Input ~ 28
 MP1
+Text HLabel 2225 3325 0    140  Input ~ 28
+DV0
 $EndSCHEMATC

Commit message: Visual fixes were made using eelint, and some nominal electrical changes were made to accommodate current state of KiCad ERC capability. Nevertheless, ERC does not pass, due (I think) to current bugs in KiCad ERC.  Netlist changes are purely nominal, and relate to the addition of non-functional nodes in the power and ground nets.
Parts:
- added N501, N502: Node2, symbol AGC_DSKY:Node2
Connections:
- net +3VDC: now also N501.1
- net 0VDC: now also N502.1
Changed lines of the file:
@@
-EESchema Schematic File Version 4
+EESchema Schematic File Version 5
 LIBS:module-cache
 EELAYER 29 0
@@
 Text HLabel 2225 3325 0    140  Input ~ 28
 DV0
+$Comp
+L AGC_DSKY:Node2 N?
+U 1 1 5CE1E4D7
+P 2550 9825
+AR Path="/5F3224B7/5CE1E4D7" Ref="N?"  Part="1"
+AR Path="/5F32147E/5CE1E4D7" Ref="N501"  Part="1"
+F 0 "N501" H 2550 9925 50  0001 C CNN
+F 1 "Node2" H 2550 10000 50  0001 C CNN
+F 2 "" H 2550 9825 50  0001 C CNN
+F 3 "" H 2550 9825 50  0001 C CNN
+F 4 "+3VDC" H 2475 9825 140 0001 R CNB "Caption"
+	1    2550 9825
+	-1   0    0    1
+$EndComp
+$Comp
+L AGC_DSKY:Node2 N?
+U 1 1 5CE1E4E0
+P 2550 10100
+AR Path="/5F3224B7/5CE1E4E0" Ref="N?"  Part="0"
+AR Path="/5F32147E/5CE1E4E0" Ref="N502"  Part="1"
+F 0 "N502" H 2550 10200 50  0001 C CNN
+F 1 "Node2" H 2550 10275 50  0001 C CNN
+F 2 "" H 2550 10100 50  0001 C CNN
+F 3 "" H 2550 10100 50  0001 C CNN
+F 4 "0VDC" H 2475 10100 140 0001 R CNB "Caption"
+	1    2550 10100
+	-1   0    0    1
+$EndComp
+Wire Wire Line
+	1625 10100 2475 10100
+Wire Wire Line
+	1625 9825 2475 9825
 $EndSCHEMATC
