File: Schematics/2005257-/2005257--p2of2.sch (KiCad schematic (older format))
At the start: 66 parts, among them J3 ConnectorA1-300, J4 ConnectorA1-400, U201 D3NOR-+4SW-0VDCA-B_C-EDF, U202 D3NOR-+4SW-0VDCA-B_C-E_F, U203 D3NOR-+4SW-0VDCA-ABC-DEF, U204 D3NOR-+4SW-0VDCA-B_C-E_F, U205 D3NOR-FAP-0VDCA-expander-ACB-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, U206 D3NOR-+4SW-0VDCA-B_C-DFE, U207 D3NOR-+4SW-0VDCA-B_C-E_F, U208 D3NOR-+4SW-0VDCA-B_C-EDF, U209 D3NOR-+4SW-0VDCA-ABC-E_F, U210 D3NOR-+4SW-0VDCA-B_C-E_F, U211 D3NOR-+4SW-0VDCA-B_C-E_F, U212 D3NOR-+4SW-0VDCA-B_C-DFE, U213 D3NOR-+4SW-0VDCA-B_C-E_F, U214 D3NOR-+4SW-0VDCA-B_C-_F_, U215 D3NOR-+4SW-0VDCA-B_C-E_F, U216 D3NOR-+4SW-0VDCA-B_C-E_F, U217 D3NOR-+4SW-0VDCA-BAC-DEF, U218 D3NOR-FAP-0VDCA-expander-B_C-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, U219 D3NOR-+4SW-0VDCA-B_C-E_F, U220 D3NOR-+4SW-0VDCA-B_C-E_F, U221 D3NOR-FAP-0VDCA-expander-ABC-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, U222 D3NOR-+4SW-0VDCA-B_C-DFE, U223 D3NOR-+4SW-0VDCA-B_C-E_F, U224 D3NOR-+4SW-0VDCA-B_C-E_F, U225 D3NOR-+4SW-0VDCA-B_C-E_F, U226 D3NOR-+4SW-0VDCA-B_C-_F_, U227 D3NOR-FAP-0VDCA-expander-ACB-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, U228 D3NOR-+4SW-0VDCA-B_C-_F_, U229 D3NOR-+4SW-0VDCA-B_C-_F_, U230 D3NOR-+4SW-0VDCA-B_C-_F_, U231 D3NOR-+4SW-0VDCA-B_C-EDF, U232 D3NOR-+4SW-0VDCA-B_C-E_F, U233 D3NOR-+4SW-0VDCA-ABC-DEF, U234 D3NOR-+4SW-0VDCA-B_C-E_F, U235 D3NOR-+4SW-0VDCA-B_C-E_F, U236 D3NOR-FAP-0VDCA-expander-ACB-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, U237 D3NOR-+4SW-0VDCA-B_C-E_F, U238 D3NOR-+4SW-0VDCA-B_C-EDF, U239 D3NOR-+4SW-0VDCA-ABC-E_F, U240 D3NOR-+4SW-0VDCA-B_C-E_F, U241 D3NOR-+4SW-0VDCA-B_C-E_F, U242 D3NOR-+4SW-0VDCA-B_C-DEF, U243 D3NOR-+4SW-0VDCA-B_C-E_F, U244 D3NOR-+4SW-0VDCA-B_C-_F_, U245 D3NOR-+4SW-0VDCA-B_C-DEF, U246 D3NOR-+4SW-0VDCA-B_C-E_F, U247 D3NOR-+4SW-0VDCA-ABC-DEF, U248 D3NOR-FAP-0VDCA-expander-B_C-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, U249 D3NOR-+4SW-0VDCA-B_C-E_F, U250 D3NOR-+4SW-0VDCA-B_C-E_F, U251 D3NOR-FAP-0VDCA-expander-ABC-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, U252 D3NOR-+4SW-0VDCA-B_C-DFE, U253 D3NOR-+4SW-0VDCA-B_C-E_F, U254 D3NOR-+4SW-0VDCA-B_C-E_F, U255 D3NOR-+4SW-0VDCA-B_C-E_F, U256 D3NOR-+4SW-0VDCA-B_C-_F_, U257 D3NOR-FAP-0VDCA-expander-ACB-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, U258 D3NOR-+4SW-0VDCA-B_C-_F_, U259 D3NOR-+4SW-0VDCA-B_C-_F_, U260 D3NOR-+4SW-0VDCA-B_C-_F_, X301 ArrowTwiddle, X302 ArrowTwiddle, X303 ArrowTwiddle

Commit message: Transcribed CAD for drawing 2005257- (Block II AGC 2003200 module A10), but have only proofed sheet 1.  Similarly, made associated changes to drawing 2005257A (for AGC 2003993), but presumably have more fixes after sheet 2 of 2005257- is proofed.
Other:
- note added: "Notes from the Virtual AGC Project:\nc). The original drawing did not indicate reference designators, so this CAD drawing\n does not do so either. For purposes of netlist generation or ERC, the NOR gates\n have reference designators U2nn, where nn is the 2-digit number shown on the\n NOR-gate symbol. The oval pads numbered 301-371 comprise connector J3, while\n those numbered 401-471 comprise con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"
- note added: "TO PIN V OF GATES"
- note removed: "Notes from the Virtual AGC Project:\n1. This CAD drawing was adapted from the previously-transcribed original Apollo Program\n drawing 2005256A, and does not itself date from the Apollo Project. — RSB 2018\n2. The original drawing did not indicate reference designators, so this CAD drawing\n does not do so either. For purposes of netlist generation or ERC, the NOR gates\n have reference designato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"
- note removed: "TO PIN V OF\nGATES"

Commit message: Finished proofing of CAD drawing 2005257- and associated changes to 2005257A.
Other:
- note added: "TO PIN G &\nUNUSED INPUTS OF\n53300 & 53400\nSERIES GATES"
- note added: "TO PIN V OF\n53300 & 53400\nSERIES GATES \nEXCEPT THOSE\nGATES TIED TO\nFAP PIN (427)"
- note removed: "TO PIN G &\nUNUSED INPUTS OF\n53300 AND 53400\nSERIES GATES"
- note removed: "TO PIN V OF\n53300 AND 53400\nSERIES GATES \nEXCEPT THOSE\nGATES TIED TO\nFAP PIN (427)"

Commit message: Visual fixes made with eelint.  ERC fails due to temporary KiCad bugs. Netlist unchanged.
Changed lines of the file:
@@
 EESchema Schematic File Version 5
-LIBS:module-cache
+LIBS:errors-cache
 EELAYER 29 0
 EELAYER END
 $Descr E 44000 34000
 encoding utf-8
-Sheet 3 3
+Sheet 1 1
 Title ""
 Date ""
@@
 	28250 3825 28250 3200
 Wire Wire Line
-	30300 5100 30325 5100
+	30300 5100 30350 5100
 Wire Wire Line
-	30325 5100 30325 5625
+	30350 5100 30350 5625
 Wire Wire Line
-	30325 5625 30475 5625
+	30350 5625 30475 5625
 Wire Wire Line
 	32325 5175 32625 5175
@@
 	23950 19625 24100 19625
 Wire Wire Line
-	26000 20250 26000 20275
-Wire Wire Line
 	26000 20775 25925 20775
 Wire Wire Line
@@
 Wire Wire Line
 	26000 20275 23950 19900
-Connection ~ 26000 20275
-Wire Wire Line
-	26000 20275 26000 20775
 Wire Wire Line
 	29375 15900 30375 15900
@@
 	2950 8200 3150 8200
 Wire Wire Line
-	2850 4775 2400 4775
+	2850 4775 2425 4775
 Wire Wire Line
-	2400 4775 2425 8750
+	2425 4775 2425 8750
 Wire Wire Line
 	2425 30125 2150 30125
@@
 	6300 17275 6025 17275
 Wire Wire Line
-	9775 19300 9775 18700
+	9775 19300 9775 18725
 Wire Wire Line
-	9775 18700 27375 18725
+	9775 18725 27375 18725
 Wire Wire Line
 	27375 18725 27375 19350
@@
 Wire Wire Line
 	8850 31125 9825 31125
+Wire Wire Line
+	26000 20275 26000 20775
 $EndSCHEMATC
