File: Schematics/2005258-/2005258--p1of2.sch (KiCad schematic (older format))
At the start: 69 parts, among them J1 ConnectorA1-100, J2 ConnectorA1-200, U101 D3NOR-+4SW-0VDCA-B_C-_F_, U102 D3NOR-+4SW-0VDCA-B_C-_F_, U103 D3NOR-+4SW-0VDCA-B_C-_F_, U104 D3NOR-FAP-0VDCA-expander-ABC-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, U105 D3NOR-+4SW-0VDCA-B_C-_F_, U106 D3NOR-+4SW-0VDCA-B_C-E_F, U107 D3NOR-+4SW-0VDCA-B_C-E_F, U108 D3NOR-+4SW-0VDCA-B_C-E_F, U109 D3NOR-+4SW-0VDCA-B_C-EDF, U110 D3NOR-FAP-0VDCA-expander-ABC-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, U111 D3NOR-+4SW-0VDCA-B_C-E_F, U112 D3NOR-+4SW-0VDCA-B_C-E_F, U113 D3NOR-FAP-0VDCA-expander-B_C-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, U114 D3NOR-+4SW-0VDCA-ABC-DFE, U115 D3NOR-+4SW-0VDCA-B_C-E_F, U116 D3NOR-+4SW-0VDCA-B_C-DFE, U117 D3NOR-+4SW-0VDCA-B_C-_F_, U118 D3NOR-+4SW-0VDCA-B_C-E_F, U119 D3NOR-+4SW-0VDCA-B_C-DFE, U120 D3NOR-+4SW-0VDCA-B_C-E_F, U121 D3NOR-+4SW-0VDCA-B_C-E_F, U122 D3NOR-+4SW-0VDCA-ACB-E_F, U123 D3NOR-+4SW-0VDCA-B_C-EDF, U124 D3NOR-+4SW-0VDCA-B_C-E_F, U125 D3NOR-FAP-0VDCA-expander-ABC-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, U126 D3NOR-+4SW-0VDCA-B_C-E_F, U127 D3NOR-+4SW-0VDCA-B_C-E_F, U128 D3NOR-+4SW-0VDCA-ACB-DFE, U129 D3NOR-+4SW-0VDCA-B_C-E_F, U130 D3NOR-+4SW-0VDCA-B_C-EDF, U131 D3NOR-+4SW-0VDCA-B_C-_F_, U132 D3NOR-+4SW-0VDCA-B_C-_F_, U133 D3NOR-+4SW-0VDCA-B_C-_F_, U134 D3NOR-FAP-0VDCA-expander-BAC-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, U135 D3NOR-+4SW-0VDCA-B_C-_F_, U136 D3NOR-+4SW-0VDCA-B_C-E_F, U137 D3NOR-+4SW-0VDCA-B_C-E_F, U138 D3NOR-+4SW-0VDCA-B_C-E_F, U139 D3NOR-+4SW-0VDCA-B_C-DEF, U140 D3NOR-FAP-0VDCA-expander-ABC-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, U141 D3NOR-+4SW-0VDCA-B_C-E_F, U142 D3NOR-+4SW-0VDCA-B_C-E_F, U143 D3NOR-FAP-0VDCA-expander-B_C-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, U144 D3NOR-+4SW-0VDCA-ACB-DFE, U145 D3NOR-+4SW-0VDCA-B_C-E_F, U146 D3NOR-+4SW-0VDCA-B_C-E_F, U147 D3NOR-+4SW-0VDCA-B_C-_F_, U148 D3NOR-+4SW-0VDCA-B_C-E_F, U149 D3NOR-+4SW-0VDCA-B_C-DFE, U150 D3NOR-+4SW-0VDCA-B_C-E_F, U151 D3NOR-+4SW-0VDCA-B_C-E_F, U152 D3NOR-+4SW-0VDCA-ACB-E_F, U153 D3NOR-+4SW-0VDCA-B_C-EDF, U154 D3NOR-+4SW-0VDCA-B_C-E_F, U155 D3NOR-+4SW-0VDCA-B_C-DEF, U156 D3NOR-FAP-0VDCA-expander-B_C-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, U157 D3NOR-+4SW-0VDCA-B_C-E_F, U158 D3NOR-+4SW-0VDCA-ACB-DFE, U159 D3NOR-+4SW-0VDCA-B_C-E_F, U160 D3NOR-+4SW-0VDCA-B_C-EDF, X201 OvalBody2, X202 DualNorBody, X203 NorExpanderBody, X204 NorBody, X205 ArrowTwiddle, X206 ArrowTwiddle, X207 ArrowTwiddle

Commit message: Added/proofed electrical CAD transcription of drawing 2005258- (module A11 for AGC 2003200), and made related cosmetic fixes to 2005258A (same, for AGC 2003993).
Other:
- note added: "Notes from the Virtual AGC Project:\na) This CAD drawing was adapted from the previously-transcribed original Apollo\n Program drawing 2005258A. — RSB 2019\nb) The original drawing did not indicate reference designators, so this CAD drawing\n does not do so either. For purposes of netlist generation or ERC, the NOR gates\n have reference designators U1nn, where nn is the 2-digit number shown on t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"
- note added: "TO PIN G &\nUNUSED INPUT OF\n54100 & 54200\nSERIES GATES"
- note removed: "A REVISED PER TDRR 30754"
- note removed: "Notes from the Virtual AGC Project:\n1. This CAD drawing was adapted from the previously-transcribed original Apollo\n Program drawing 2005257A, but does not itself date from the Apollo Project. \n — RSB 2018\n2. The original drawing did not indicate reference designators, so this CAD drawing\n does not do so either. For purposes of netlist generation or ERC, the NOR gates\n have reference design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"
- note removed: "TO PIN G &\nUNUSED INPUT OF\n54100 AND 54200\nSERIES GATES"

Commit message: Visual fixes made with eelint.  ERC fails due to temporary KiCad bugs. Netlist unchanged.
Changed lines of the file:
@@
 EESchema Schematic File Version 5
-LIBS:module-cache
+LIBS:errors-cache
 EELAYER 29 0
 EELAYER END
 $Descr E 44000 34000
 encoding utf-8
-Sheet 2 3
+Sheet 1 1
 Title ""
 Date ""
@@
 L AGC_DSKY:ConnectorA1-100 J1
 U 20 1 61AB5E1B
-P 1925 13600
-F 0 "J1" H 1925 13925 140 0001 C CNN
-F 1 "ConnectorA1-100" H 1925 14025 140 0001 C CNN
-F 2 "" H 1925 14075 140 0001 C CNN
-F 3 "" H 1925 14075 140 0001 C CNN
-F 4 "WALSG/" H 1175 13525 140 0000 C BNB "Caption"
-	20   1925 13600
+P 1925 13625
+F 0 "J1" H 1925 13950 140 0001 C CNN
+F 1 "ConnectorA1-100" H 1925 14050 140 0001 C CNN
+F 2 "" H 1925 14100 140 0001 C CNN
+F 3 "" H 1925 14100 140 0001 C CNN
+F 4 "WALSG/" H 1175 13550 140 0000 C BNB "Caption"
+	20   1925 13625
 	1    0    0    -1
 $EndComp
@@
 	26225 8225 26100 8225
 Wire Wire Line
-	20100 4850 20100 8750
+	20125 4850 20125 8750
 Wire Wire Line
-	20100 8750 20900 8750
+	20125 8750 20900 8750
 Wire Wire Line
-	20625 4850 20100 4850
+	20625 4850 20125 4850
 Wire Wire Line
 	17400 5950 17500 5950
@@
 	24325 13600 24150 13600
 Wire Wire Line
-	20100 8750 20100 12425
+	20125 8750 20125 12425
 Wire Wire Line
-	20100 12425 20900 12425
-Connection ~ 20100 8750
+	20125 12425 20900 12425
+Connection ~ 20125 8750
 Wire Wire Line
 	20900 13025 19900 13025
@@
 	3150 13625 3000 13625
 Wire Wire Line
-	2200 13625 2200 13600
-Wire Wire Line
 	4950 12200 5075 12200
 Wire Wire Line
@@
 	20825 15575 20650 15575
 Wire Wire Line
-	20100 12425 20125 16125
+	20125 12425 20125 16125
 Wire Wire Line
 	20125 16125 20825 16125
-Connection ~ 20100 12425
+Connection ~ 20125 12425
 Wire Wire Line
 	20125 16125 20125 19825
