File: Schematics/2005259-/2005259--p1of2.sch (KiCad schematic (older format))
At the start: 63 parts, among them J1 ConnectorA1-100, J2 ConnectorA1-200, U101 D3NOR-+4VDC-0VDCA-B_C-E_F, U102 D3NOR-+4VDC-0VDCA-B_C-E_F, U103 D3NOR-+4VDC-0VDCA-ABC-E_F, U104 D3NOR-+4VDC-0VDCA-ABC-E_F, U105 D3NOR-+4VDC-0VDCA-B_C-E_F, U106 D3NOR-+4VDC-0VDCA-B_C-E_F, U107 D3NOR-+4VDC-0VDCA-ABC-E_F, U108 D3NOR-+4VDC-0VDCA-ABC-E_F, U109 D3NOR-+4VDC-0VDCA-B_C-E_F, U110 D3NOR-+4VDC-0VDCA-ACB-E_F, U111 D3NOR-+4VDC-0VDCA-BAC-E_F, U112 D3NOR-+4VDC-0VDCA-A_B-E_F, U113 D3NOR-+4VDC-0VDCA-B_C-E_F, U114 D3NOR-+4VDC-0VDCA-ACB-E_F, U115 D3NOR-+4VDC-0VDCA-BAC-E_F, U116 D3NOR-+4VDC-0VDCA-B_C-E_F, U117 D3NOR-+4VDC-0VDCA-ACB-E_F, U118 D3NOR-+4VDC-0VDCA-ABC-E_F, U119 D3NOR-+4VDC-0VDCA-A_B-E_F, U120 D3NOR-+4VDC-0VDCA-B_C-E_F, U121 D3NOR-+4VDC-0VDCA-ACB-E_F, U122 D3NOR-+4VDC-0VDCA-BAC-E_F, U123 D3NOR-+4VDC-0VDCA-B_C-E_F, U124 D3NOR-+4VDC-0VDCA-A_C-E_F, U125 D3NOR-+4VDC-0VDCA-ABC-DFE, U126 D3NOR-+4VDC-0VDCA-A_B-E_F, U127 D3NOR-+4VDC-0VDCA-B_C-E_F, U128 D3NOR-+4VDC-0VDCA-ABC-E_F, U129 D3NOR-+4VDC-0VDCA-ABC-E_F, U132 D3NOR-+4VDC-0VDCA-B_C-EDF, U133 D3NOR-+4VDC-0VDCA-B_C-EDF, U134 D3NOR-+4VDC-0VDCA-B_C-E_F, U135 D3NOR-+4VDC-0VDCA-B_C-E_F, U136 D3NOR-+4VDC-0VDCA-B_C-E_F, U137 D3NOR-+4VDC-0VDCA-BAC-DEF, U138 D3NOR-+4VDC-0VDCA-B_C-E_F, U139 D3NOR-+4VDC-0VDCA-B_C-E_F, U140 D3NOR-+4VDC-0VDCA-BAC-DEF, U141 D3NOR-+4VDC-0VDCA-B_C-E_F, U142 D3NOR-+4VDC-0VDCA-B_C-E_F, U143 D3NOR-+4VDC-0VDCA-B_C-E_F, U144 D3NOR-+4VDC-0VDCA-ABC-DFE, U145 D3NOR-+4VDC-0VDCA-B_C-E_F, U146 D3NOR-+4VDC-0VDCA-BAC-E_F, U147 D3NOR-+4VDC-0VDCA-BAC-E_F, U148 D3NOR-+4VDC-0VDCA-B_C-E_F, U149 D3NOR-+4VDC-0VDCA-B_C-E_F, U150 D3NOR-+4VDC-0VDCA-ABC-E_F, U151 D3NOR-+4VDC-0VDCA-BAC-E_F, U152 D3NOR-+4VDC-0VDCA-B_C-E_F, U153 D3NOR-+4VDC-0VDCA-B_C-E_F, U154 D3NOR-+4VDC-0VDCA-ABC-E_F, U155 D3NOR-+4VDC-0VDCA-B_C-E_F, U156 D3NOR-+4VDC-0VDCA-B_C-E_F, U157 D3NOR-+4VDC-0VDCA-BAC-E_F, U158 D3NOR-+4VDC-0VDCA-BAC-E_F, U159 D3NOR-+4VDC-0VDCA-B_C-E_F, U160 D3NOR-+4VDC-0VDCA-B_C-E_F, X1 OvalBody, X2 NorBody, X3 NorExpanderBody

Commit message: Added/proofed CAD transcription for drawing 2005259- (electrical schematic of Block II AGC 2003200 logic module A1).  Fixed several bugs in related drawing 2005259A (same thing but for AGC 2003993), so I now regard 2005259A as being "proofed".  None of the fixes were electrical, except that two input pins of NOR gate 38125 had been swapped.  I found no differences of any kind (other than the revision-letter change itself) between these two revisions of the drawing.
Other:
- note added: "2."
- note added: "3. SEE DWG. NO.2005011 FOR LOGIC DESIGN CRITERIA\n4. SYMBOLIC REPRESENTATION OF DUAL\n NOR GATE\n"
- note added: "5. SPARE PINS DENOTE NO CONNECTION WITHIN\n THE MODULE FOR EXTERNAL CONNECTION\n INFORMATION SEE COMPUTER WIRE LIST\n"
- note added: "6."
- note added: "7."
- note added: "DENOTES PIN NO.\n"
- note added: "Notes from the Virtual AGC Project:\na) This CAD sheet was adapted from sheet 1 of the previously-transcribed original\n Apollo Program drawing 2005259A, to conform to the original drawing 2005259-.\n — RSB 2019\nb) The original drawing did not assign reference designators as such to components.\n The transcription process has assigned the reference designators U1nn to the NOR\n gates, where nn i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"
- note added: "SYMBOL FOR EXPANDER DUAL NOR GATE\nSCD NO.1006394"
- note added: "UPPER NUMBER DENOTES GATE SHOWN.\nLOWER DENOTES PHYSICAL\nLOCATION OF GATE ON CIRCUIT BOARD,\nMULTILAYER SCD NO.1006395\n"
- note removed: "2. DENOTES PIN NO.\n"
- note removed: "3. SEE DWG. NO.2005011 FOR LOGIC DESIGN CRITERIA\n 4. SYMBOLIC REPRESENTATION OF DUAL\n NOR GATE\n\n\n\n 5. SPARE PINS DENOTE NO CONNECTION WITHIN\n THE MODULE FOR EXTERNAL CONNECTION\n INFORMATION SEE COMPUTER WIRE LIST\n \n UPPER NUMBER DENOTES GATE SHOWN.\n 6. LOWER DENOTES PHYSICAL\n LOCATION OF GATE ON CIRCUIT BOARD,\n MULTILAYER SCD NO.1006395\n\n 7. SYMBOL FOR EXPANDER DUAL NOR GATE\n SCD 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"
- note removed: "A"
- note removed: "Notes from the Virtual AGC Project:\n1. This CAD drawing was manually transcribed from the original Apollo Program\n drawing 2005259A, page 1 of 2, but is not itself from the time of Apollo — RSB 2018\n2. The original drawing did not assign reference designators as such to components.\n The transcription process has assigned the reference designators U1nn to the NOR\n gates, where nn is the two-d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"
- note removed: "REVISED PER TDRR 30754"
