File: Schematics/2005919A/2005919A-p1of2.sch (KiCad schematic (older format))
At the start: 58 parts, among them J1 ConnectorB8-100, J2 ConnectorB8-200, Q10 Transistor-PNP, Q11 Transistor-NPN, Q2 Transistor-NPN, Q3 Transistor-NPN, Q4 Transistor-PNP, Q5 Transistor-NPN, Q6 Transistor-NPN, Q7 Transistor-PNP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

Commit message: Added CAD transcription of drawing 2005919A (sense amplifier module B14 for AGC 2003200).  Since B14 is structurally identical to yesterday's module B13, with just some signal names changed, this also highlighted several errors in drawing 2005920B that I fixed as well.
Parts:
- removed unit 42 of J1
- removed unit 16 of J1
- removed unit 62 of J1
- removed unit 52 of J1
- removed unit 9 of J1
- removed unit 2 of J1
- removed unit 1 of J1
- removed unit 7 of J1
- removed unit 5 of J1
- removed unit 4 of J1
- removed unit 13 of J1
- removed unit 10 of J1
- removed unit 14 of J1
- removed unit 38 of J1
- removed unit 64 of J1
- removed unit 18 of J1
- removed unit 21 of J1
- removed unit 58 of J1
- removed unit 54 of J1
- removed unit 56 of J1
- removed unit 50 of J1
- removed unit 51 of J1
- removed unit 40 of J1
- removed unit 57 of J1
- removed unit 36 of J1
- removed unit 20 of J1
- removed unit 23 of J1
- removed unit 25 of J1
- removed unit 27 of J1
- removed unit 47 of J1
- removed unit 45 of J1
- removed unit 43 of J1
- removed unit 15 of J2
- removed unit 56 of J2
- removed unit 55 of J2
- removed unit 18 of J2
- removed unit 53 of J2
- removed unit 51 of J2
- removed unit 12 of J2
- removed unit 16 of J2
- removed unit 14 of J2
- removed unit 44 of J2
- removed unit 10 of J2
- removed unit 5 of J2
- removed unit 39 of J2
- removed unit 37 of J2
- removed unit 38 of J2
- removed unit 58 of J2
- removed unit 2 of J2
- removed unit 62 of J2
- removed unit 9 of J2
- removed unit 46 of J2
- removed unit 61 of J2
- removed unit 40 of J2
- removed unit 41 of J2
- removed unit 42 of J2
- removed unit 1 of J2
- removed unit 3 of J2
- removed unit 4 of J2
- removed unit 49 of J2
- removed unit 7 of J2
- removed unit 63 of J2
- removed unit 8 of J2
- removed unit 25 of J2
- removed unit 60 of J2
- removed unit 45 of J2
- removed unit 26 of J2
- removed unit 19 of J2
- removed unit 22 of J2
- removed unit 23 of J2
- removed unit 21 of J2
- removed unit 52 of J2
- added Q301: Transistor-PNP, symbol AGC_DSKY:Transistor-PNP
- added R301, R302, R303, R304: 2700, symbol AGC_DSKY:Resistor
- added R305, R306, R307, R308: 470, symbol AGC_DSKY:Resistor
- added R309, R310: NOM, symbol AGC_DSKY:Resistor
- added R311, R312: 1000, symbol AGC_DSKY:Resistor
- added R313: 5100, symbol AGC_DSKY:Resistor
- added R314: 2000, symbol AGC_DSKY:Resistor
- added SA301, SA302: SENSEAMP, symbol AGC_DSKY:SENSEAMP
- added T301: Transformer2, symbol AGC_DSKY:Transformer2
- added T302: Transformer2A, symbol AGC_DSKY:Transformer2A
- J1: Caption STROBE -> STROBF
- J2: Caption SBE -> SBF
- J2: Caption VYE2 -> VYF2
- J2: Caption VYE1 -> VYF1
- J2: Caption VZE -> VZF
- J2: Caption VXE -> VXF
- J2: Caption CGB13 -> CGB14
Connections:
- net labels added: A, B, C, D, E, F, G, H, I, J, STROBF, VXF, VZF
- net labels removed: STROBE, VXE, VYE1, VYE2, VZE
- wire segments 316 -> 268
Other:
- note added: "1 2"
- note added: "2005919"
- note added: "CIRCUIT NO. 40611-40618"
- note added: "CIRCUIT NO. 40619"
- note added: "CIRCUIT NO. 40620"
- note added: "CIRCUIT NO. 40621"
- note added: "ERASABLE MEMORY B14"
- note added: "Notes from the Virtual AGC Project:\n1. This drawing was adapted from a CAD drawing previously transcribed from the \n original Apollo Program drawing 2005920B, and then cross-checked against the\n original Apollo Program drawing 2005919A. This CAD drawing itself does not \n date from the Apollo period. — RSB 2018\n2. This CAD drawing is intended only to represent the visual appearance of the ori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"
- note added: "REVISED PER TDRR 30751\nDR CHK APPD"
- note added: "SENSE AMPLIFIER ASSY DWG NO. 2003981"
- note added: "VYF1\nVYF2"
- note removed: "-"
- note removed: "2005920"
- note removed: "B"
- note removed: "CIRCUIT NO. 40600"
- note removed: "CIRCUIT NO. 40601-40608"
- note removed: "CIRCUIT NO. 40609"
- note removed: "CIRCUIT NO. 40610"
- note removed: "ERASABLE MEMORY B13"
- note removed: "Notes from the Virtual AGC Project:\n1. This drawing was manually transcribed from the original Apollo Program drawing\n 2005920B, but does not itself date from the Apollo period. — RSB 2018\n2. The oval pads numbered 101-169 comprise connector J1, while those numbered\n 201-269 comprise connector J2. — RSB 2018\n3. The CAD drawing differs in the visual appearance of circuits 40601 - 40608, \n co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"
- note removed: "RELEASED PER TDRR"
- note removed: "REVISED PER TDRR 29077\nDR CHK APPD"
- note removed: "REVISED PER TDRR 29821\nDR CHK APPD"
- note removed: "SENSE AMPLIFIER ASSY DWG NO. 2003982"
- moved on the sheet: C2, CR1, CR2, Q2, Q3, R15, R16, R17, R18, R19, R36

Commit message: Made visual fixes with eelint.  ERC passes.  Netlist unchanged.
Other:
- moved on the sheet: Q10
Changed lines of the file:
@@
-EESchema Schematic File Version 4
-LIBS:original-cache
+EESchema Schematic File Version 5
+LIBS:errors-cache
 EELAYER 29 0
 EELAYER END
 $Descr E 44000 34000
 encoding utf-8
-Sheet 2 3
+Sheet 1 1
 Title ""
 Date ""
@@
 L AGC_DSKY:Transistor-PNP Q10
 U 1 1 5C65279F
-P 30125 20200
-F 0 "Q10" H 30875 20200 130 0000 C CNN
-F 1 "Transistor-PNP" H 30125 20765 130 0001 C CNN
-F 2 "" H 30125 19950 130 0001 C CNN
-F 3 "" H 30125 19950 130 0001 C CNN
-	1    30125 20200
+P 30125 20225
+F 0 "Q10" H 30875 20225 130 0000 C CNN
+F 1 "Transistor-PNP" H 30125 20790 130 0001 C CNN
+F 2 "" H 30125 19975 130 0001 C CNN
+F 3 "" H 30125 19975 130 0001 C CNN
+	1    30125 20225
 	1    0    0    -1
 $EndComp
@@
 	15875 16300 15875 19400
 Wire Wire Line
-	15875 19400 17400 19400
-Wire Wire Line
-	18900 19400 18900 20600
-Wire Wire Line
 	16675 19100 16675 20250
 Connection ~ 16675 20250
 Wire Wire Line
 	16675 20250 16950 20250
-Wire Wire Line
-	17400 18525 17400 19400
-Connection ~ 17400 19400
-Wire Wire Line
-	17400 19400 18900 19400
-Wire Wire Line
-	17400 20000 17400 19400
-Wire Wire Line
-	17400 19400 17375 19400
-Wire Wire Line
-	18900 19400 18900 19150
-Connection ~ 18900 19400
 Wire Wire Line
 	18900 18350 18900 17850
@@
 	31300 20800 30275 20800
 Wire Wire Line
-	30275 20800 30275 20450
-Wire Wire Line
-	30275 19350 30275 19950
+	30275 20800 30275 20475
+Wire Wire Line
+	30275 19350 30275 19975
 Connection ~ 30275 19350
 Wire Wire Line
@@
 Wire Wire Line
 	29550 17850 30275 17850
-Wire Wire Line
-	29825 20200 29825 20225
 Wire Wire Line
 	29825 20225 29550 20225
@@
 AR Path="/5C96678A/5C5C30E4" Ref="SA1001"  Part="1"
 AR Path="/5B8E7731/5C5C30E4" Ref="SA901"  Part="1"
+AR Path="/5C5C30E4" Ref="SA901"  Part="1"
 F 0 "SA901" H 11075 5750 50  0001 C CNN
 F 1 "SENSEAMP" H 11150 6150 140 0001 C CNN
@@
 AR Path="/5C96678A/5C5C59F8" Ref="SA1002"  Part="1"
 AR Path="/5B8E7731/5C5C59F8" Ref="SA902"  Part="1"
+AR Path="/5C5C59F8" Ref="SA902"  Part="1"
 F 0 "SA902" H 11100 11975 50  0001 C CNN
 F 1 "SENSEAMP" H 11150 12150 140 0001 C CNN
@@
 AR Path="/5C96678A/5C5CD693" Ref="T1001"  Part="1"
 AR Path="/5B8E7731/5C5CD693" Ref="T901"  Part="1"
+AR Path="/5C5CD693" Ref="T901"  Part="1"
 F 0 "T901" H 6225 6650 50  0001 C CNN
 F 1 "Transformer2" H 6300 7025 130 0001 C CNN
@@
 AR Path="/5C96678A/5C5D9082" Ref="T1002"  Part="1"
 AR Path="/5B8E7731/5C5D9082" Ref="T902"  Part="1"
+AR Path="/5C5D9082" Ref="T902"  Part="1"
 F 0 "T902" H 6300 11050 50  0001 C CNN
 F 1 "Transformer2A" H 6325 12975 130 0001 C CNN
@@
 AR Path="/5C96678A/5C5DAD11" Ref="R1001"  Part="1"
 AR Path="/5B8E7731/5C5DAD11" Ref="R901"  Part="1"
+AR Path="/5C5DAD11" Ref="R901"  Part="1"
 F 0 "R901" V 4375 5875 50  0001 C CNN
 F 1 "2700" V 4600 5775 130 0000 C CNN
@@
 AR Path="/5C96678A/5C5DB871" Ref="R1002"  Part="1"
 AR Path="/5B8E7731/5C5DB871" Ref="R902"  Part="1"
+AR Path="/5C5DB871" Ref="R902"  Part="1"
 F 0 "R902" V 4375 6900 50  0001 C CNN
 F 1 "2700" V 4600 6800 130 0000 C CNN
@@
 AR Path="/5C96678A/5C5DC27A" Ref="R1003"  Part="1"
 AR Path="/5B8E7731/5C5DC27A" Ref="R903"  Part="1"
+AR Path="/5C5DC27A" Ref="R903"  Part="1"
 F 0 "R903" V 4400 11875 50  0001 C CNN
 F 1 "2700" V 4625 11775 130 0000 C CNN
@@
 AR Path="/5C96678A/5C5DCE72" Ref="R1004"  Part="1"
 AR Path="/5B8E7731/5C5DCE72" Ref="R904"  Part="1"
+AR Path="/5C5DCE72" Ref="R904"  Part="1"
 F 0 "R904" V 4400 12825 50  0001 C CNN
 F 1 "2700" V 4625 12725 130 0000 C CNN
@@
 L AGC_DSKY:Resistor R305
 U 1 1 5C5DF009
-P 8000 5425
+P 8000 5400
 AR Path="/5C5B2A2B/5C5DF009" Ref="R305"  Part="1"
 AR Path="/5C92E690/5C5DF009" Ref="R405"  Part="1"
@@
 AR Path="/5C96678A/5C5DF009" Ref="R1005"  Part="1"
 AR Path="/5B8E7731/5C5DF009" Ref="R905"  Part="1"
-F 0 "R905" V 7825 5900 50  0001 C CNN
-F 1 "470" V 8050 5800 130 0000 C CNN
-F 2 "" H 8000 5425 130 0001 C CNN
-F 3 "" H 8000 5425 130 0001 C CNN
-F 4 "R5" V 7825 5675 130 0000 C CNN "OREFD"
-	1    8000 5425
+AR Path="/5C5DF009" Ref="R905"  Part="1"
+F 0 "R905" V 7825 5875 50  0001 C CNN
+F 1 "470" V 8050 5775 130 0000 C CNN
+F 2 "" H 8000 5400 130 0001 C CNN
+F 3 "" H 8000 5400 130 0001 C CNN
+F 4 "R5" V 7825 5650 130 0000 C CNN "OREFD"
+	1    8000 5400
 	0    1    1    0
 $EndComp
@@
 AR Path="/5C96678A/5C5E0172" Ref="R1006"  Part="1"
 AR Path="/5B8E7731/5C5E0172" Ref="R906"  Part="1"
+AR Path="/5C5E0172" Ref="R906"  Part="1"
 F 0 "R906" V 7825 6850 50  0001 C CNN
 F 1 "470" V 8050 6750 130 0000 C CNN
@@
 L AGC_DSKY:Resistor R307
 U 1 1 5C5E0AA5
-P 8000 11400
+P 8000 11375
 AR Path="/5C5B2A2B/5C5E0AA5" Ref="R307"  Part="1"
 AR Path="/5C92E690/5C5E0AA5" Ref="R407"  Part="1"
@@
 AR Path="/5C96678A/5C5E0AA5" Ref="R1007"  Part="1"
 AR Path="/5B8E7731/5C5E0AA5" Ref="R907"  Part="1"
-F 0 "R907" V 7825 11875 50  0001 C CNN
-F 1 "470" V 8050 11775 130 0000 C CNN
-F 2 "" H 8000 11400 130 0001 C CNN
-F 3 "" H 8000 11400 130 0001 C CNN
-F 4 "R7" V 7825 11650 130 0000 C CNN "OREFD"
-	1    8000 11400
+AR Path="/5C5E0AA5" Ref="R907"  Part="1"
+F 0 "R907" V 7825 11850 50  0001 C CNN
+F 1 "470" V 8050 11750 130 0000 C CNN
+F 2 "" H 8000 11375 130 0001 C CNN
+F 3 "" H 8000 11375 130 0001 C CNN
+F 4 "R7" V 7825 11625 130 0000 C CNN "OREFD"
+	1    8000 11375
 	0    1    1    0
 $EndComp
@@
 AR Path="/5C96678A/5C5E1613" Ref="R1008"  Part="1"
 AR Path="/5B8E7731/5C5E1613" Ref="R908"  Part="1"
+AR Path="/5C5E1613" Ref="R908"  Part="1"
 F 0 "R908" V 7825 12825 50  0001 C CNN
 F 1 "470" V 8050 12725 130 0000 C CNN
@@
 AR Path="/5C96678A/5C5E1E2C" Ref="R1010"  Part="1"
 AR Path="/5B8E7731/5C5E1E2C" Ref="R910"  Part="1"
+AR Path="/5C5E1E2C" Ref="R910"  Part="1"
 F 0 "R910" V 11500 10225 50  0001 C CNN
 F 1 "NOM" V 11700 9975 130 0000 C CNN
@@
 AR Path="/5C96678A/5C5E2915" Ref="R1009"  Part="1"
 AR Path="/5B8E7731/5C5E2915" Ref="R909"  Part="1"
+AR Path="/5C5E2915" Ref="R909"  Part="1"
 F 0 "R909" V 11500 8750 50  0001 C CNN
 F 1 "NOM" V 11700 8500 130 0000 C CNN
@@
 AR Path="/5C96678A/5C5E3868" Ref="R1012"  Part="1"
 AR Path="/5B8E7731/5C5E3868" Ref="R912"  Part="1"
+AR Path="/5C5E3868" Ref="R912"  Part="1"
 F 0 "R912" V 13825 8775 50  0001 C CNN
 F 1 "1000" V 14025 8525 130 0000 C CNN
@@
 AR Path="/5C96678A/5C5E3E61" Ref="R1013"  Part="1"
 AR Path="/5B8E7731/5C5E3E61" Ref="R913"  Part="1"
+AR Path="/5C5E3E61" Ref="R913"  Part="1"
 F 0 "R913" V 13825 10200 50  0001 C CNN
 F 1 "5100" V 14025 9950 130 0000 C CNN
@@
 AR Path="/5C96678A/5C5E4528" Ref="R1014"  Part="1"
 AR Path="/5B8E7731/5C5E4528" Ref="R914"  Part="1"
+AR Path="/5C5E4528" Ref="R914"  Part="1"
 F 0 "R914" V 14125 13000 50  0001 C CNN
 F 1 "2000" V 14375 12750 130 0000 C CNN
@@
 AR Path="/5C96678A/5C5E4F94" Ref="R1011"  Part="1"
 AR Path="/5B8E7731/5C5E4F94" Ref="R911"  Part="1"
+AR Path="/5C5E4F94" Ref="R911"  Part="1"
 F 0 "R911" H 12925 12050 50  0001 C CNN
 F 1 "1000" H 13175 12250 130 0000 C CNN
@@
 AR Path="/5C96678A/5C5E622F" Ref="Q1001"  Part="1"
 AR Path="/5B8E7731/5C5E622F" Ref="Q901"  Part="1"
+AR Path="/5C5E622F" Ref="Q901"  Part="1"
 F 0 "Q901" V 14175 9775 50  0001 C CNN
 F 1 "Transistor-PNP" H 14275 10915 130 0001 C CNN
@@
 	9975 4850 8000 4850
 Wire Wire Line
-	8000 4850 8000 5025
+	8000 4850 8000 5000
 Wire Wire Line
 	8000 4850 6675 4850
@@
 	6675 6875 8000 6875
 Wire Wire Line
-	8000 5825 8000 5850
+	8000 5800 8000 5850
 Wire Wire Line
 	8000 6775 8000 6875
@@
 	8000 12850 9975 12850
 Wire Wire Line
-	8000 11800 8000 11825
+	8000 11775 8000 11825
 Wire Wire Line
 	8975 11825 8000 11825
@@
 	6700 10825 8000 10825
 Wire Wire Line
-	8000 11000 8000 10825
+	8000 10975 8000 10825
 Connection ~ 8000 10825
 Wire Wire Line
@@
 Wire Notes Line style solid
 	37965 921  37965 1440
+Wire Wire Line
+	18900 19150 18900 19400
+Wire Wire Line
+	15875 19400 17400 19400
+Connection ~ 18900 19400
+Wire Wire Line
+	18900 19400 18900 20600
+Wire Wire Line
+	17400 20000 17400 19400
+Connection ~ 17400 19400
+Wire Wire Line
+	17400 19400 18900 19400
+Wire Wire Line
+	17400 19400 17400 18525
 $EndSCHEMATC
