File: Schematics/2005919A/module.sch (KiCad schematic (older format))
At the start: 58 parts, among them J1 ConnectorB8-100, J2 ConnectorB8-200, Q10 Transistor-PNP, Q11 Transistor-NPN, Q2 Transistor-NPN, Q3 Transistor-NPN, Q4 Transistor-PNP, Q5 Transistor-NPN, Q6 Transistor-NPN, Q7 Transistor-PNP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

Commit message: Added CAD transcription of drawing 2005919A (sense amplifier module B14 for AGC 2003200).  Since B14 is structurally identical to yesterday's module B13, with just some signal names changed, this also highlighted several errors in drawing 2005920B that I fixed as well.
Parts:
- J1: Caption SA06 -> SA05
- J1: Caption STROBE -> STROBF
- J1: Caption SAF10 -> GAR09
- J1, J2: Caption 0VDC -> BPLSWX
- J1: Caption SAF02 -> GAR01
- J1: Caption SAF12 -> GAR11
- J1: Caption SAF14 -> GAR13
- J1: Caption SBF14 -> GBR13
- J1: Caption SBF12 -> GBR11
- J1: Caption SA14 -> SA13
- J1: Caption SA12 -> SA11
- J1: Caption SBF10 -> GBR09
- J1: Caption SAF06 -> GAR05
- J1: Caption SA16 -> SAP
- J1: Caption SBF08 -> GBR07
- J1: Caption SAF16 -> GAR15
- J1: Caption SA02 -> SA01
- J1: Caption SA04 -> SA03
- J1: Caption SBF02 -> GBR01
- J1: Caption SBF16 -> GBR15
- J1: Caption SBF06 -> GBR05
- J1: Caption SA10 -> SA09
- J1: Caption SAF08 -> GAR07
- J1: Caption SA08 -> SA07
- J1: Caption SAF04 -> GAR03
- J1: Caption SBF04 -> GBR03
- J2: Caption SBE -> SBF
- J2: Caption VYE2 -> VYF2
- J2: Caption VYE1 -> VYF1
- J2: Caption VZE -> VZF
- J2: Caption VXE -> VXF
- J2: Caption 40615A -> 40605A
- J2: Caption 40601A -> 40611A
- J2: Caption SAF01 -> GAR02
- J2: Caption SAF09 -> GAR10
- J2: Caption SBF01 -> GBR02
- J2: Caption 40606A -> 40616A
- J2: Caption SBF09 -> GBR10
- J2: Caption SAF11 -> GAR12
- J2: Caption 40607A -> 40617A
- J2: Caption SBF05 -> GBR06
- J2: Caption 40613A -> 40603A
- J2: Caption 40617A -> 40607A
- J2: Caption SAF15 -> GAR16
- J2: Caption SBF11 -> GBR12
- J2: Caption SBF03 -> GBR04
- J2: Caption SBF15 -> GBR16
- J2: Caption SAF03 -> GAR04
- J2: Caption SAF05 -> GAR06
- J2: Caption 40603A -> 40613A
- J2: Caption SBF13 -> GBR14
- J2: Caption SAF13 -> GAR14
- J2: Caption 40602A -> 40612A
- J2: Caption 40608A -> 40618A
- J2: Caption 40616A -> 40606A
- J2: Caption SAF07 -> GAR08
- J2: Caption 40618A -> 40608A
- J2: Caption 40612A -> 40602A
- J2: Caption 40604A -> 40614A
- J2: Caption 40605A -> 40615A
- J2: Caption 40614A -> 40604A
- J2: Caption SBF07 -> GBR08
- J2: Caption 40611A -> 40601A
Connections:
- net labels added: STROBF, VXF, VYF1, VYF2, VZF
- net labels removed: STROBE, VXE, VYE1, VYE2, VZE
Other:
- note added: "2005919"
- note added: "CIRCUIT NO. 40611-40618"
- note added: "CIRCUIT NO. 40619"
- note added: "CIRCUIT NO. 40620"
- note added: "CIRCUIT NO. 40621"
- note added: "ERASABLE MEMORY B14"
- note added: "Notes from the Virtual AGC Project:\n1. This CAD drawing was adapted from a CAD drawing previously transcribed from \n the original Apollo Program drawing 2005920B, and then cross-checked against \n the original Apollo Program drawing 2005919A. However, this CAD drawing does\n not itself date from the Apollo period. — RSB 2018\n2. The oval pads numbered 101-169 comprise connector J1, while those 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"
- note added: "REVISED PER TDRR 30751\nDR CHK APPD"
- note removed: "-"
- note removed: "2005920"
- note removed: "B"
- note removed: "CIRCUIT NO. 40600"
- note removed: "CIRCUIT NO. 40601-40608"
- note removed: "CIRCUIT NO. 40609"
- note removed: "CIRCUIT NO. 40610"
- note removed: "ERASABLE MEMORY B13"
- note removed: "Notes from the Virtual AGC Project:\n1. This drawing was manually transcribed from the original Apollo Program drawing\n 2005920B, but does not itself date from the Apollo period. — RSB 2018\n2. The oval pads numbered 101-169 comprise connector J1, while those numbered\n 201-269 comprise connector J2. — RSB 2018\n3. The CAD drawing differs in the visual appearance of circuits 40601 - 40608, \n co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"
- note removed: "RELEASED PER TDRR"
- note removed: "REVISED PER TDRR 29077\nDR CHK APPD"
- note removed: "REVISED PER TDRR 29821\nDR CHK APPD"

Commit message: Made visual fixes with eelint.  ERC passes.  Netlist unchanged.
Connections:
- wire segments 316 -> 306
Other:
- moved on the sheet: Q10
Changed lines of the file:
@@
-EESchema Schematic File Version 4
-LIBS:module-cache
+EESchema Schematic File Version 5
+LIBS:errors-cache
 EELAYER 29 0
 EELAYER END
@@
 $EndComp
 $Comp
-L AGC_DSKY:Transistor-PNP Q10
-U 1 1 5C65279F
-P 30125 20200
-F 0 "Q10" H 30875 20200 130 0000 C CNN
-F 1 "Transistor-PNP" H 30125 20765 130 0001 C CNN
-F 2 "" H 30125 19950 130 0001 C CNN
-F 3 "" H 30125 19950 130 0001 C CNN
-	1    30125 20200
-	1    0    0    -1
-$EndComp
-$Comp
 L AGC_DSKY:Diode CR12
 U 1 1 5C653496
@@
 	15875 16300 15875 19400
 Wire Wire Line
-	15875 19400 17400 19400
-Wire Wire Line
-	18900 19400 18900 20600
-Wire Wire Line
 	16675 19100 16675 20250
 Connection ~ 16675 20250
@@
 	16675 20250 16950 20250
 Wire Wire Line
-	17400 18925 17400 19400
-Connection ~ 17400 19400
-Wire Wire Line
-	17400 19400 18900 19400
-Wire Wire Line
-	17400 20000 17400 19400
-Wire Wire Line
-	17400 19400 17375 19400
-Wire Wire Line
-	18900 19400 18900 19150
-Connection ~ 18900 19400
-Wire Wire Line
 	18900 18350 18900 17850
 Wire Wire Line
@@
 Wire Wire Line
 	31300 20800 30275 20800
-Wire Wire Line
-	30275 20800 30275 20450
-Wire Wire Line
-	30275 19350 30275 19950
 Connection ~ 30275 19350
 Wire Wire Line
@@
 	29550 17850 30275 17850
 Wire Wire Line
-	29825 20200 29825 20225
-Wire Wire Line
 	29825 20225 29550 20225
 Wire Wire Line
@@
 Wire Wire Line
 	22400 10150 22775 10150
-Text GLabel 22775 10950 2    140  UnSpc ~ 0
-0VDC
-Wire Wire Line
-	22775 10925 22775 10950
-Wire Wire Line
-	22775 10950 22400 10950
 Text GLabel 22750 12150 2    140  UnSpc ~ 0
 BPLSWY
@@
 Wire Wire Line
 	22400 5650 22775 5650
-Text GLabel 22775 6450 2    140  UnSpc ~ 0
-0VDC
-Wire Wire Line
-	22775 6425 22775 6450
-Wire Wire Line
-	22775 6450 22400 6450
 Text GLabel 22750 7650 2    140  UnSpc ~ 0
 BPLSWY
@@
 Wire Wire Line
 	17150 10150 17525 10150
-Text GLabel 17525 10950 2    140  UnSpc ~ 0
-0VDC
-Wire Wire Line
-	17525 10925 17525 10950
-Wire Wire Line
-	17525 10950 17150 10950
 Text GLabel 17525 5650 2    140  UnSpc ~ 0
 VYF2
 Wire Wire Line
 	17150 5650 17525 5650
-Text GLabel 17525 6450 2    140  UnSpc ~ 0
-0VDC
-Wire Wire Line
-	17525 6425 17525 6450
-Wire Wire Line
-	17525 6450 17150 6450
 Text GLabel 17500 12150 2    140  UnSpc ~ 0
 BPLSWY
@@
 Wire Wire Line
 	11875 10150 12250 10150
-Text GLabel 12250 10950 2    140  UnSpc ~ 0
-0VDC
-Wire Wire Line
-	12250 10925 12250 10950
-Wire Wire Line
-	12250 10950 11875 10950
 Text GLabel 12275 5650 2    140  UnSpc ~ 0
 VYF2
@@
 0VDC
 Wire Wire Line
-	12275 6425 12275 6450
-Wire Wire Line
 	12275 6450 11900 6450
 Text GLabel 12225 12150 2    140  UnSpc ~ 0
@@
 0VDC
 Wire Wire Line
-	6875 10925 6875 10950
-Wire Wire Line
 	6875 10950 6500 10950
 Text GLabel 6875 5650 2    140  UnSpc ~ 0
@@
 0VDC
 Wire Wire Line
-	6875 6425 6875 6450
-Wire Wire Line
 	6875 6450 6500 6450
 Text GLabel 6850 12150 2    140  UnSpc ~ 0
@@
 	21700 26450 21700 25900
 Connection ~ 21700 25900
+Wire Wire Line
+	12225 10950 11875 10950
+Text GLabel 12225 10950 2    140  UnSpc ~ 0
+0VDC
+Wire Wire Line
+	17500 6450 17150 6450
+Text GLabel 17500 6450 2    140  UnSpc ~ 0
+0VDC
+Wire Wire Line
+	17550 10950 17150 10950
+Text GLabel 17550 10950 2    140  UnSpc ~ 0
+0VDC
+Wire Wire Line
+	22775 6450 22400 6450
+Text GLabel 22775 6450 2    140  UnSpc ~ 0
+0VDC
+Wire Wire Line
+	22775 10950 22400 10950
+Text GLabel 22775 10950 2    140  UnSpc ~ 0
+0VDC
+Wire Wire Line
+	30275 19350 30275 19975
+Wire Wire Line
+	30275 20800 30275 20475
+$Comp
+L AGC_DSKY:Transistor-PNP Q10
+U 1 1 5C65279F
+P 30125 20225
+F 0 "Q10" H 30875 20225 130 0000 C CNN
+F 1 "Transistor-PNP" H 30125 20790 130 0001 C CNN
+F 2 "" H 30125 19975 130 0001 C CNN
+F 3 "" H 30125 19975 130 0001 C CNN
+	1    30125 20225
+	1    0    0    -1
+$EndComp
+Wire Wire Line
+	18900 19150 18900 19400
+Wire Wire Line
+	15875 19400 17400 19400
+Connection ~ 18900 19400
+Wire Wire Line
+	18900 19400 18900 20600
+Wire Wire Line
+	17400 20000 17400 19400
+Connection ~ 17400 19400
+Wire Wire Line
+	17400 19400 18900 19400
+Wire Wire Line
+	17400 19400 17400 18925
 $EndSCHEMATC

Commit message: Added CAD transcription for drawing 2005929A (sense amplifier module for erasable memory, B14, for AGC 2003993).  Fixed more (and more-serious) problems than I'm accustomed to in the earlier-generation circuit 2005919A at the same time ... which is curious, since the drawing 2005919A itself was adapted from (namely 2005920B) didn't have any of those errors in it!  Oh, well.
Parts:
- Q3: value Transistor-NPN -> Transistor-PNP; symbol AGC_DSKY:Transistor-NPN -> AGC_DSKY:Transistor-PNP
Connections:
- net 6A/A: now also J2.248; no longer J2.240
- net STROBF: now also Q3.3 (C); no longer Q3.1 (C)
- net at CR2.1 (K): now also Q3.1 (E); no longer Q3.3 (E)
- net at Q2.1 (C): now also R17.1; no longer CR1.2 (A)
- net at Q2.3 (E): now also CR1.2 (A); no longer R17.1
Other:
- note added: "Notes from the Virtual AGC Project:\na) This CAD drawing was adapted from a CAD drawing previously transcribed from \n the original Apollo Program drawing 2005920B, and then cross-checked against \n the original Apollo Program drawing 2005919A. However, this CAD drawing does\n not itself date from the Apollo period. — RSB 2018\nb) The oval pads numbered 101-169 comprise connector J1, while those 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"
- note added: "SENSE AMPLIFIER ASSY DWG NO. 2003981"
- note removed: "Notes from the Virtual AGC Project:\n1. This CAD drawing was adapted from a CAD drawing previously transcribed from \n the original Apollo Program drawing 2005920B, and then cross-checked against \n the original Apollo Program drawing 2005919A. However, this CAD drawing does\n not itself date from the Apollo period. — RSB 2018\n2. The oval pads numbered 101-169 comprise connector J1, while those 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"
- note removed: "SENSE AMPLIFIER ASSY DWG NO. 2003982"
Changed lines of the file:
@@
 EESchema Schematic File Version 5
-LIBS:errors-cache
+LIBS:module-cache
 EELAYER 29 0
 EELAYER END
@@
 	34875 4675 28750 4675
 $Comp
-L AGC_DSKY:Transistor-NPN Q3
+L AGC_DSKY:Transistor-PNP Q3
 U 1 1 5C62FBCA
 P 33600 10475
-F 0 "Q3" H 34125 10650 130 0000 C CNN
-F 1 "Transistor-NPN" H 33600 11040 130 0001 C CNN
+F 0 "Q3" H 34050 10225 130 0000 C CNN
+F 1 "Transistor-PNP" H 33600 11040 130 0001 C CNN
 F 2 "" H 33600 10725 130 0001 C CNN
 F 3 "" H 33600 10725 130 0001 C CNN
 	1    33600 10475
-	1    0    0    -1
+	1    0    0    1
 $EndComp
 $Comp
@@
 U 1 1 5C630F6D
 P 32225 8200
-F 0 "Q2" H 32625 8450 130 0000 C CNN
+F 0 "Q2" H 32675 7950 130 0000 C CNN
 F 1 "Transistor-NPN" H 32225 8765 130 0001 C CNN
 F 2 "" H 32225 8450 130 0001 C CNN
 F 3 "" H 32225 8450 130 0001 C CNN
 	1    32225 8200
-	1    0    0    -1
+	1    0    0    1
 $EndComp
 $Comp
@@
 	34600 9775 35500 9775
 Wire Wire Line
-	33750 11175 33750 10725
-Wire Wire Line
 	34600 11225 34600 12125
 Wire Wire Line
@@
 $Comp
 L AGC_DSKY:ConnectorB8-200 J2
-U 40 1 5E0B4E05
-P 9600 5250
-F 0 "J2" H 9600 5575 140 0001 C CNN
-F 1 "ConnectorB8-200" H 9600 5675 140 0001 C CNN
-F 2 "" H 9600 5725 140 0001 C CNN
-F 3 "" H 9600 5725 140 0001 C CNN
-F 4 "GAR04" H 8875 5175 140 0000 C BNB "Caption"
-	40   9600 5250
+U 48 1 5E0B4E05
+P 9575 5250
+F 0 "J2" H 9575 5575 140 0001 C CNN
+F 1 "ConnectorB8-200" H 9575 5675 140 0001 C CNN
+F 2 "" H 9575 5725 140 0001 C CNN
+F 3 "" H 9575 5725 140 0001 C CNN
+F 4 "GAR04" H 8850 5175 140 0000 C BNB "Caption"
+	48   9575 5250
 	1    0    0    -1
 $EndComp
@@
 	10200 5650 9875 5650
 Wire Wire Line
-	10200 5250 9875 5250
+	10200 5250 9850 5250
 Text GLabel 6875 10150 2    140  UnSpc ~ 0
 VYF1
@@
 REF DWG.
 Text Notes 35700 23300 0    140  ~ 28
-SENSE AMPLIFIER ASSY DWG NO. 2003982
+SENSE AMPLIFIER ASSY DWG NO. 2003981
 $Comp
 L AGC_DSKY:ConnectorB8-200 J2
@@
 1. INTERPRET DRAWING IN ACCORDANCE WITH STANDARDS\n   PRESCRIBED BY MIL-D-70327\n2. RESISTOR VALUES SHALL BE IN OHMS UNLESS OTHERWISE SPECIFIED\n3. CAPACITOR VALUES SHALL BE IN MICROFARADS UNLESS OTHERWISE SPECIFIED\n4. NOMINAL VALUES ARE TO BE SELECTED BY ELECTRICAL TEST, CHART A AND B\n5. ONE, TWO OR THREE DIODES TO BE SELECTED BY ELECTRICAL TEST
 Text Notes 2025 33375 0    140  ~ 28
-Notes from the Virtual AGC Project:\n1. This CAD drawing was adapted from a CAD drawing previously transcribed from \n   the original Apollo Program drawing 2005920B, and then cross-checked against \n   the original Apollo Program drawing 2005919A.  However, this CAD drawing does\n   not itself date from the Apollo period. — RSB 2018\n2. The oval pads numbered 101-169 comprise connector J1, while those numbered\n   201-269 comprise connector J2. — RSB 2018\n3. The CAD drawing differs in the visual appearance of circuits 40611 - 40618, \n   compared to the original drawing.  This was necessary to correctly represent \n   the electrical connectivity for these circuits, since the original drawing provided \n   that information in tabular form rather than using wires or net labels to do so.\n   A separate drawing has been created that matches the visual appearance of the\n   original drawing. — RSB 2018
+Notes from the Virtual AGC Project:\na) This CAD drawing was adapted from a CAD drawing previously transcribed from \n   the original Apollo Program drawing 2005920B, and then cross-checked against \n   the original Apollo Program drawing 2005919A.  However, this CAD drawing does\n   not itself date from the Apollo period. — RSB 2018\nb) The oval pads numbered 101-169 comprise connector J1, while those numbered\n   201-269 comprise connector J2. — RSB 2018\nc) The CAD drawing differs in the visual appearance of circuits 40611 - 40618, \n   compared to the original drawing.  This was necessary to correctly represent \n   the electrical connectivity for these circuits, since the original drawing provided \n   that information in tabular form rather than using wires or net labels to do so.\n   A separate drawing has been created that matches the visual appearance of the\n   original drawing. — RSB 2018
 $Bitmap
 Pos 1725 30500
@@
 Wire Wire Line
 	17400 19400 17400 18925
+Wire Wire Line
+	33750 11175 33750 10725
 $EndSCHEMATC
