File: Schematics/2005922-/2005922--p1of3.sch (KiCad schematic (older format))
At the start: 120 parts, among them Q1 Transistor-PNP, Q10 Transistor-PNP, Q11 Transistor-NPN, Q12 Transistor-NPN, Q13 Transistor-PNP, Q14 Transistor-NPN, Q15 Transistor-NPN, Q16 Transistor-NPN, Q17 Transistor-PNP, Q18 Transistor-NPN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

Commit message: Finished (the first draft of) the transcription of drawing 2005922- (alarm module B8 for AGC 2003200) into KiCad.
Parts:
- added G1: Ground-chassis, symbol AGC_DSKY:Ground-chassis
- added J1: ConnectorB8-100, symbol AGC_DSKY:ConnectorB8-100
- added J2: ConnectorB8-200, symbol AGC_DSKY:ConnectorB8-200
- renumbered R56 to R58
Connections:
- net labels added: 0VDC_135, 0VDC_211, 0VDC_227, BPLUS_124
- wire segments 403 -> 439
Other:
- note added: "1. INTERPET DRAWING IN ACCORDANCE WITH STANDARDS\n PRESCRIBED BY MIL-D-70327\n2. SELECT R3,R11,R12,R93,R94 PER APPLICABLE PS FROM APPROPRIATE CHART"
- note added: "ALARM MODULE ASSY"
- note added: "DWG NO. 2003983"
- note added: "NOTES:"
- note added: "Notes from the Virtual AGC Project:\n1. This CAD drawing was transcribed from the original Apollo Program drawing\n 2005922-, but is not itself orginal to the Apollo Program. — RSB 2018\n2. The original drawing did not indicate reference designators for connectors.\n In this drawing, the oval pads numbered 101-169 comprise connector J1, while\n those numbered 201-269 comprise connector J2. — RSB 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"
- note added: "REF DWG:"

Commit message: Corrected resistor values R54,R55 in drawing 2005922-, which I noticed were wrong whilst proofing drawing 2005028A.
Parts:
- R54, R57: value 10K -> 10
Changed lines of the file:
@@
 P 6450 25950
 F 0 "R54" V 6325 25575 130 0000 C CNN
-F 1 "10K" V 6575 25575 130 0000 C CNN
+F 1 "10" V 6575 25575 130 0000 C CNN
 F 2 "" H 6450 25950 130 0001 C CNN
 F 3 "" H 6450 25950 130 0001 C CNN
@@
 P 8725 25975
 F 0 "R57" V 8600 25600 130 0000 C CNN
-F 1 "10K" V 8850 25600 130 0000 C CNN
+F 1 "10" V 8850 25600 130 0000 C CNN
 F 2 "" H 8725 25975 130 0001 C CNN
 F 3 "" H 8725 25975 130 0001 C CNN

Commit message: Visual fixes made with eelint.  A disconnected global net label was found and corrected.  ERC passes (with the reconnected global net label).  Netlist differs from before, due to reconnected global net label.
Changed lines of the file:
@@
-EESchema Schematic File Version 4
+EESchema Schematic File Version 5
 LIBS:module-cache
 EELAYER 29 0
@@
 	31075 21750 31175 21675
 Wire Wire Line
-	31175 21675 31175 20275
-Wire Wire Line
-	31175 20275 28400 20275
-Wire Wire Line
-	28400 20275 28400 20300
+	31175 21675 31175 20300
+Wire Wire Line
+	31175 20300 28400 20300
 Wire Wire Line
 	28400 20300 26975 20300
@@
 L AGC_DSKY:Ground-chassis G1
 U 1 1 5C5E87AE
-P 5175 14650
-F 0 "G1" H 5415 14663 130 0001 L CNN
-F 1 "Ground-chassis" H 5175 15150 130 0001 C CNN
-F 2 "" H 5175 14650 130 0001 C CNN
-F 3 "" H 5175 14650 130 0001 C CNN
-	1    5175 14650
+P 5175 14625
+F 0 "G1" H 5415 14638 130 0001 L CNN
+F 1 "Ground-chassis" H 5175 15125 130 0001 C CNN
+F 2 "" H 5175 14625 130 0001 C CNN
+F 3 "" H 5175 14625 130 0001 C CNN
+	1    5175 14625
 	1    0    0    -1
 $EndComp
@@
 	4400 14375 5175 14375
 Wire Wire Line
-	5175 14375 5175 14400
-Wire Wire Line
 	4425 16025 4575 16025
