File: Schematics/2005268-/2005268--p2of2.sch (KiCad schematic (older format))
At the start: 66 parts, among them J3 ConnectorA1-300, J4 ConnectorA1-400, U201 D3NOR-+4SW-0VDCA-B_C-E_F, U202 D3NOR-+4SW-0VDCA-_C_-_F_, U203 D3NOR-+4SW-0VDCA-B_C-_F_, U204 D3NOR-+4SW-0VDCA-BAC-_F_, U205 D3NOR-+4SW-0VDCA-BAC-_F_, U206 D3NOR-+4SW-0VDCA-BAC-_F_, U207 D3NOR-+4SW-0VDCA-B_C-FE_, U208 D3NOR-+4SW-0VDCA-BAC-FE_, U209 D3NOR-+4SW-0VDCA-_C_-EDF, U210 D3NOR-+4SW-0VDCA-ACB-DFE, U211 D3NOR-+4SW-0VDCA-BC_-FE_, U212 D3NOR-+4SW-0VDCA-ACB-E_F, U213 D3NOR-+4SW-0VDCA-CB_-_F_, U214 D3NOR-+4SW-0VDCA-CB_-DEF, U215 D3NOR-+4SW-0VDCA-ACB-DEF, U216 D3NOR-+4SW-0VDCA-ACB-DFE, U217 D3NOR-+4SW-0VDCA-BC_-DFE, U218 D3NOR-+4SW-0VDCA-_C_-_F_, U219 D3NOR-+4SW-0VDCA-ABC-_F_, U220 D3NOR-+4SW-0VDCA-ABC-EDF, U221 D3NOR-+4SW-0VDCA-CB_-E_F, U222 D3NOR-+4SW-0VDCA-B_C-FE_, U223 D3NOR-+4SW-0VDCA-B_C-E_F, U224 D3NOR-+4SW-0VDCA-CB_-E_F, U225 D3NOR-+4SW-0VDCA-B_C-FE_, U226 D3NOR-+4SW-0VDCA-_C_-_F_, U227 D3NOR-+4SW-0VDCA-B_C-EF_, U228 D3NOR-+4SW-0VDCA-_C_-E_F, U229 D3NOR-+4SW-0VDCA-BAC-EF_, U230 D3NOR-+4SW-0VDCA-BC_-EF_, U231 D3NOR-+4SW-0VDCA-ABC-E_F, U232 D3NOR-+4SW-0VDCA-B_C-E_F, U233 D3NOR-FAP-0VDCA-expander-B_C-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, U234 D3NOR-+4SW-0VDCA-BAC-FE_, U235 D3NOR-+4SW-0VDCA-B_C-FE_, U236 D3NOR-+4SW-0VDCA-BC_-DFE, U237 D3NOR-+4SW-0VDCA-B_C-EF_, U238 D3NOR-FAP-0VDCA-expander-B_C-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, U239 D3NOR-+4SW-0VDCA-BC_-FE_, U240 D3NOR-+4SW-0VDCA-ACB-E_F, U241 D3NOR-+4SW-0VDCA-CB_-FE_, U242 D3NOR-+4SW-0VDCA-B_C-E_F, U243 D3NOR-FAP-0VDCA-expander-B_C-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, U244 D3NOR-+4SW-0VDCA-BAC-FE_, U245 D3NOR-+4SW-0VDCA-CB_-E_F, U246 D3NOR-+4SW-0VDCA-BC_-E_F, U247 D3NOR-FAP-0VDCA-expander-B_C-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, U248 D3NOR-+4SW-0VDCA-ACB-E_F, U249 D3NOR-+4SW-0VDCA-B_C-FE_, U250 D3NOR-FAP-0VDCA-expander-B_C-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, U251 D3NOR-+4SW-0VDCA-BAC-FE_, U252 D3NOR-FAP-0VDCA-expander-BC_-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, U253 D3NOR-+4SW-0VDCA-CB_-EF_, U254 D3NOR-FAP-0VDCA-expander-ABC-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, U255 D3NOR-+4SW-0VDCA-_C_-_F_, U256 D3NOR-+4SW-0VDCA-B_C-EF_, U257 D3NOR-+4SW-0VDCA-B_C-E_F, U258 D3NOR-+4SW-0VDCA-B_C-E_F, U259 D3NOR-+4SW-0VDCA-ACB-DEF, U260 D3NOR-+4SW-0VDCA-ABC-FE_, X301 ArrowTwiddle, X302 ArrowTwiddle, X303 ArrowTwiddle

Commit message: Added CAD transcription for drawing 2005268- (module A18 for AGC 2003200).  Made a couple of minor, non-electrical fixes to 2005268A (module A18 for AGC 2003993) at the same time.  The netlists are identical and ERC passes.  In fact, I couldn't see any difference between rev - and rev A.
Other:
- note removed: "A REVISED PER TDRR 30754"
