File: Schematics/2005268-/module.sch (KiCad schematic (older format))
At the start: 0 parts

Commit message: Added CAD transcription for drawing 2005268- (module A18 for AGC 2003200).  Made a couple of minor, non-electrical fixes to 2005268A (module A18 for AGC 2003993) at the same time.  The netlists are identical and ERC passes.  In fact, I couldn't see any difference between rev - and rev A.
Other:
- note removed: "A REVISED PER TDRR 30754"
Changed lines of the file:
@@
 U 5B8E7731
 F0 "1" 140
-F1 "2005268A-p1of2.sch" 140
+F1 "2005268--p1of2.sch" 140
 F2 "0VDCA" U R 20700 17550 140
 F3 "+4SW" U R 20700 16425 140
@@
 Text Notes 39925 32475 0    200  ~ 40
 INOUT III
-Wire Notes Line width 6 style solid
-	36839 983  36839 1300
-Wire Notes Line width 6 style solid
-	36461 1300 43500 1300
-Wire Notes Line width 6 style solid
-	36461 983  36461 1300
-Wire Notes Line width 6 style solid
-	37350 982  37350 1299
-Wire Notes Line width 6 style solid
-	40831 983  40831 1300
-Wire Notes Line width 6 style solid
-	41331 983  41331 1300
-Wire Notes Line width 6 style solid
-	41831 983  41831 1300
-Wire Notes Line width 6 style solid
-	42480 983  42480 1300
-Text Notes 36550 1250 0    160  ~ 32
-A      REVISED PER TDRR 30754
 $Comp
 L AGC_DSKY:PWR_FLAG #FLG0104
@@
 U 5B8E7796
 F0 "2" 140
-F1 "2005268A-p2of2.sch" 140
+F1 "2005268--p2of2.sch" 140
 F2 "0VDCA" U L 25125 17550 140
 F3 "+4SW" U L 25125 16425 140
 F4 "FAP" U L 25125 15375 140
 $EndSheet
+Text Label 22075 14325 0    140  ~ 28
++4VDC
+Text Label 22300 15375 0    140  ~ 28
+FAP
+Text Label 22150 16425 0    140  ~ 28
++4SW
+Text Label 22075 17550 0    140  ~ 28
+0VDCA
 $EndSCHEMATC
