File: Schematics/2005104B/module.sch (KiCad schematic (older format))
At the start: 88 parts, among them J1 ConnectorB8-100, J2 ConnectorB8-200, Q10 Transistor-NPN, Q11 Transistor-PNP, Q12 Transistor-NPN, Q13 Transistor-NPN, Q14 Transistor-NPN, Q15 Transistor-NPN, Q16 Transistor-PNP, Q17 Transistor-NPN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

Commit message: Somehow I had left my eelint-based fixups for drawing 2005104B half finished, and the schematic broken.  This was apparently due to my snapKiCad.awk script not handling repositioning of off-grid hierarchical pins within sheet symbols, so I added that functionality to the script.
Connections:
- wire segments 415 -> 413
Other:
- moved on the sheet: CR16, CR17, CR31
