File: Schematics/2005930A/2005930A-p2of3.sch (KiCad schematic (older format))
At the start: 0 parts

Commit message: Added CAD transcription of drawing 2005930A, and made some related corrections to the similar drawing 2005003E.
Other:
- note added: "2005930"
- note added: "A INITIAL RELEASE TDRR 32559"
- note added: "NONE"
- note removed: "2005003"
- note removed: "A REVISED PER TDRR 18681"
- note removed: "B REVISED PER TDRR 19761"
- note removed: "C REVISED PER TDRR 23218"
- note removed: "D"
- note removed: "E"
- note removed: "REVISED PER TDRR 23956\nDR CHK"
Changed lines of the file:
@@
 Comment4 ""
 $EndDescr
-Wire Notes Line style solid
-	27965 920  27965 2650
-Wire Notes Line style solid
-	33500 2175 27965 2175
-Wire Notes Line style solid
-	28464 921  28464 2649
-Wire Notes Line style solid
-	31799 919  31799 2648
-Wire Notes Line style solid
-	32465 920  32465 2649
-Wire Notes Line style solid
-	27965 2650 33500 2650
-Wire Notes Line style solid
-	33510 1716 27975 1716
-Wire Notes Line style solid
-	33506 1438 27971 1438
-Wire Notes Line style solid
-	33502 1169 27967 1169
-Text Notes 28125 1150 0    140  ~ 28
-A   REVISED PER TDRR 18681
-Text Notes 28100 1425 0    140  ~ 28
-B   REVISED PER TDRR 19761
-Text Notes 28100 1700 0    140  ~ 28
-C   REVISED PER TDRR 23218
-Text Notes 28100 2050 0    140  ~ 28
-D
-Text Notes 28125 2500 0    140  ~ 28
-E
-Text Notes 28550 2150 0    130  ~ 26
-REVISED PER TDRR 23956\nDR              CHK
-Text Notes 28525 2625 0    130  ~ 26
-REVISED PER TDRR 23956\nDR              CHK
 Text Notes 29750 19775 0    250  ~ 50
 SCHEMATIC
@@
 MODULE NO. B7
 Text Notes 31000 21125 0    225  ~ 45
-2005003
+2005930
 Text Notes 28325 21100 0    225  ~ 45
 80230
@@
 Wire Notes Line width 50 style solid
 	23900 10950 23850 11200
+Wire Notes Line style solid
+	28465 910  28465 1155
+Wire Notes Line style solid
+	27965 910  27965 1155
+Wire Notes Line style solid
+	33502 1159 27967 1159
+Text Notes 28125 1140 0    140  ~ 28
+A   INITIAL RELEASE TDRR 32559
+Wire Notes Line style solid
+	32465 910  32465 1155
+Wire Notes Line style solid
+	31795 910  31795 1155
+Text Notes 28800 21475 0    140  ~ 28
+NONE
 $EndSCHEMATC
